File: schematic/PCBVersion/1BitFullAdder.sch (KiCad schematic (older format))
At the start: 6 parts, among them U1 74LS86, U2 74LS86, U3 74LS86, U4 74LS08, U5 74LS08, U6 74LS32

Commit message: pcbVersion: kicad alu design
Parts:
- removed U1: 74LS86, Package_DIP:DIP-14_W7.62mm, symbol 74xx:74LS86
- renumbered U2 to U1, U4 to U2, U5 to U4, U6 to U5
Connections:
- net B: now also U1.2, U2.2
- net and: now reaches U2.3, U5.1
- net xor: now reaches U1.3, U3.2, U4.2
Other:
- moved on the sheet: U6A, U8A

Commit message: pcbVersion: regset + alu
Connections:
- net A: now also U1.12, U2.12; no longer U1.1, U2.1
- net B: now also U1.13, U2.13; no longer U1.2, U2.2
- net Cin: now also U3.12, U4.12; no longer U3.1, U4.1
- net Cout: now also U5.11; no longer U5.3
- net Y: now also U3.11; no longer U3.3
- net and: now also U2.11, U5.12; no longer U2.3, U5.1
- net xor: now also U1.11, U3.13, U4.13; no longer U1.3, U3.2, U4.2
- new net: U4.11, U5.13
Changed lines of the file:
@@
 $Descr A4 11693 8268
 encoding utf-8
-Sheet 7 13
+Sheet 5 14
 Title ""
 Date ""
@@
 $Comp
 L 74xx:74LS08 U2
-U 1 1 60149FB6
+U 4 1 60149FB6
 P 4000 2300
 AR Path="/600C5001/60248238/6016C9C5/60149FB6" Ref="U2"  Part="4"
@@
 F 2 "Package_DIP:DIP-14_W7.62mm" H 4000 2300 50  0001 C CNN
 F 3 "http://www.ti.com/lit/gpn/sn74LS08" H 4000 2300 50  0001 C CNN
-	1    4000 2300
+	4    4000 2300
 	1    0    0    -1
 $EndComp
@@
 $Comp
 L 74xx:74LS08 U4
-U 1 1 60149FCA
+U 4 1 60149FCA
 P 5450 2750
 AR Path="/600C5001/60248238/6016C9C5/60149FCA" Ref="U4"  Part="4"
@@
 F 2 "Package_DIP:DIP-14_W7.62mm" H 5450 2750 50  0001 C CNN
 F 3 "http://www.ti.com/lit/gpn/sn74LS08" H 5450 2750 50  0001 C CNN
-	1    5450 2750
+	4    5450 2750
 	1    0    0    -1
 $EndComp
 $Comp
 L 74xx:74LS86 U3
-U 1 1 60149FD6
+U 4 1 60149FD6
 P 5600 1800
 AR Path="/600C5001/60248238/6016C9C5/60149FD6" Ref="U3"  Part="4"
@@
 F 2 "Package_DIP:DIP-14_W7.62mm" H 5600 1800 50  0001 C CNN
 F 3 "74xx/74ls86.pdf" H 5600 1800 50  0001 C CNN
-	1    5600 1800
+	4    5600 1800
 	1    0    0    -1
 $EndComp
@@
 $Comp
 L 74xx:74LS32 U5
-U 1 1 60149FEF
+U 4 1 60149FEF
 P 6300 2450
 AR Path="/600C5001/60248238/6016C9C5/60149FEF" Ref="U5"  Part="4"
@@
 F 2 "Package_DIP:DIP-14_W7.62mm" H 6300 2450 50  0001 C CNN
 F 3 "http://www.ti.com/lit/gpn/sn74LS32" H 6300 2450 50  0001 C CNN
-	1    6300 2450
+	4    6300 2450
 	1    0    0    -1
 $EndComp
 $Comp
 L 74xx:74LS86 U1
-U 1 1 60149FD0
+U 4 1 60149FD0
 P 4100 2850
 AR Path="/600C5001/60248238/6016C9C5/60149FD0" Ref="U1"  Part="4"
@@
 F 2 "Package_DIP:DIP-14_W7.62mm" H 4100 2850 50  0001 C CNN
 F 3 "74xx/74ls86.pdf" H 4100 2850 50  0001 C CNN
-	1    4100 2850
+	4    4100 2850
 	1    0    0    -1
 $EndComp

Commit message: pcbversion: ram, started pc
Connections:
- net A: now also U1.1, U2.1; no longer U1.12, U2.12
- net B: now also U1.2, U2.2; no longer U1.13, U2.13
- net Cin: now also U3.1, U4.1; no longer U3.12, U4.12
- net Cout: now also U5.3; no longer U5.11
- net Y: now also U3.3; no longer U3.11
- net and: now also U2.3, U5.1; no longer U2.11, U5.12
- net xor: now also U1.3, U3.2, U4.2; no longer U1.11, U3.13, U4.13
- new net: U4.3, U5.2
Changed lines of the file:
@@
 $Descr A4 11693 8268
 encoding utf-8
-Sheet 5 14
+Sheet 13 18
 Title ""
 Date ""
@@
 $Comp
 L 74xx:74LS08 U2
-U 4 1 60149FB6
+U 1 1 60149FB6
 P 4000 2300
 AR Path="/600C5001/60248238/6016C9C5/60149FB6" Ref="U2"  Part="4"
@@
 AR Path="/600C5001/60260EB9/6016C4DC/60149FB6" Ref="U7"  Part="2"
 AR Path="/600C5001/60260EB9/6014201D/60149FB6" Ref="U7"  Part="1"
-F 0 "U7" H 4000 2625 50  0000 C CNN
+F 0 "U2" H 4000 2625 50  0000 C CNN
 F 1 "74LS08" H 4000 2534 50  0000 C CNN
 F 2 "Package_DIP:DIP-14_W7.62mm" H 4000 2300 50  0001 C CNN
 F 3 "http://www.ti.com/lit/gpn/sn74LS08" H 4000 2300 50  0001 C CNN
-	4    4000 2300
+	1    4000 2300
 	1    0    0    -1
 $EndComp
@@
 $Comp
 L 74xx:74LS08 U4
-U 4 1 60149FCA
+U 1 1 60149FCA
 P 5450 2750
 AR Path="/600C5001/60248238/6016C9C5/60149FCA" Ref="U4"  Part="4"
@@
 AR Path="/600C5001/60260EB9/6016C4DC/60149FCA" Ref="U9"  Part="2"
 AR Path="/600C5001/60260EB9/6014201D/60149FCA" Ref="U9"  Part="1"
-F 0 "U9" H 5450 3075 50  0000 C CNN
+F 0 "U4" H 5450 3075 50  0000 C CNN
 F 1 "74LS08" H 5450 2984 50  0000 C CNN
 F 2 "Package_DIP:DIP-14_W7.62mm" H 5450 2750 50  0001 C CNN
 F 3 "http://www.ti.com/lit/gpn/sn74LS08" H 5450 2750 50  0001 C CNN
-	4    5450 2750
+	1    5450 2750
 	1    0    0    -1
 $EndComp
 $Comp
 L 74xx:74LS86 U3
-U 4 1 60149FD6
+U 1 1 60149FD6
 P 5600 1800
 AR Path="/600C5001/60248238/6016C9C5/60149FD6" Ref="U3"  Part="4"
@@
 AR Path="/600C5001/60260EB9/6016C4DC/60149FD6" Ref="U8"  Part="2"
 AR Path="/600C5001/60260EB9/6014201D/60149FD6" Ref="U8"  Part="1"
-F 0 "U8" H 5600 2125 50  0000 C CNN
+F 0 "U3" H 5600 2125 50  0000 C CNN
 F 1 "74LS86" H 5600 2034 50  0000 C CNN
 F 2 "Package_DIP:DIP-14_W7.62mm" H 5600 1800 50  0001 C CNN
 F 3 "74xx/74ls86.pdf" H 5600 1800 50  0001 C CNN
-	4    5600 1800
+	1    5600 1800
 	1    0    0    -1
 $EndComp
@@
 $Comp
 L 74xx:74LS32 U5
-U 4 1 60149FEF
+U 1 1 60149FEF
 P 6300 2450
 AR Path="/600C5001/60248238/6016C9C5/60149FEF" Ref="U5"  Part="4"
@@
 AR Path="/600C5001/60260EB9/6016C4DC/60149FEF" Ref="U10"  Part="2"
 AR Path="/600C5001/60260EB9/6014201D/60149FEF" Ref="U10"  Part="1"
-F 0 "U10" H 6300 2775 50  0000 C CNN
+F 0 "U5" H 6300 2775 50  0000 C CNN
 F 1 "74LS32" H 6300 2684 50  0000 C CNN
 F 2 "Package_DIP:DIP-14_W7.62mm" H 6300 2450 50  0001 C CNN
 F 3 "http://www.ti.com/lit/gpn/sn74LS32" H 6300 2450 50  0001 C CNN
-	4    6300 2450
+	1    6300 2450
 	1    0    0    -1
 $EndComp
 $Comp
 L 74xx:74LS86 U1
-U 4 1 60149FD0
+U 1 1 60149FD0
 P 4100 2850
 AR Path="/600C5001/60248238/6016C9C5/60149FD0" Ref="U1"  Part="4"
@@
 AR Path="/600C5001/60260EB9/6016C4DC/60149FD0" Ref="U6"  Part="2"
 AR Path="/600C5001/60260EB9/6014201D/60149FD0" Ref="U6"  Part="1"
-F 0 "U6" H 4100 3175 50  0000 C CNN
+F 0 "U1" H 4100 3175 50  0000 C CNN
 F 1 "74LS86" H 4100 3084 50  0000 C CNN
 F 2 "Package_DIP:DIP-14_W7.62mm" H 4100 2850 50  0001 C CNN
 F 3 "74xx/74ls86.pdf" H 4100 2850 50  0001 C CNN
-	4    4100 2850
+	1    4100 2850
 	1    0    0    -1
 $EndComp
