File: schematic/PCBVersion/4BitFullAdder.sch (KiCad schematic (older format))
At the start: 6 parts, among them U1 74LS86, U2 74LS86, U3 74LS86, U4 74LS08, U5 74LS08, U6 74LS32

Commit message: pcbVersion: kicad alu design
Parts:
- removed U1: 74LS86, Package_DIP:DIP-14_W7.62mm, symbol 74xx:74LS86
- renumbered U2 to U1, U4 to U2, U5 to U4, U6 to U5
Other:
- moved on the sheet: U7E, U8E

Commit message: pcbVersion: regset + alu
Changed lines of the file:
@@
 $Descr A4 11693 8268
 encoding utf-8
-Sheet 8 13
+Sheet 9 14
 Title "ALU"
 Date "2021-01-20"
@@
 AR Path="/600C5001/60248238/601C37F5" Ref="#PWR013"  Part="1"
 AR Path="/600C5001/60260EB9/601C37F5" Ref="#PWR023"  Part="1"
-F 0 "#PWR023" H 5650 850 50  0001 C CNN
+F 0 "#PWR013" H 5650 850 50  0001 C CNN
 F 1 "+5V" H 5665 1173 50  0000 C CNN
 F 2 "" H 5650 1000 50  0001 C CNN
@@
 AR Path="/600C5001/60248238/601C25DD" Ref="#PWR011"  Part="1"
 AR Path="/600C5001/60260EB9/601C25DD" Ref="#PWR021"  Part="1"
-F 0 "#PWR021" H 5000 850 50  0001 C CNN
+F 0 "#PWR011" H 5000 850 50  0001 C CNN
 F 1 "+5V" H 5015 1173 50  0000 C CNN
 F 2 "" H 5000 1000 50  0001 C CNN
@@
 AR Path="/600C5001/60248238/60189268" Ref="U4"  Part="5"
 AR Path="/600C5001/60260EB9/60189268" Ref="U9"  Part="5"
-F 0 "U9" H 5230 1596 50  0000 L CNN
+F 0 "U4" H 5230 1596 50  0000 L CNN
 F 1 "74LS08" H 5230 1505 50  0000 L CNN
 F 2 "Package_DIP:DIP-14_W7.62mm" H 5000 1550 50  0001 C CNN
@@
 AR Path="/600C5001/60248238/601A9C21" Ref="#PWR06"  Part="1"
 AR Path="/600C5001/60260EB9/601A9C21" Ref="#PWR016"  Part="1"
-F 0 "#PWR016" H 2900 1850 50  0001 C CNN
+F 0 "#PWR06" H 2900 1850 50  0001 C CNN
 F 1 "GND" H 2905 1927 50  0000 C CNN
 F 2 "" H 2900 2100 50  0001 C CNN
@@
 AR Path="/600C5001/60248238/601A9101" Ref="#PWR08"  Part="1"
 AR Path="/600C5001/60260EB9/601A9101" Ref="#PWR018"  Part="1"
-F 0 "#PWR018" H 3650 1850 50  0001 C CNN
+F 0 "#PWR08" H 3650 1850 50  0001 C CNN
 F 1 "GND" H 3655 1927 50  0000 C CNN
 F 2 "" H 3650 2100 50  0001 C CNN
@@
 AR Path="/600C5001/60248238/601A8BDE" Ref="#PWR010"  Part="1"
 AR Path="/600C5001/60260EB9/601A8BDE" Ref="#PWR020"  Part="1"
-F 0 "#PWR020" H 4300 1850 50  0001 C CNN
+F 0 "#PWR010" H 4300 1850 50  0001 C CNN
 F 1 "GND" H 4305 1927 50  0000 C CNN
 F 2 "" H 4300 2100 50  0001 C CNN
@@
 AR Path="/600C5001/60248238/601A8769" Ref="#PWR012"  Part="1"
 AR Path="/600C5001/60260EB9/601A8769" Ref="#PWR022"  Part="1"
-F 0 "#PWR022" H 5000 1850 50  0001 C CNN
+F 0 "#PWR012" H 5000 1850 50  0001 C CNN
 F 1 "GND" H 5005 1927 50  0000 C CNN
 F 2 "" H 5000 2100 50  0001 C CNN
@@
 AR Path="/600C5001/60248238/601A81A4" Ref="#PWR014"  Part="1"
 AR Path="/600C5001/60260EB9/601A81A4" Ref="#PWR024"  Part="1"
-F 0 "#PWR024" H 5650 1850 50  0001 C CNN
+F 0 "#PWR014" H 5650 1850 50  0001 C CNN
 F 1 "GND" H 5655 1927 50  0000 C CNN
 F 2 "" H 5650 2100 50  0001 C CNN
@@
 AR Path="/600C5001/60248238/601A601F" Ref="#PWR09"  Part="1"
 AR Path="/600C5001/60260EB9/601A601F" Ref="#PWR019"  Part="1"
-F 0 "#PWR019" H 4300 850 50  0001 C CNN
+F 0 "#PWR09" H 4300 850 50  0001 C CNN
 F 1 "+5V" H 4315 1173 50  0000 C CNN
 F 2 "" H 4300 1000 50  0001 C CNN
@@
 AR Path="/600C5001/60248238/601A5A36" Ref="#PWR07"  Part="1"
 AR Path="/600C5001/60260EB9/601A5A36" Ref="#PWR017"  Part="1"
-F 0 "#PWR017" H 3650 850 50  0001 C CNN
+F 0 "#PWR07" H 3650 850 50  0001 C CNN
 F 1 "+5V" H 3665 1173 50  0000 C CNN
 F 2 "" H 3650 1000 50  0001 C CNN
@@
 AR Path="/600C5001/60248238/601A53ED" Ref="#PWR05"  Part="1"
 AR Path="/600C5001/60260EB9/601A53ED" Ref="#PWR015"  Part="1"
-F 0 "#PWR015" H 2900 850 50  0001 C CNN
+F 0 "#PWR05" H 2900 850 50  0001 C CNN
 F 1 "+5V" H 2915 1173 50  0000 C CNN
 F 2 "" H 2900 1000 50  0001 C CNN
@@
 AR Path="/600C5001/60248238/6018B67E" Ref="U5"  Part="5"
 AR Path="/600C5001/60260EB9/6018B67E" Ref="U10"  Part="5"
-F 0 "U10" H 5880 1596 50  0000 L CNN
+F 0 "U5" H 5880 1596 50  0000 L CNN
 F 1 "74LS32" H 5880 1505 50  0000 L CNN
 F 2 "Package_DIP:DIP-14_W7.62mm" H 5650 1550 50  0001 C CNN
@@
 AR Path="/600C5001/60248238/60186DED" Ref="U2"  Part="5"
 AR Path="/600C5001/60260EB9/60186DED" Ref="U7"  Part="5"
-F 0 "U7" H 3880 1596 50  0000 L CNN
+F 0 "U2" H 3880 1596 50  0000 L CNN
 F 1 "74LS08" H 3880 1505 50  0000 L CNN
 F 2 "Package_DIP:DIP-14_W7.62mm" H 3650 1550 50  0001 C CNN
@@
 AR Path="/600C5001/60248238/6018470D" Ref="U3"  Part="5"
 AR Path="/600C5001/60260EB9/6018470D" Ref="U8"  Part="5"
-F 0 "U8" H 4530 1596 50  0000 L CNN
+F 0 "U3" H 4530 1596 50  0000 L CNN
 F 1 "74LS86" H 4530 1505 50  0000 L CNN
 F 2 "Package_DIP:DIP-14_W7.62mm" H 4300 1550 50  0001 C CNN
@@
 AR Path="/600C5001/60248238/601820B8" Ref="U1"  Part="5"
 AR Path="/600C5001/60260EB9/601820B8" Ref="U6"  Part="5"
-F 0 "U6" H 3130 1596 50  0000 L CNN
+F 0 "U1" H 3130 1596 50  0000 L CNN
 F 1 "74LS86" H 3130 1505 50  0000 L CNN
 F 2 "Package_DIP:DIP-14_W7.62mm" H 2900 1550 50  0001 C CNN
