File: schematic/PCBVersion/Alu.sch (KiCad schematic (older format))
At the start: 8 parts, among them U11 74LS86, U12 74LS86, U13 74LS157, U14 74LS157, U15 74LS157, U16 74LS157, U17 74LS157, U18 74LS157

Commit message: pcbVersion: regset + alu
Parts:
- added U29: 74LS377, Package_DIP:DIP-20_W7.62mm, symbol 74xx:74LS377
- added U36: 74LS245, Package_DIP:DIP-20_W7.62mm, symbol 74xx:74LS245
Connections:
- net +5V: now also U15.16 (VCC), U29.20 (VCC), U36.1 (A->B), U36.20 (VCC); no longer U11.7 (GND), U12.7 (GND), U13.15 (E), U13.8 (GND), U14.15 (E), U14.8 (GND), U15.15 (E), U15.8 (GND), U16.15 (E), U16.8 (GND), U17.15 (E), U17.8 (GND), U18.15 (E), U18.8 (GND)
- net y0: now also U36.18 (B0); no longer U17.4 (Za)
- net y1: now also U36.17 (B1); no longer U17.7 (Zb)
- net y2: now also U36.16 (B2); no longer U17.9 (Zc)
- net y3: now also U36.15 (B3); no longer U17.12 (Zd)
- net y4: now also U36.14 (B4); no longer U18.4 (Za)
- net y5: now also U36.13 (B5); no longer U18.7 (Zb)
- net y6: now also U36.12 (B6); no longer U18.9 (Zc)
- net y7: now also U36.11 (B7); no longer U18.12 (Zd)
- new net: U29.12 (Q4), U36.6 (A4)
- new net: U18.4 (Za), U29.13 (D4)
- new net: U18.7 (Zb), U29.14 (D5)
- new net: U29.15 (Q5), U36.7 (A5)
- new net: U29.16 (Q6), U36.8 (A6)
- new net: U18.9 (Zc), U29.17 (D6)
- new net: U18.12 (Zd), U29.18 (D7)
- new net: U29.19 (Q7), U36.9 (A7)
- new net: U29.2 (Q0), U36.2 (A0)
- new net: U17.4 (Za), U29.3 (D0)
- new net: U17.7 (Zb), U29.4 (D1)
- new net: U29.5 (Q1), U36.3 (A1)
- new net: U29.6 (Q2), U36.4 (A2)
- new net: U17.9 (Zc), U29.7 (D2)
- new net: U17.12 (Zd), U29.8 (D3)
- new net: U29.9 (Q3), U36.5 (A3)
- new net GND: U11.7 (GND), U12.7 (GND), U13.15 (E), U13.8 (GND), U14.15 (E), U14.8 (GND), U15.15 (E), U15.8 (GND), U16.15 (E), U16.8 (GND), U17.15 (E), U17.8 (GND), U18.15 (E), U18.8 (GND), U29.10 (GND), U36.10 (GND)
- new net clk: U29.11 (CP)
- new net ctrlAluNOE: U36.19 (CE)
- new net ctrlAluNWrY: U29.1 (~E)
- no-connect marks 0 -> 1
Other:
- moved on the sheet: U11A, U11B, U11C, U11D, U11E, U12A, U12B, U12C, U12D, U12E, U13, U14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

Commit message: pcbversion: ram, started pc
Parts:
- added D1, D2, D3, D4, D5, D6, D7, D8: LED, LED_THT:LED_D3.0mm, symbol Device:LED
- added R1, R2, R3, R4, R5, R6, R7, R8: 1k, Resistor_THT:R_Axial_DIN0207_L6.3mm_D2.5mm_P7.62mm_Horizontal, symbol Device:R
- added U41, U42: 74LS32, Package_DIP:DIP-14_W7.62mm, symbol 74xx:74LS32
Connections:
- net +5V: now also U41.14 (VCC), U42.14 (VCC)
- net GND: now also D1.1 (K), D2.1 (K), D3.1 (K), D4.1 (K), D5.1 (K), D6.1 (K), D7.1 (K), D8.1 (K), U41.12, U41.13, U41.7 (GND), U42.7 (GND)
- net at U29.12 (Q4), U36.6 (A4): now also R4.2, U41.2
- net at U29.15 (Q5), U36.7 (A5): now also R3.2, U41.5
- net at U29.16 (Q6), U36.8 (A6): now also R2.2, U41.10
- net flagNegative: now reaches U29.19 (Q7), U36.9 (A7)
- net flagNegative: now also R1.2, U41.9
- net at U29.2 (Q0), U36.2 (A0): now also R8.2, U42.2
- net at U29.5 (Q1), U36.3 (A1): now also R7.2, U42.5
- net at U29.6 (Q2), U36.4 (A2): now also R6.2, U42.10
- net at U29.9 (Q3), U36.5 (A3): now also R5.2, U42.13
- net ctrlAluNWrY renamed ctrlAluYNWE
- new net: U42.1, U42.6
- new net: U42.4, U42.8
- new net: U42.11, U42.9
- new net: U41.3, U42.12
- new net: U41.1, U41.6
- new net: U41.4, U41.8
- new net: D8.2 (A), R8.1
- new net: D7.2 (A), R7.1
- new net: D6.2 (A), R6.1
- new net: D5.2 (A), R5.1
- new net: D4.2 (A), R4.1
- new net: D3.2 (A), R3.1
- new net: D2.2 (A), R2.1
- new net: D1.2 (A), R1.1
- new net flagNZero: U42.3
- no-connect marks 1 -> 2
Other:
- moved on the sheet: U11A, U11B, U11C, U11D, U11E, U12A, U12B, U12C, U12D, U12E, U13, U14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
