File: schematic/PCBVersion/Regset.sch (KiCad schematic (older format))
At the start: 6 parts, among them U30 74LS377, U31 74LS377, U32 74LS157, U33 74LS157, U34 74LS257, U35 74LS257

Commit message: pcbversion: ram, started pc
Parts:
- added D10, D11, D12, D13, D14, D15, D16, D17, D18, D19, D20, D21, D22, D23, D24, D9: LED, LED_THT:LED_D3.0mm, symbol Device:LED
- added R10, R11, R12, R13, R14, R15, R16, R17, R18, R19, R20, R21, R22, R23, R24, R9: 1k, Resistor_THT:R_Axial_DIN0207_L6.3mm_D2.5mm_P7.62mm_Horizontal, symbol Device:R
Connections:
- net GND: now also D10.1 (K), D11.1 (K), D12.1 (K), D13.1 (K), D14.1 (K), D15.1 (K), D16.1 (K), D17.1 (K), D18.1 (K), D19.1 (K), D20.1 (K), D21.1 (K), D22.1 (K), D23.1 (K), D24.1 (K), D9.1 (K)
- net r00: now also R9.2
- net r01: now also R10.2
- net r02: now also R11.2
- net r03: now also R12.2
- net r04: now also R13.2
- net r05: now also R14.2
- net r06: now also R15.2
- net r07: now also R16.2
- net r10: now also R17.2
- net r11: now also R18.2
- net r12: now also R19.2
- net r13: now also R20.2
- net r14: now also R21.2
- net r15: now also R22.2
- net r16: now also R23.2
- net r17: now also R24.2
- net ctrlReg0NWr renamed ctrlReg0NWE
- net ctrlReg1NWr renamed ctrlReg1NWE
- new net: D9.2 (A), R9.1
- new net: D10.2 (A), R10.1
- new net: D11.2 (A), R11.1
- new net: D12.2 (A), R12.1
- new net: D13.2 (A), R13.1
- new net: D14.2 (A), R14.1
- new net: D15.2 (A), R15.1
- new net: D16.2 (A), R16.1
- new net: D17.2 (A), R17.1
- new net: D18.2 (A), R18.1
- new net: D19.2 (A), R19.1
- new net: D20.2 (A), R20.1
- new net: D21.2 (A), R21.1
- new net: D22.2 (A), R22.1
- new net: D23.2 (A), R23.1
- new net: D24.2 (A), R24.1
