File: schematic/PCBVersion/Clock.sch (KiCad schematic (older format))
At the start: 16 parts, among them SW1 SW_Push, U50 NA555P, U51 NA555P

Commit message: pcbVersion: kinda done
Parts:
- C1, C3, C4, C5: footprint (none) -> Capacitor_THT:C_Radial_D6.3mm_H5.0mm_P2.50mm
- C2: footprint (none) -> Capacitor_THT:CP_Radial_D5.0mm_P2.50mm
- R51, R52, R53, R54, R55, R56, R57: footprint (none) -> Resistor_THT:R_Axial_DIN0207_L6.3mm_D2.5mm_P7.62mm_Horizontal
- RV1: footprint (none) -> Potentiometer_THT:Potentiometer_Bourns_PTV09A-1_Single_Vertical
- SW1: footprint (none) -> Button_Switch_THT:SW_PUSH_6mm
Changed lines of the file:
@@
 F 0 "R57" H 6220 2346 50  0000 L CNN
 F 1 "1k" H 6220 2255 50  0000 L CNN
-F 2 "" V 6080 2300 50  0001 C CNN
+F 2 "Resistor_THT:R_Axial_DIN0207_L6.3mm_D2.5mm_P7.62mm_Horizontal" V 6080 2300 50  0001 C CNN
 F 3 "~" H 6150 2300 50  0001 C CNN
 	1    6150 2300
@@
 F 0 "C1" H 4242 2696 50  0000 L CNN
 F 1 "0.01u" H 4242 2605 50  0000 L CNN
-F 2 "" H 4150 2650 50  0001 C CNN
+F 2 "Capacitor_THT:C_Radial_D6.3mm_H5.0mm_P2.50mm" H 4150 2650 50  0001 C CNN
 F 3 "~" H 4150 2650 50  0001 C CNN
 	1    4150 2650
@@
 F 0 "C2" H 5941 3496 50  0000 L CNN
 F 1 "0.1u" H 5941 3405 50  0000 L CNN
-F 2 "" H 5850 3450 50  0001 C CNN
+F 2 "Capacitor_THT:CP_Radial_D5.0mm_P2.50mm" H 5850 3450 50  0001 C CNN
 F 3 "~" H 5850 3450 50  0001 C CNN
 	1    5850 3450
@@
 F 0 "RV1" H 5780 3046 50  0000 R CNN
 F 1 "1M" H 5780 2955 50  0000 R CNN
-F 2 "" H 5850 3000 50  0001 C CNN
+F 2 "Potentiometer_THT:Potentiometer_Bourns_PTV09A-1_Single_Vertical" H 5850 3000 50  0001 C CNN
 F 3 "~" H 5850 3000 50  0001 C CNN
 	1    5850 3000
@@
 F 0 "R52" H 6220 2846 50  0000 L CNN
 F 1 "1k" H 6220 2755 50  0000 L CNN
-F 2 "" V 6080 2800 50  0001 C CNN
+F 2 "Resistor_THT:R_Axial_DIN0207_L6.3mm_D2.5mm_P7.62mm_Horizontal" V 6080 2800 50  0001 C CNN
 F 3 "~" H 6150 2800 50  0001 C CNN
 	1    6150 2800
@@
 F 0 "R56" H 9820 2246 50  0000 L CNN
 F 1 "1M" H 9820 2155 50  0000 L CNN
-F 2 "" V 9680 2200 50  0001 C CNN
+F 2 "Resistor_THT:R_Axial_DIN0207_L6.3mm_D2.5mm_P7.62mm_Horizontal" V 9680 2200 50  0001 C CNN
 F 3 "~" H 9750 2200 50  0001 C CNN
 	1    9750 2200
@@
 F 0 "C3" H 7842 2596 50  0000 L CNN
 F 1 "0.01u" H 7842 2505 50  0000 L CNN
-F 2 "" H 7750 2550 50  0001 C CNN
+F 2 "Capacitor_THT:C_Radial_D6.3mm_H5.0mm_P2.50mm" H 7750 2550 50  0001 C CNN
 F 3 "~" H 7750 2550 50  0001 C CNN
 	1    7750 2550
@@
 F 0 "R51" H 5820 1946 50  0000 L CNN
 F 1 "10M" H 5820 1855 50  0000 L CNN
-F 2 "" V 5680 1900 50  0001 C CNN
+F 2 "Resistor_THT:R_Axial_DIN0207_L6.3mm_D2.5mm_P7.62mm_Horizontal" V 5680 1900 50  0001 C CNN
 F 3 "~" H 5750 1900 50  0001 C CNN
 	1    5750 1900
@@
 F 0 "R55" H 9370 1846 50  0000 L CNN
 F 1 "10M" H 9370 1755 50  0000 L CNN
-F 2 "" V 9230 1800 50  0001 C CNN
+F 2 "Resistor_THT:R_Axial_DIN0207_L6.3mm_D2.5mm_P7.62mm_Horizontal" V 9230 1800 50  0001 C CNN
 F 3 "~" H 9300 1800 50  0001 C CNN
 	1    9300 1800
@@
 F 0 "SW1" H 7550 2535 50  0000 C CNN
 F 1 "SW_Push" H 7550 2444 50  0000 C CNN
-F 2 "" H 7550 2450 50  0001 C CNN
+F 2 "Button_Switch_THT:SW_PUSH_6mm" H 7550 2450 50  0001 C CNN
 F 3 "~" H 7550 2450 50  0001 C CNN
 	1    7550 2250
@@
 F 0 "C4" H 8092 2296 50  0000 L CNN
 F 1 "0.1u" H 8092 2205 50  0000 L CNN
-F 2 "" H 8000 2250 50  0001 C CNN
+F 2 "Capacitor_THT:C_Radial_D6.3mm_H5.0mm_P2.50mm" H 8000 2250 50  0001 C CNN
 F 3 "~" H 8000 2250 50  0001 C CNN
 	1    8000 2250
@@
 F 0 "R53" H 7870 2146 50  0000 L CNN
 F 1 "1k" H 7870 2055 50  0000 L CNN
-F 2 "" V 7730 2100 50  0001 C CNN
+F 2 "Resistor_THT:R_Axial_DIN0207_L6.3mm_D2.5mm_P7.62mm_Horizontal" V 7730 2100 50  0001 C CNN
 F 3 "~" H 7800 2100 50  0001 C CNN
 	1    7800 2100
@@
 F 0 "R54" H 8220 2146 50  0000 L CNN
 F 1 "1k" H 8220 2055 50  0000 L CNN
-F 2 "" V 8080 2100 50  0001 C CNN
+F 2 "Resistor_THT:R_Axial_DIN0207_L6.3mm_D2.5mm_P7.62mm_Horizontal" V 8080 2100 50  0001 C CNN
 F 3 "~" H 8150 2100 50  0001 C CNN
 	1    8150 2100
@@
 F 0 "C5" H 9342 2796 50  0000 L CNN
 F 1 "0.1u" H 9342 2705 50  0000 L CNN
-F 2 "" H 9250 2750 50  0001 C CNN
+F 2 "Capacitor_THT:C_Radial_D6.3mm_H5.0mm_P2.50mm" H 9250 2750 50  0001 C CNN
 F 3 "~" H 9250 2750 50  0001 C CNN
 	1    9250 2750
