File: schematic/PCBVersion/Control.sch (KiCad schematic (older format))
At the start: 43 parts, among them U43 74LS377, U44 74LS273, U45 74LS273, U46 74LS08, U47 74LS86, U48 28C64, U49 28C64

Commit message: pcbVersion: kinda done
Parts:
- added D51: instrNWE, LED_THT:LED_D3.0mm, symbol Device:LED
- added R58: 1k, Resistor_THT:R_Axial_DIN0207_L6.3mm_D2.5mm_P7.62mm_Horizontal, symbol Device:R
Connections:
- net GND: now also D51.1 (K)
- net ctrlInstrNWE: now also R58.2
- net ctrlPCLoad: now reaches U49.13 (D2)
- net ctrlPCLoad: now also R45.2
- net ctrlPCNOE: now reaches U49.17 (D5)
- net ctrlPCNOE: now also R48.2
- new net: D51.2 (A), R58.1
- no-connect marks 14 -> 10
Other:
- moved on the sheet: D33, D34, D35, D36, D37, D38, D39, D40, D41, D42, D43, D44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
