File: schematic/PCBVersion/PCBVersion.kicad_pcb (KiCad board)
At the start: 2 copper layers, 17 parts, among them J1 Conn_01x08_FemaleOutput, J2 Conn_01x08_FemaleOutput, J3 C, J4 Conn_01x01_FemaleInput, J5 Conn_01x08_FemaleInput, U1 74LS86, U10 74LS08, U11 74LS08, U12 74LS32, U2 74LS86, U3 74LS86, U4 74LS08, U5 74LS08, U6 74LS32, U7 74LS86, U8 74LS86, U9 74LS86

Commit message: pcbversion: ram, started pc
Parts:
- removed J1, J2: Conn_01x08_FemaleOutput, Connector_PinHeader_2.54mm:PinHeader_1x08_P2.54mm_Vertical
- removed J3: C, Connector_PinHeader_2.54mm:PinHeader_1x01_P2.54mm_Vertical
- removed J4: Conn_01x01_FemaleInput, Connector_PinHeader_2.54mm:PinHeader_1x01_P2.54mm_Vertical
- removed J5: Conn_01x08_FemaleInput, Connector_PinHeader_2.54mm:PinHeader_1x08_P2.54mm_Vertical
- added D1: LED, LED_THT:LED_D3.0mm, F.Cu at (88.4, 52.1)
- added D10: LED, LED_THT:LED_D3.0mm, F.Cu at (247.6, 57.6)
- added D11: LED, LED_THT:LED_D3.0mm, F.Cu at (262.7, 24.6)
- added D12: LED, LED_THT:LED_D3.0mm, F.Cu at (229.9, 54.6)
- added D13: LED, LED_THT:LED_D3.0mm, F.Cu at (251.6, 46.5)
- added D14: LED, LED_THT:LED_D3.0mm, F.Cu at (268.6, 24.6)
- added D15: LED, LED_THT:LED_D3.0mm, F.Cu at (262.7, 30.1)
- added D16: LED, LED_THT:LED_D3.0mm, F.Cu at (235.8, 54.6)
- added D17: LED, LED_THT:LED_D3.0mm, F.Cu at (262.7, 35.7)
- added D18: LED, LED_THT:LED_D3.0mm, F.Cu at (235.8, 60.1)
- added D19: LED, LED_THT:LED_D3.0mm, F.Cu at (241.7, 50.5)
- added D2: LED, LED_THT:LED_D3.0mm, F.Cu at (77.6, 64.2)
- added D20: LED, LED_THT:LED_D3.0mm, F.Cu at (241.7, 56.1)
- added D21: LED, LED_THT:LED_D3.0mm, F.Cu at (247.6, 52.0)
- added D22: LED, LED_THT:LED_D3.0mm, F.Cu at (229.9, 60.1)
- added D23: LED, LED_THT:LED_D3.0mm, F.Cu at (268.6, 30.1)
- added D24: LED, LED_THT:LED_D3.0mm, F.Cu at (241.7, 61.6)
- added D25: LED, LED_THT:LED_D3.0mm, F.Cu at (152.6, 59.7)
- added D26: LED, LED_THT:LED_D3.0mm, F.Cu at (187.9, 24.6)
- added D27: LED, LED_THT:LED_D3.0mm, F.Cu at (171.1, 44.0)
- added D28: LED, LED_THT:LED_D3.0mm, F.Cu at (182.0, 24.6)
- added D29: LED, LED_THT:LED_D3.0mm, F.Cu at (171.2, 38.2)
- added D3: LED, LED_THT:LED_D3.0mm, F.Cu at (83.5, 58.6)
- added D30: LED, LED_THT:LED_D3.0mm, F.Cu at (177.1, 32.7)
- added D31: LED, LED_THT:LED_D3.0mm, F.Cu at (160.3, 51.6)
- added D32: LED, LED_THT:LED_D3.0mm, F.Cu at (171.2, 32.7)
- added D4: LED, LED_THT:LED_D3.0mm, F.Cu at (99.2, 44.0)
- added D5: LED, LED_THT:LED_D3.0mm, F.Cu at (99.3, 35.7)
- added D6: LED, LED_THT:LED_D3.0mm, F.Cu at (77.6, 58.6)
- added D7: LED, LED_THT:LED_D3.0mm, F.Cu at (99.3, 30.1)
- added D8: LED, LED_THT:LED_D3.0mm, F.Cu at (99.3, 24.6)
- added D9: LED, LED_THT:LED_D3.0mm, F.Cu at (257.5, 46.5)
- added R1: 1k, Resistor_THT:R_Axial_DIN0207_L6.3mm_D2.5mm_P7.62mm_Horizontal, F.Cu at (45.0, 67.6)
- added R10: 1k, Resistor_THT:R_Axial_DIN0207_L6.3mm_D2.5mm_P7.62mm_Horizontal, F.Cu at (208.2, 54.9)
- added R11: 1k, Resistor_THT:R_Axial_DIN0207_L6.3mm_D2.5mm_P7.62mm_Horizontal, F.Cu at (197.5, 63.0)
- added R12: 1k, Resistor_THT:R_Axial_DIN0207_L6.3mm_D2.5mm_P7.62mm_Horizontal, F.Cu at (219.2, 45.7)
- added R13: 1k, Resistor_THT:R_Axial_DIN0207_L6.3mm_D2.5mm_P7.62mm_Horizontal, F.Cu at (197.5, 58.9)
- added R14: 1k, Resistor_THT:R_Axial_DIN0207_L6.3mm_D2.5mm_P7.62mm_Horizontal, F.Cu at (197.5, 54.9)
- added R15: 1k, Resistor_THT:R_Axial_DIN0207_L6.3mm_D2.5mm_P7.62mm_Horizontal, F.Cu at (208.2, 50.8)
- added R16: 1k, Resistor_THT:R_Axial_DIN0207_L6.3mm_D2.5mm_P7.62mm_Horizontal, F.Cu at (219.0, 50.8)
- added R17: 1k, Resistor_THT:R_Axial_DIN0207_L6.3mm_D2.5mm_P7.62mm_Horizontal, F.Cu at (197.5, 50.8)
- added R18: 1k, Resistor_THT:R_Axial_DIN0207_L6.3mm_D2.5mm_P7.62mm_Horizontal, F.Cu at (208.2, 58.9)
- added R19: 1k, Resistor_THT:R_Axial_DIN0207_L6.3mm_D2.5mm_P7.62mm_Horizontal, F.Cu at (219.0, 63.0)
- added R2: 1k, Resistor_THT:R_Axial_DIN0207_L6.3mm_D2.5mm_P7.62mm_Horizontal, F.Cu at (88.3, 47.3)
- added R20: 1k, Resistor_THT:R_Axial_DIN0207_L6.3mm_D2.5mm_P7.62mm_Horizontal, F.Cu at (219.0, 58.9)
- added R21: 1k, Resistor_THT:R_Axial_DIN0207_L6.3mm_D2.5mm_P7.62mm_Horizontal, F.Cu at (229.8, 49.8)
- added R22: 1k, Resistor_THT:R_Axial_DIN0207_L6.3mm_D2.5mm_P7.62mm_Horizontal, F.Cu at (240.7, 45.7)
- added R23: 1k, Resistor_THT:R_Axial_DIN0207_L6.3mm_D2.5mm_P7.62mm_Horizontal, F.Cu at (219.0, 54.9)
- added R24: 1k, Resistor_THT:R_Axial_DIN0207_L6.3mm_D2.5mm_P7.62mm_Horizontal, F.Cu at (208.2, 63.0)
- added R25: 1k, Resistor_THT:R_Axial_DIN0207_L6.3mm_D2.5mm_P7.62mm_Horizontal, F.Cu at (149.4, 50.8)
- added R26: 1k, Resistor_THT:R_Axial_DIN0207_L6.3mm_D2.5mm_P7.62mm_Horizontal, F.Cu at (171.1, 23.8)
- added R27: 1k, Resistor_THT:R_Axial_DIN0207_L6.3mm_D2.5mm_P7.62mm_Horizontal, F.Cu at (160.2, 43.2)
- added R28: 1k, Resistor_THT:R_Axial_DIN0207_L6.3mm_D2.5mm_P7.62mm_Horizontal, F.Cu at (171.1, 27.9)
- added R29: 1k, Resistor_THT:R_Axial_DIN0207_L6.3mm_D2.5mm_P7.62mm_Horizontal, F.Cu at (141.8, 61.0)
- added R3: 1k, Resistor_THT:R_Axial_DIN0207_L6.3mm_D2.5mm_P7.62mm_Horizontal, F.Cu at (77.5, 53.8)
- added R30: 1k, Resistor_THT:R_Axial_DIN0207_L6.3mm_D2.5mm_P7.62mm_Horizontal, F.Cu at (149.4, 54.9)
- added R31: 1k, Resistor_THT:R_Axial_DIN0207_L6.3mm_D2.5mm_P7.62mm_Horizontal, F.Cu at (131.0, 61.0)
- added R32: 1k, Resistor_THT:R_Axial_DIN0207_L6.3mm_D2.5mm_P7.62mm_Horizontal, F.Cu at (131.0, 65.0)
- added R4: 1k, Resistor_THT:R_Axial_DIN0207_L6.3mm_D2.5mm_P7.62mm_Horizontal, F.Cu at (66.7, 65.1)
- added R5: 1k, Resistor_THT:R_Axial_DIN0207_L6.3mm_D2.5mm_P7.62mm_Horizontal, F.Cu at (55.7, 67.6)
- added R6: 1k, Resistor_THT:R_Axial_DIN0207_L6.3mm_D2.5mm_P7.62mm_Horizontal, F.Cu at (77.5, 49.8)
- added R7: 1k, Resistor_THT:R_Axial_DIN0207_L6.3mm_D2.5mm_P7.62mm_Horizontal, F.Cu at (88.4, 43.2)
- added R8: 1k, Resistor_THT:R_Axial_DIN0207_L6.3mm_D2.5mm_P7.62mm_Horizontal, F.Cu at (77.5, 45.7)
- added R9: 1k, Resistor_THT:R_Axial_DIN0207_L6.3mm_D2.5mm_P7.62mm_Horizontal, F.Cu at (229.9, 45.7)
- added U13: 74LS157, Package_DIP:DIP-16_W7.62mm, F.Cu at (45.0, 23.9)
- added U14: 74LS157, Package_DIP:DIP-16_W7.62mm, F.Cu at (55.9, 23.9)
- added U15: 74LS157, Package_DIP:DIP-16_W7.62mm, F.Cu at (45.0, 45.8)
- added U16: 74LS157, Package_DIP:DIP-16_W7.62mm, F.Cu at (66.7, 23.9)
- added U17: 74LS157, Package_DIP:DIP-16_W7.62mm, F.Cu at (55.9, 45.8)
- added U18: 74LS157, Package_DIP:DIP-16_W7.62mm, F.Cu at (77.6, 23.9)
- added U19: 74LS157, Package_DIP:DIP-16_W7.62mm, F.Cu at (109.6, 97.3)
- added U20: 74LS157, Package_DIP:DIP-16_W7.62mm, F.Cu at (109.6, 75.4)
- added U21: 74LS157, Package_DIP:DIP-16_W7.62mm, F.Cu at (120.5, 75.4)
- added U22: 74LS157, Package_DIP:DIP-16_W7.62mm, F.Cu at (131.3, 75.4)
- added U23: 74LS157, Package_DIP:DIP-16_W7.62mm, F.Cu at (142.2, 75.4)
- added U24: 74LS157, Package_DIP:DIP-16_W7.62mm, F.Cu at (153.0, 75.4)
- added U25: 74LS157, Package_DIP:DIP-16_W7.62mm, F.Cu at (120.5, 97.3)
- added U26: 74LS157, Package_DIP:DIP-16_W7.62mm, F.Cu at (131.3, 97.3)
- added U27: 74LS157, Package_DIP:DIP-16_W7.62mm, F.Cu at (142.2, 97.3)
- added U28: 74LS157, Package_DIP:DIP-16_W7.62mm, F.Cu at (163.9, 75.4)
- added U29: 74LS377, Package_DIP:DIP-20_W7.62mm, F.Cu at (34.2, 23.9)
- added U30: 74LS377, Package_DIP:DIP-20_W7.62mm, F.Cu at (197.5, 23.9)
- added U31: 74LS377, Package_DIP:DIP-20_W7.62mm, F.Cu at (208.4, 23.9)
- added U32: 74LS157, Package_DIP:DIP-16_W7.62mm, F.Cu at (219.2, 23.9)
- added U33: 74LS157, Package_DIP:DIP-16_W7.62mm, F.Cu at (251.8, 23.9)
- added U34: 74LS257, Package_DIP:DIP-16_W7.62mm, F.Cu at (240.9, 23.9)
- added U35: 74LS257, Package_DIP:DIP-16_W7.62mm, F.Cu at (230.1, 23.9)
- added U36: 74LS245, Package_DIP:DIP-20_W7.62mm, F.Cu at (23.3, 23.9)
- added U37: 28C64, Package_DIP:DIP-28_W15.24mm, F.Cu at (131.0, 23.9)
- added U38: AS6C1008-55PCN, Package_DIP:DIP-32_W15.24mm, F.Cu at (112.6, 23.9)
- added U39: 74LS377, Package_DIP:DIP-20_W7.62mm, F.Cu at (149.4, 23.9)
- added U40: 74LS00, Package_DIP:DIP-14_W7.62mm, F.Cu at (160.3, 23.9)
- added U41: 74LS32, Package_DIP:DIP-14_W7.62mm, F.Cu at (66.7, 45.8)
- added U42: 74LS32, Package_DIP:DIP-14_W7.62mm, F.Cu at (23.3, 50.9)
- added U43: 74LS377, Package_DIP:DIP-20_W7.62mm, F.Cu at (60.1, 75.4)
- added U44: 74LS273, Package_DIP:DIP-20_W7.62mm, F.Cu at (71.0, 75.4)
- added U45: 74LS273, Package_DIP:DIP-20_W7.62mm, F.Cu at (81.8, 75.4)
- added U46: 74LS08, Package_DIP:DIP-14_W7.62mm, F.Cu at (60.1, 102.4)
- added U47: 74LS86, Package_DIP:DIP-14_W7.62mm, F.Cu at (71.0, 102.4)
- added U48: 28C64, Package_DIP:DIP-28_W15.24mm, F.Cu at (41.7, 75.4)
- added U49: 28C64, Package_DIP:DIP-28_W15.24mm, F.Cu at (23.3, 75.4)
- U10, U5: value 74LS08 -> 74LS32
- U11: value 74LS08 -> 74LS86
- U12, U6: value 74LS32 -> 74LS86
- U2, U7, U9: value 74LS86 -> 74LS08
- moved U12 113.1 mm to (88.4, 23.9)
- moved U11 107.5 mm to (34.2, 50.9)
- moved U5 80.4 mm to (34.2, 125.3)
- moved U1 79.9 mm to (23.3, 125.3)
- moved U6 72.5 mm to (153.0, 122.7)
- moved U2 72.2 mm to (66.7, 125.3)
- moved U3 72.2 mm to (55.9, 125.3)
- moved U4 64.8 mm to (45.0, 125.3)
- moved U7 56.2 mm to (142.2, 122.7)
- moved U8 47.3 mm to (131.3, 122.7)
- moved U10 13.7 mm to (120.5, 122.7)
- moved U9 13.7 mm to (109.6, 122.7)
Connections:
- net +5V renamed clk
- U1 pad 1: /Adder0/Cin -> /Alu/a0
- U1 pad 10: /b2 -> /Alu/Adder0/b2
- U1 pad 11: Net-(U1-Pad11) -> /Alu/xor3
- U1 pad 12: /Adder0/Cin -> /Alu/a3
- U1 pad 13: /b1 -> /Alu/Adder0/b3
- U1 pad 2: /b0 -> /Alu/Adder0/b0
- U1 pad 3: Net-(U1-Pad3) -> /Alu/xor0
- U1 pad 4: /Adder0/Cin -> /Alu/a1
- U1 pad 5: /b3 -> /Alu/Adder0/b1
- U1 pad 6: Net-(U1-Pad6) -> /Alu/xor1
- U1 pad 8: Net-(U1-Pad8) -> /Alu/xor2
- U1 pad 9: /Adder0/Cin -> /Alu/a2
- U10 pad 1: /a4 -> /Alu/and4
- U10 pad 11: Net-(U10-Pad11) -> (no net)
- U10 pad 12: /a7 -> /Alu/and7
- U10 pad 3: Net-(U10-Pad3) -> /Alu/Adder1/Bit1/Cin
- U10 pad 4: /a5 -> /Alu/and5
- U10 pad 6: Net-(U10-Pad6) -> /Alu/Adder1/Bit2/Cin
- U10 pad 8: Net-(U10-Pad8) -> /Alu/Adder1/Bit3/Cin
- U10 pad 9: /a6 -> /Alu/and6
- U11 pad 1: /Adder1/Cin -> /bus0
- U11 pad 10: Net-(U11-Pad10) -> ctrlAluSub
- U11 pad 11: Net-(U11-Pad11) -> /Alu/Adder0/b3
- U11 pad 12: /Adder1/Bit3/Cin -> /bus3
- U11 pad 13: Net-(U11-Pad13) -> ctrlAluSub
- U11 pad 2: Net-(U11-Pad2) -> ctrlAluSub
- U11 pad 3: Net-(U11-Pad3) -> /Alu/Adder0/b0
- U11 pad 4: /Adder1/Bit1/Cin -> /bus1
- U11 pad 5: Net-(U11-Pad5) -> ctrlAluSub
- U11 pad 6: Net-(U11-Pad6) -> /Alu/Adder0/b1
- U11 pad 8: Net-(U11-Pad8) -> /Alu/Adder0/b2
- U11 pad 9: /Adder1/Bit2/Cin -> /bus2
- U12 pad 1: Net-(U10-Pad3) -> /bus4
- U12 pad 10: Net-(U11-Pad8) -> ctrlAluSub
- U12 pad 11: /Adder1/Cout -> /Alu/Adder1/b3
- U12 pad 12: Net-(U10-Pad11) -> /bus7
- U12 pad 13: Net-(U11-Pad11) -> ctrlAluSub
- U12 pad 2: Net-(U11-Pad3) -> ctrlAluSub
- U12 pad 3: /Adder1/Bit1/Cin -> /Alu/Adder1/b0
- U12 pad 4: Net-(U10-Pad6) -> /bus5
- U12 pad 5: Net-(U11-Pad6) -> ctrlAluSub
- U12 pad 6: /Adder1/Bit2/Cin -> /Alu/Adder1/b1
- U12 pad 8: /Adder1/Bit3/Cin -> /Alu/Adder1/b2
- U12 pad 9: Net-(U10-Pad8) -> /bus6
- U2 pad 1: /a0 -> /Alu/a0
- U2 pad 10: Net-(U1-Pad8) -> /Alu/Adder0/b2
- U2 pad 11: Net-(U2-Pad11) -> /Alu/and3
- U2 pad 12: /a1 -> /Alu/a3
- U2 pad 13: Net-(U1-Pad11) -> /Alu/Adder0/b3
- U2 pad 2: Net-(U1-Pad3) -> /Alu/Adder0/b0
- U2 pad 3: Net-(U2-Pad3) -> /Alu/and0
- U2 pad 4: /a3 -> /Alu/a1
- U2 pad 5: Net-(U1-Pad6) -> /Alu/Adder0/b1
- U2 pad 6: Net-(U2-Pad6) -> /Alu/and1
- U2 pad 8: Net-(U2-Pad8) -> /Alu/and2
- U2 pad 9: /a2 -> /Alu/a2
- U3 pad 1: /Adder0/Cin -> ctrlAluSub
- U3 pad 10: Net-(U2-Pad8) -> /Alu/xor2
- U3 pad 11: /y1 -> /Alu/adderY3
- U3 pad 12: /Adder0/Bit1/Cin -> /Alu/Adder0/Bit3/Cin
- U3 pad 13: Net-(U2-Pad11) -> /Alu/xor3
- U3 pad 2: Net-(U2-Pad3) -> /Alu/xor0
- U3 pad 3: /y0 -> /Alu/adderY0
- U3 pad 4: /Adder0/Bit3/Cin -> /Alu/Adder0/Bit1/Cin
- U3 pad 5: Net-(U2-Pad6) -> /Alu/xor1
- U3 pad 6: /y3 -> /Alu/adderY1
- U3 pad 8: /y2 -> /Alu/adderY2
- U3 pad 9: /Adder0/Bit2/Cin -> /Alu/Adder0/Bit2/Cin
- U4 pad 1: /a0 -> ctrlAluSub
- U4 pad 10: Net-(U1-Pad8) -> /Alu/xor2
- U4 pad 12: /a1 -> /Alu/Adder0/Bit3/Cin
- U4 pad 13: Net-(U1-Pad11) -> /Alu/xor3
- U4 pad 2: Net-(U1-Pad3) -> /Alu/xor0
- U4 pad 4: /a3 -> /Alu/Adder0/Bit1/Cin
- U4 pad 5: Net-(U1-Pad6) -> /Alu/xor1
- U4 pad 9: /a2 -> /Alu/Adder0/Bit2/Cin
- U5 pad 1: /Adder0/Cin -> /Alu/and0
- U5 pad 10: Net-(U2-Pad8) -> Net-(U4-Pad8)
- U5 pad 11: Net-(U5-Pad11) -> /Alu/Adder1/Cin
- U5 pad 12: /Adder0/Bit1/Cin -> /Alu/and3
- U5 pad 13: Net-(U2-Pad11) -> Net-(U4-Pad11)
- U5 pad 2: Net-(U2-Pad3) -> Net-(U4-Pad3)
- U5 pad 3: Net-(U5-Pad3) -> /Alu/Adder0/Bit1/Cin
- U5 pad 4: /Adder0/Bit3/Cin -> /Alu/and1
- U5 pad 5: Net-(U2-Pad6) -> Net-(U4-Pad6)
- U5 pad 6: Net-(U5-Pad6) -> /Alu/Adder0/Bit2/Cin
- U5 pad 8: Net-(U5-Pad8) -> /Alu/Adder0/Bit3/Cin
- U5 pad 9: /Adder0/Bit2/Cin -> /Alu/and2
- U6 pad 1: Net-(U4-Pad3) -> /Alu/a4
- U6 pad 10: Net-(U5-Pad8) -> /Alu/Adder1/b2
- U6 pad 11: /Adder0/Bit2/Cin -> /Alu/xor7
- U6 pad 12: Net-(U4-Pad11) -> /Alu/a7
- U6 pad 13: Net-(U5-Pad11) -> /Alu/Adder1/b3
- U6 pad 2: Net-(U5-Pad3) -> /Alu/Adder1/b0
- U6 pad 3: /Adder0/Bit1/Cin -> /Alu/xor4
- U6 pad 4: Net-(U4-Pad6) -> /Alu/a5
- U6 pad 5: Net-(U5-Pad6) -> /Alu/Adder1/b1
- U6 pad 6: /Adder1/Cin -> /Alu/xor5
- U6 pad 8: /Adder0/Bit3/Cin -> /Alu/xor6
- U6 pad 9: Net-(U4-Pad8) -> /Alu/a6
- U7 pad 1: /Adder0/Cin -> /Alu/a4
- U7 pad 10: /b6 -> /Alu/Adder1/b2
- U7 pad 11: Net-(U10-Pad13) -> /Alu/and7
- U7 pad 12: /Adder0/Cin -> /Alu/a7
- U7 pad 13: /b7 -> /Alu/Adder1/b3
- U7 pad 2: /b4 -> /Alu/Adder1/b0
- U7 pad 3: Net-(U10-Pad2) -> /Alu/and4
- U7 pad 4: /Adder0/Cin -> /Alu/a5
- U7 pad 5: /b5 -> /Alu/Adder1/b1
- U7 pad 6: Net-(U10-Pad5) -> /Alu/and5
- U7 pad 8: Net-(U10-Pad10) -> /Alu/and6
- U7 pad 9: /Adder0/Cin -> /Alu/a6
- U8 pad 1: /a4 -> /Alu/Adder1/Cin
- U8 pad 10: Net-(U10-Pad10) -> /Alu/xor6
- U8 pad 11: Net-(U11-Pad13) -> /Alu/adderY7
- U8 pad 12: /a7 -> /Alu/Adder1/Bit3/Cin
- U8 pad 13: Net-(U10-Pad13) -> /Alu/xor7
- U8 pad 2: Net-(U10-Pad2) -> /Alu/xor4
- U8 pad 3: Net-(U11-Pad2) -> /Alu/adderY4
- U8 pad 4: /a5 -> /Alu/Adder1/Bit1/Cin
- U8 pad 5: Net-(U10-Pad5) -> /Alu/xor5
- U8 pad 6: Net-(U11-Pad5) -> /Alu/adderY5
- U8 pad 8: Net-(U11-Pad10) -> /Alu/adderY6
- U8 pad 9: /a6 -> /Alu/Adder1/Bit2/Cin
- U9 pad 1: /Adder1/Cin -> /Alu/Adder1/Cin
- U9 pad 10: Net-(U11-Pad10) -> /Alu/xor6
- U9 pad 11: /y7 -> Net-(U10-Pad13)
- U9 pad 12: /Adder1/Bit3/Cin -> /Alu/Adder1/Bit3/Cin
- U9 pad 13: Net-(U11-Pad13) -> /Alu/xor7
- U9 pad 2: Net-(U11-Pad2) -> /Alu/xor4
- U9 pad 3: /y4 -> Net-(U10-Pad2)
- U9 pad 4: /Adder1/Bit1/Cin -> /Alu/Adder1/Bit1/Cin
- U9 pad 5: Net-(U11-Pad5) -> /Alu/xor5
- U9 pad 6: /y5 -> Net-(U10-Pad5)
- U9 pad 8: /y6 -> Net-(U10-Pad10)
- U9 pad 9: /Adder1/Bit2/Cin -> /Alu/Adder1/Bit2/Cin

Commit message: pcbVersion: kinda done
Parts:
- added C1: 0.01u, Capacitor_THT:C_Radial_D6.3mm_H5.0mm_P2.50mm, F.Cu at (125.7, 146.3)
- added C2: 0.1u, Capacitor_THT:CP_Radial_D5.0mm_P2.50mm, F.Cu at (124.9, 153.5)
- added C3: 0.01u, Capacitor_THT:C_Radial_D6.3mm_H5.0mm_P2.50mm, F.Cu at (125.7, 138.5)
- added C4: 0.1u, Capacitor_THT:C_Radial_D6.3mm_H5.0mm_P2.50mm, F.Cu at (117.7, 150.4)
- added C5: 0.1u, Capacitor_THT:C_Radial_D6.3mm_H5.0mm_P2.50mm, F.Cu at (117.9, 142.5)
- added D33: instrNWE, LED_THT:LED_D3.0mm, F.Cu at (82.4, 56.8)
- added D34: instrSel, LED_THT:LED_D3.0mm, F.Cu at (93.2, 52.8)
- added D35: aluNOE, LED_THT:LED_D3.0mm, F.Cu at (82.4, 62.4)
- added D36: aluYNWE, LED_THT:LED_D3.0mm, F.Cu at (93.3, 46.0)
- added D37: reg0NWE, LED_THT:LED_D3.0mm, F.Cu at (99.2, 46.0)
- added D38: reg1NWE, LED_THT:LED_D3.0mm, F.Cu at (109.9, 33.9)
- added D39: regBusSel, LED_THT:LED_D3.0mm, F.Cu at (104.0, 33.9)
- added D40: regBusNOE, LED_THT:LED_D3.0mm, F.Cu at (77.8, 72.2)
- added D41: aluSel, LED_THT:LED_D3.0mm, F.Cu at (109.9, 39.4)
- added D42: marNWE, LED_THT:LED_D3.0mm, F.Cu at (88.3, 58.3)
- added D43: ramWE, LED_THT:LED_D3.0mm, F.Cu at (105.1, 45.0)
- added D44: ramOE, LED_THT:LED_D3.0mm, F.Cu at (99.1, 51.6)
- added D45: LED, LED_THT:LED_D3.0mm, F.Cu at (94.2, 58.3)
- added D46: ramSelect, LED_THT:LED_D3.0mm, F.Cu at (88.3, 63.9)
- added D47: LED, LED_THT:LED_D3.0mm, F.Cu at (83.7, 69.4)
- added D48: LED, LED_THT:LED_D3.0mm, F.Cu at (105.1, 50.5)
- added D49: LED, LED_THT:LED_D3.0mm, F.Cu at (111.0, 45.0)
- added D50: LED, LED_THT:LED_D3.0mm, F.Cu at (94.2, 63.9)
- added D51: instrNWE, LED_THT:LED_D3.0mm, F.Cu at (104.0, 39.4)
- added R33: 1k, Resistor_THT:R_Axial_DIN0207_L6.3mm_D2.5mm_P7.62mm_Horizontal, F.Cu at (56.1, 71.4)
- added R34: 1k, Resistor_THT:R_Axial_DIN0207_L6.3mm_D2.5mm_P7.62mm_Horizontal, F.Cu at (34.6, 66.2)
- added R35: 1k, Resistor_THT:R_Axial_DIN0207_L6.3mm_D2.5mm_P7.62mm_Horizontal, F.Cu at (93.2, 25.0)
- added R36: 1k, Resistor_THT:R_Axial_DIN0207_L6.3mm_D2.5mm_P7.62mm_Horizontal, F.Cu at (23.8, 70.3)
- added R37: 1k, Resistor_THT:R_Axial_DIN0207_L6.3mm_D2.5mm_P7.62mm_Horizontal, F.Cu at (23.8, 66.2)
- added R38: 1k, Resistor_THT:R_Axial_DIN0207_L6.3mm_D2.5mm_P7.62mm_Horizontal, F.Cu at (34.6, 62.2)
- added R39: 1k, Resistor_THT:R_Axial_DIN0207_L6.3mm_D2.5mm_P7.62mm_Horizontal, F.Cu at (45.4, 62.2)
- added R40: 1k, Resistor_THT:R_Axial_DIN0207_L6.3mm_D2.5mm_P7.62mm_Horizontal, F.Cu at (23.8, 62.2)
- added R41: 1k, Resistor_THT:R_Axial_DIN0207_L6.3mm_D2.5mm_P7.62mm_Horizontal, F.Cu at (45.4, 66.2)
- added R42: 1k, Resistor_THT:R_Axial_DIN0207_L6.3mm_D2.5mm_P7.62mm_Horizontal, F.Cu at (45.4, 70.3)
- added R43: 1k, Resistor_THT:R_Axial_DIN0207_L6.3mm_D2.5mm_P7.62mm_Horizontal, F.Cu at (103.9, 25.0)
- added R44: 1k, Resistor_THT:R_Axial_DIN0207_L6.3mm_D2.5mm_P7.62mm_Horizontal, F.Cu at (93.2, 29.1)
- added R45: 1k, Resistor_THT:R_Axial_DIN0207_L6.3mm_D2.5mm_P7.62mm_Horizontal, F.Cu at (93.2, 33.1)
- added R46: 1k, Resistor_THT:R_Axial_DIN0207_L6.3mm_D2.5mm_P7.62mm_Horizontal, F.Cu at (93.2, 41.2)
- added R47: 1k, Resistor_THT:R_Axial_DIN0207_L6.3mm_D2.5mm_P7.62mm_Horizontal, F.Cu at (103.9, 29.1)
- added R48: 1k, Resistor_THT:R_Axial_DIN0207_L6.3mm_D2.5mm_P7.62mm_Horizontal, F.Cu at (66.9, 71.4)
- added R49: 1k, Resistor_THT:R_Axial_DIN0207_L6.3mm_D2.5mm_P7.62mm_Horizontal, F.Cu at (93.2, 37.2)
- added R50: 1k, Resistor_THT:R_Axial_DIN0207_L6.3mm_D2.5mm_P7.62mm_Horizontal, F.Cu at (82.3, 52.0)
- added R51: 10M, Resistor_THT:R_Axial_DIN0207_L6.3mm_D2.5mm_P7.62mm_Horizontal, F.Cu at (95.2, 155.0)
- added R52: 1k, Resistor_THT:R_Axial_DIN0207_L6.3mm_D2.5mm_P7.62mm_Horizontal, F.Cu at (121.5, 132.5)
- added R53: 1k, Resistor_THT:R_Axial_DIN0207_L6.3mm_D2.5mm_P7.62mm_Horizontal, F.Cu at (110.7, 136.6)
- added R54: 1k, Resistor_THT:R_Axial_DIN0207_L6.3mm_D2.5mm_P7.62mm_Horizontal, F.Cu at (106.0, 144.3)
- added R55: 10M, Resistor_THT:R_Axial_DIN0207_L6.3mm_D2.5mm_P7.62mm_Horizontal, F.Cu at (95.2, 150.9)
- added R56: 1M, Resistor_THT:R_Axial_DIN0207_L6.3mm_D2.5mm_P7.62mm_Horizontal, F.Cu at (110.7, 132.5)
- added R57: 1k, Resistor_THT:R_Axial_DIN0207_L6.3mm_D2.5mm_P7.62mm_Horizontal, F.Cu at (95.2, 146.9)
- added R58: 1k, Resistor_THT:R_Axial_DIN0207_L6.3mm_D2.5mm_P7.62mm_Horizontal, F.Cu at (34.6, 70.3)
- added RV1: 1M, Potentiometer_THT:Potentiometer_Bourns_PTV09A-1_Single_Vertical, F.Cu at (84.5, 140.2)
- added SW1: SW_Push, Button_Switch_THT:SW_PUSH_6mm, F.Cu at (106.5, 148.3)
- added U50: NA555P, Package_DIP:DIP-8_W7.62mm, F.Cu at (84.4, 146.9)
- added U51: NA555P, Package_DIP:DIP-8_W7.62mm, F.Cu at (99.9, 132.6)
- added U52: 74LS86, Package_DIP:DIP-14_W7.62mm, F.Cu at (216.5, 142.3)
- added U53: 74LS08, Package_DIP:DIP-14_W7.62mm, F.Cu at (238.2, 120.4)
- added U54: 74LS86, Package_DIP:DIP-14_W7.62mm, F.Cu at (249.1, 120.4)
- added U55: 74LS08, Package_DIP:DIP-14_W7.62mm, F.Cu at (227.4, 142.3)
- added U56: 74LS273, Package_DIP:DIP-20_W7.62mm, F.Cu at (205.7, 120.4)
- added U57: 74LS157, Package_DIP:DIP-16_W7.62mm, F.Cu at (227.4, 120.4)
- added U58: 74LS157, Package_DIP:DIP-16_W7.62mm, F.Cu at (216.5, 120.4)
- added U59: 74LS32, Package_DIP:DIP-14_W7.62mm, F.Cu at (238.2, 139.8)
- added U60: 74LS245, Package_DIP:DIP-20_W7.62mm, F.Cu at (194.8, 120.4)
- moved U9 144.9 mm to (216.7, 25.1)
- moved U6 137.1 mm to (249.3, 25.1)
- moved U7 137.1 mm to (238.4, 25.1)
- moved U8 137.1 mm to (227.6, 25.1)
- moved U10 129.7 mm to (205.9, 25.1)
- moved D23 85.4 mm to (227.2, 104.8)
- moved U18 85.3 mm to (45.6, 102.9)
- moved R8 81.8 mm to (56.3, 124.7)
- moved U12 81.8 mm to (67.3, 102.9)
- moved D14 81.2 mm to (244.9, 102.3)
- moved D17 80.3 mm to (233.1, 110.4)
- moved D15 79.8 mm to (239.0, 106.3)
- moved R3 77.8 mm to (45.5, 124.7)
- moved U41 75.6 mm to (23.9, 108.0)
- moved R9 72.5 mm to (194.8, 109.2)
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Connections:
- net ctrlMarNE renamed ctrlMarNWE
- U49 pad 13: (no net) -> ctrlPCLoad
- U49 pad 17: (no net) -> ctrlPCNOE
