File: schematic/CPU/Ram.sch (KiCad schematic (older format))
At the start: 21 parts, among them U37 28C64, U38 AS6C1008-55PCN, U40 74LS00, U46 74LS08, U47 74LS374

Commit message: schematic finished
Parts:
- added R? (x10): 1k, Resistor_THT:R_Axial_DIN0207_L6.3mm_D2.5mm_P7.62mm_Horizontal, symbol Device:R
Connections:
- net +5V: now also R?.2, R?.2, R?.2, R?.2, R?.2, R?.2, R?.2, R?.2, R?.2, R?.2
- net ramNOE: now also R?.1
- net ramNWE: now also R?.1
- net at R30.2, U37.8 (A2), U38.10 (A2)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: now also R?.1
- net at R31.2, U37.9 (A1), U38.11 (A1)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: now also R?.1
- net at R32.2, U37.10 (A0), U38.12 (A0)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: now also R?.1
- net at R25.2, U37.3 (A7), U38.5 (A7)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: now also R?.1
- net at R26.2, U37.4 (A6), U38.6 (A6)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: now also R?.1
- net at R27.2, U37.5 (A5), U38.7 (A5)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: now also R?.1
- net at R28.2, U37.6 (A4), U38.8 (A4)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: now also R?.1
- net at R29.2, U37.7 (A3), U38.9 (A3)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: now also R?.1
Other:
- note added: "PullUp for 5V/3V3 compatibility\nDQ is connected to bus which is pulled up externaly"
- note added: "noe is not pulled up in hw for some reason but ctrlRamOE is..."

Commit message: pre upgrade to vivado 2021
Parts:
- added U30: 28C256, symbol Memory_EEPROM:28C256
- added U31: AS6C4008-55PCN, Package_DIP:DIP-32_W15.24mm, symbol Memory_RAM:AS6C4008-55PCN
- gave numbers to parts that had none: 10
Changed lines of the file:
@@
 $Descr A4 11693 8268
 encoding utf-8
-Sheet 15 19
+Sheet 14 20
 Title ""
 Date ""
@@
 AR Path="/601B5CAE/60F648C2" Ref="R?"  Part="1"
 AR Path="/600C5001/60F648C2" Ref="R?"  Part="1"
-AR Path="/60ECA4CB/60F648C2" Ref="R?"  Part="1"
-F 0 "R?" V 6343 5100 50  0000 C CNN
+AR Path="/60ECA4CB/60F648C2" Ref="R41"  Part="1"
+F 0 "R41" V 6343 5100 50  0000 C CNN
 F 1 "1k" V 6434 5100 50  0000 C CNN
 F 2 "Resistor_THT:R_Axial_DIN0207_L6.3mm_D2.5mm_P7.62mm_Horizontal" V 6480 5100 50  0001 C CNN
@@
 AR Path="/601B5CAE/60F64ED1" Ref="R?"  Part="1"
 AR Path="/600C5001/60F64ED1" Ref="R?"  Part="1"
-AR Path="/60ECA4CB/60F64ED1" Ref="R?"  Part="1"
-F 0 "R?" V 6493 5100 50  0000 C CNN
+AR Path="/60ECA4CB/60F64ED1" Ref="R42"  Part="1"
+F 0 "R42" V 6493 5100 50  0000 C CNN
 F 1 "1k" V 6584 5100 50  0000 C CNN
 F 2 "Resistor_THT:R_Axial_DIN0207_L6.3mm_D2.5mm_P7.62mm_Horizontal" V 6630 5100 50  0001 C CNN
@@
 	6550 5250 6550 5300
 $Comp
-L power:+5V #PWR?
+L power:+5V #PWR0178
 U 1 1 60F72F78
 P 6700 4950
-F 0 "#PWR?" H 6700 4800 50  0001 C CNN
+F 0 "#PWR0178" H 6700 4800 50  0001 C CNN
 F 1 "+5V" H 6715 5123 50  0000 C CNN
 F 2 "" H 6700 4950 50  0001 C CNN
@@
 $EndComp
 $Comp
-L power:+5V #PWR?
+L power:+5V #PWR0177
 U 1 1 60F7383B
 P 6550 4950
-F 0 "#PWR?" H 6550 4800 50  0001 C CNN
+F 0 "#PWR0177" H 6550 4800 50  0001 C CNN
 F 1 "+5V" H 6565 5123 50  0000 C CNN
 F 2 "" H 6550 4950 50  0001 C CNN
@@
 AR Path="/601B5CAE/60F7FEC7" Ref="R?"  Part="1"
 AR Path="/600C5001/60F7FEC7" Ref="R?"  Part="1"
-AR Path="/60ECA4CB/60F7FEC7" Ref="R?"  Part="1"
-F 0 "R?" V 2243 2100 50  0000 C CNN
+AR Path="/60ECA4CB/60F7FEC7" Ref="R34"  Part="1"
+F 0 "R34" V 2243 2100 50  0000 C CNN
 F 1 "1k" V 2334 2100 50  0000 C CNN
 F 2 "Resistor_THT:R_Axial_DIN0207_L6.3mm_D2.5mm_P7.62mm_Horizontal" V 2380 2100 50  0001 C CNN
@@
 AR Path="/601B5CAE/60F7FECD" Ref="R?"  Part="1"
 AR Path="/600C5001/60F7FECD" Ref="R?"  Part="1"
-AR Path="/60ECA4CB/60F7FECD" Ref="R?"  Part="1"
-F 0 "R?" V 2593 2100 50  0000 C CNN
+AR Path="/60ECA4CB/60F7FECD" Ref="R35"  Part="1"
+F 0 "R35" V 2593 2100 50  0000 C CNN
 F 1 "1k" V 2684 2100 50  0000 C CNN
 F 2 "Resistor_THT:R_Axial_DIN0207_L6.3mm_D2.5mm_P7.62mm_Horizontal" V 2730 2100 50  0001 C CNN
@@
 AR Path="/601B5CAE/60F7FED3" Ref="R?"  Part="1"
 AR Path="/600C5001/60F7FED3" Ref="R?"  Part="1"
-AR Path="/60ECA4CB/60F7FED3" Ref="R?"  Part="1"
-F 0 "R?" V 2943 2100 50  0000 C CNN
+AR Path="/60ECA4CB/60F7FED3" Ref="R36"  Part="1"
+F 0 "R36" V 2943 2100 50  0000 C CNN
 F 1 "1k" V 3034 2100 50  0000 C CNN
 F 2 "Resistor_THT:R_Axial_DIN0207_L6.3mm_D2.5mm_P7.62mm_Horizontal" V 3080 2100 50  0001 C CNN
@@
 AR Path="/601B5CAE/60F7FED9" Ref="R?"  Part="1"
 AR Path="/600C5001/60F7FED9" Ref="R?"  Part="1"
-AR Path="/60ECA4CB/60F7FED9" Ref="R?"  Part="1"
-F 0 "R?" V 3293 2100 50  0000 C CNN
+AR Path="/60ECA4CB/60F7FED9" Ref="R37"  Part="1"
+F 0 "R37" V 3293 2100 50  0000 C CNN
 F 1 "1k" V 3384 2100 50  0000 C CNN
 F 2 "Resistor_THT:R_Axial_DIN0207_L6.3mm_D2.5mm_P7.62mm_Horizontal" V 3430 2100 50  0001 C CNN
@@
 AR Path="/601B5CAE/60F7FEDF" Ref="R?"  Part="1"
 AR Path="/600C5001/60F7FEDF" Ref="R?"  Part="1"
-AR Path="/60ECA4CB/60F7FEDF" Ref="R?"  Part="1"
-F 0 "R?" V 3643 2100 50  0000 C CNN
+AR Path="/60ECA4CB/60F7FEDF" Ref="R38"  Part="1"
+F 0 "R38" V 3643 2100 50  0000 C CNN
 F 1 "1k" V 3734 2100 50  0000 C CNN
 F 2 "Resistor_THT:R_Axial_DIN0207_L6.3mm_D2.5mm_P7.62mm_Horizontal" V 3780 2100 50  0001 C CNN
@@
 AR Path="/601B5CAE/60F7FEE5" Ref="R?"  Part="1"
 AR Path="/600C5001/60F7FEE5" Ref="R?"  Part="1"
-AR Path="/60ECA4CB/60F7FEE5" Ref="R?"  Part="1"
-F 0 "R?" V 3993 2100 50  0000 C CNN
+AR Path="/60ECA4CB/60F7FEE5" Ref="R39"  Part="1"
+F 0 "R39" V 3993 2100 50  0000 C CNN
 F 1 "1k" V 4084 2100 50  0000 C CNN
 F 2 "Resistor_THT:R_Axial_DIN0207_L6.3mm_D2.5mm_P7.62mm_Horizontal" V 4130 2100 50  0001 C CNN
@@
 AR Path="/601B5CAE/60F7FEEB" Ref="R?"  Part="1"
 AR Path="/600C5001/60F7FEEB" Ref="R?"  Part="1"
-AR Path="/60ECA4CB/60F7FEEB" Ref="R?"  Part="1"
-F 0 "R?" V 4343 2100 50  0000 C CNN
+AR Path="/60ECA4CB/60F7FEEB" Ref="R40"  Part="1"
+F 0 "R40" V 4343 2100 50  0000 C CNN
 F 1 "1k" V 4434 2100 50  0000 C CNN
 F 2 "Resistor_THT:R_Axial_DIN0207_L6.3mm_D2.5mm_P7.62mm_Horizontal" V 4480 2100 50  0001 C CNN
@@
 AR Path="/601B5CAE/60F7FEF1" Ref="R?"  Part="1"
 AR Path="/600C5001/60F7FEF1" Ref="R?"  Part="1"
-AR Path="/60ECA4CB/60F7FEF1" Ref="R?"  Part="1"
-F 0 "R?" V 1893 2100 50  0000 C CNN
+AR Path="/60ECA4CB/60F7FEF1" Ref="R33"  Part="1"
+F 0 "R33" V 1893 2100 50  0000 C CNN
 F 1 "1k" V 1984 2100 50  0000 C CNN
 F 2 "Resistor_THT:R_Axial_DIN0207_L6.3mm_D2.5mm_P7.62mm_Horizontal" V 2030 2100 50  0001 C CNN
@@
 	4550 2250 4550 2350
 $Comp
-L power:+5V #PWR?
+L power:+5V #PWR0148
 U 1 1 60FC7158
 P 2100 1950
-F 0 "#PWR?" H 2100 1800 50  0001 C CNN
+F 0 "#PWR0148" H 2100 1800 50  0001 C CNN
 F 1 "+5V" H 2115 2123 50  0000 C CNN
 F 2 "" H 2100 1950 50  0001 C CNN
@@
 $EndComp
 $Comp
-L power:+5V #PWR?
+L power:+5V #PWR0154
 U 1 1 60FC78F6
 P 2450 1950
-F 0 "#PWR?" H 2450 1800 50  0001 C CNN
+F 0 "#PWR0154" H 2450 1800 50  0001 C CNN
 F 1 "+5V" H 2465 2123 50  0000 C CNN
 F 2 "" H 2450 1950 50  0001 C CNN
@@
 $EndComp
 $Comp
-L power:+5V #PWR?
+L power:+5V #PWR0160
 U 1 1 60FC7D71
 P 2800 1950
-F 0 "#PWR?" H 2800 1800 50  0001 C CNN
+F 0 "#PWR0160" H 2800 1800 50  0001 C CNN
 F 1 "+5V" H 2815 2123 50  0000 C CNN
 F 2 "" H 2800 1950 50  0001 C CNN
@@
 $EndComp
 $Comp
-L power:+5V #PWR?
+L power:+5V #PWR0161
 U 1 1 60FC8120
 P 3150 1950
-F 0 "#PWR?" H 3150 1800 50  0001 C CNN
+F 0 "#PWR0161" H 3150 1800 50  0001 C CNN
 F 1 "+5V" H 3165 2123 50  0000 C CNN
 F 2 "" H 3150 1950 50  0001 C CNN
@@
 $EndComp
 $Comp
-L power:+5V #PWR?
+L power:+5V #PWR0162
 U 1 1 60FC9B78
 P 3500 1950
-F 0 "#PWR?" H 3500 1800 50  0001 C CNN
+F 0 "#PWR0162" H 3500 1800 50  0001 C CNN
 F 1 "+5V" H 3515 2123 50  0000 C CNN
 F 2 "" H 3500 1950 50  0001 C CNN
@@
 $EndComp
 $Comp
-L power:+5V #PWR?
+L power:+5V #PWR0163
 U 1 1 60FC9B7E
 P 3850 1950
-F 0 "#PWR?" H 3850 1800 50  0001 C CNN
+F 0 "#PWR0163" H 3850 1800 50  0001 C CNN
 F 1 "+5V" H 3865 2123 50  0000 C CNN
 F 2 "" H 3850 1950 50  0001 C CNN
@@
 $EndComp
 $Comp
-L power:+5V #PWR?
+L power:+5V #PWR0175
 U 1 1 60FC9B84
 P 4200 1950
-F 0 "#PWR?" H 4200 1800 50  0001 C CNN
+F 0 "#PWR0175" H 4200 1800 50  0001 C CNN
 F 1 "+5V" H 4215 2123 50  0000 C CNN
 F 2 "" H 4200 1950 50  0001 C CNN
@@
 $EndComp
 $Comp
-L power:+5V #PWR?
+L power:+5V #PWR0176
 U 1 1 60FC9B8A
 P 4550 1950
-F 0 "#PWR?" H 4550 1800 50  0001 C CNN
+F 0 "#PWR0176" H 4550 1800 50  0001 C CNN
 F 1 "+5V" H 4565 2123 50  0000 C CNN
 F 2 "" H 4550 1950 50  0001 C CNN
@@
 	1    0    0    -1
 $EndComp
+$Comp
+L Memory_EEPROM:28C256 U30
+U 1 1 6148CEAB
+P 10000 2100
+F 0 "U30" H 10000 3381 50  0000 C CNN
+F 1 "28C256" H 10000 3290 50  0000 C CNN
+F 2 "" H 10000 2100 50  0001 C CNN
+F 3 "http://ww1.microchip.com/downloads/en/DeviceDoc/doc0006.pdf" H 10000 2100 50  0001 C CNN
+	1    10000 2100
+	1    0    0    -1
+$EndComp
+$Comp
+L Memory_RAM:AS6C4008-55PCN U31
+U 1 1 61491453
+P 10150 4800
+F 0 "U31" H 10150 6081 50  0000 C CNN
+F 1 "AS6C4008-55PCN" H 10150 5990 50  0000 C CNN
+F 2 "Package_DIP:DIP-32_W15.24mm" H 10150 4900 50  0001 C CNN
+F 3 "https://www.alliancememory.com/wp-content/uploads/pdf/AS6C4008.pdf" H 10150 4900 50  0001 C CNN
+	1    10150 4800
+	1    0    0    -1
+$EndComp
