File: schematic/CPU/1BitFullAdder.sch (KiCad schematic (older format))
At the start: 5 parts, among them U1 74LS86, U2 74LS08, U3 74LS86, U4 74LS08, U5 74LS32

Commit message: schematic with henry
Parts:
- renumbered U1 to U28, U2 to U29, U3 to U30, U4 to U31, U5 to U32
Changed lines of the file:
@@
 $Descr A4 11693 8268
 encoding utf-8
-Sheet 13 17
+Sheet 13 18
 Title ""
 Date ""
@@
 $EndDescr
 $Comp
-L 74xx:74LS08 U2
+L 74xx:74LS08 U29
 U 1 1 60149FB6
 P 4000 2300
-AR Path="/600C5001/60248238/6016C9C5/60149FB6" Ref="U2"  Part="4"
-AR Path="/600C5001/60248238/6016C700/60149FB6" Ref="U2"  Part="3"
-AR Path="/600C5001/60248238/6016C4DC/60149FB6" Ref="U2"  Part="2"
-AR Path="/600C5001/60248238/6014201D/60149FB6" Ref="U2"  Part="1"
-AR Path="/600C5001/60260EB9/6016C9C5/60149FB6" Ref="U7"  Part="4"
-AR Path="/600C5001/60260EB9/6016C700/60149FB6" Ref="U7"  Part="3"
-AR Path="/600C5001/60260EB9/6016C4DC/60149FB6" Ref="U7"  Part="2"
-AR Path="/600C5001/60260EB9/6014201D/60149FB6" Ref="U7"  Part="1"
-F 0 "U2" H 4000 2625 50  0000 C CNN
+AR Path="/600C5001/60248238/6016C9C5/60149FB6" Ref="U29"  Part="4"
+AR Path="/600C5001/60248238/6016C700/60149FB6" Ref="U29"  Part="3"
+AR Path="/600C5001/60248238/6016C4DC/60149FB6" Ref="U29"  Part="2"
+AR Path="/600C5001/60248238/6014201D/60149FB6" Ref="U29"  Part="1"
+AR Path="/600C5001/60260EB9/6016C9C5/60149FB6" Ref="U24"  Part="4"
+AR Path="/600C5001/60260EB9/6016C700/60149FB6" Ref="U24"  Part="3"
+AR Path="/600C5001/60260EB9/6016C4DC/60149FB6" Ref="U24"  Part="2"
+AR Path="/600C5001/60260EB9/6014201D/60149FB6" Ref="U24"  Part="1"
+F 0 "U29" H 4000 2625 50  0000 C CNN
 F 1 "74LS08" H 4000 2534 50  0000 C CNN
 F 2 "Package_DIP:DIP-14_W7.62mm" H 4000 2300 50  0001 C CNN
@@
 Connection ~ 3450 2950
 $Comp
-L 74xx:74LS08 U4
+L 74xx:74LS08 U31
 U 1 1 60149FCA
 P 5450 2750
-AR Path="/600C5001/60248238/6016C9C5/60149FCA" Ref="U4"  Part="4"
-AR Path="/600C5001/60248238/6016C700/60149FCA" Ref="U4"  Part="3"
-AR Path="/600C5001/60248238/6016C4DC/60149FCA" Ref="U4"  Part="2"
-AR Path="/600C5001/60248238/6014201D/60149FCA" Ref="U4"  Part="1"
-AR Path="/600C5001/60260EB9/6016C9C5/60149FCA" Ref="U9"  Part="4"
-AR Path="/600C5001/60260EB9/6016C700/60149FCA" Ref="U9"  Part="3"
-AR Path="/600C5001/60260EB9/6016C4DC/60149FCA" Ref="U9"  Part="2"
-AR Path="/600C5001/60260EB9/6014201D/60149FCA" Ref="U9"  Part="1"
-F 0 "U4" H 5450 3075 50  0000 C CNN
+AR Path="/600C5001/60248238/6016C9C5/60149FCA" Ref="U31"  Part="4"
+AR Path="/600C5001/60248238/6016C700/60149FCA" Ref="U31"  Part="3"
+AR Path="/600C5001/60248238/6016C4DC/60149FCA" Ref="U31"  Part="2"
+AR Path="/600C5001/60248238/6014201D/60149FCA" Ref="U31"  Part="1"
+AR Path="/600C5001/60260EB9/6016C9C5/60149FCA" Ref="U26"  Part="4"
+AR Path="/600C5001/60260EB9/6016C700/60149FCA" Ref="U26"  Part="3"
+AR Path="/600C5001/60260EB9/6016C4DC/60149FCA" Ref="U26"  Part="2"
+AR Path="/600C5001/60260EB9/6014201D/60149FCA" Ref="U26"  Part="1"
+F 0 "U31" H 5450 3075 50  0000 C CNN
 F 1 "74LS08" H 5450 2984 50  0000 C CNN
 F 2 "Package_DIP:DIP-14_W7.62mm" H 5450 2750 50  0001 C CNN
@@
 $EndComp
 $Comp
-L 74xx:74LS86 U3
+L 74xx:74LS86 U30
 U 1 1 60149FD6
 P 5600 1800
-AR Path="/600C5001/60248238/6016C9C5/60149FD6" Ref="U3"  Part="4"
-AR Path="/600C5001/60248238/6016C700/60149FD6" Ref="U3"  Part="3"
-AR Path="/600C5001/60248238/6016C4DC/60149FD6" Ref="U3"  Part="2"
-AR Path="/600C5001/60248238/6014201D/60149FD6" Ref="U3"  Part="1"
-AR Path="/600C5001/60260EB9/6016C9C5/60149FD6" Ref="U8"  Part="4"
-AR Path="/600C5001/60260EB9/6016C700/60149FD6" Ref="U8"  Part="3"
-AR Path="/600C5001/60260EB9/6016C4DC/60149FD6" Ref="U8"  Part="2"
-AR Path="/600C5001/60260EB9/6014201D/60149FD6" Ref="U8"  Part="1"
-F 0 "U3" H 5600 2125 50  0000 C CNN
+AR Path="/600C5001/60248238/6016C9C5/60149FD6" Ref="U30"  Part="4"
+AR Path="/600C5001/60248238/6016C700/60149FD6" Ref="U30"  Part="3"
+AR Path="/600C5001/60248238/6016C4DC/60149FD6" Ref="U30"  Part="2"
+AR Path="/600C5001/60248238/6014201D/60149FD6" Ref="U30"  Part="1"
+AR Path="/600C5001/60260EB9/6016C9C5/60149FD6" Ref="U25"  Part="4"
+AR Path="/600C5001/60260EB9/6016C700/60149FD6" Ref="U25"  Part="3"
+AR Path="/600C5001/60260EB9/6016C4DC/60149FD6" Ref="U25"  Part="2"
+AR Path="/600C5001/60260EB9/6014201D/60149FD6" Ref="U25"  Part="1"
+F 0 "U30" H 5600 2125 50  0000 C CNN
 F 1 "74LS86" H 5600 2034 50  0000 C CNN
 F 2 "Package_DIP:DIP-14_W7.62mm" H 5600 1800 50  0001 C CNN
@@
 Cout
 $Comp
-L 74xx:74LS32 U5
+L 74xx:74LS32 U32
 U 1 1 60149FEF
 P 6300 2450
-AR Path="/600C5001/60248238/6016C9C5/60149FEF" Ref="U5"  Part="4"
-AR Path="/600C5001/60248238/6016C700/60149FEF" Ref="U5"  Part="3"
-AR Path="/600C5001/60248238/6016C4DC/60149FEF" Ref="U5"  Part="2"
-AR Path="/600C5001/60248238/6014201D/60149FEF" Ref="U5"  Part="1"
-AR Path="/600C5001/60260EB9/6016C9C5/60149FEF" Ref="U10"  Part="4"
-AR Path="/600C5001/60260EB9/6016C700/60149FEF" Ref="U10"  Part="3"
-AR Path="/600C5001/60260EB9/6016C4DC/60149FEF" Ref="U10"  Part="2"
-AR Path="/600C5001/60260EB9/6014201D/60149FEF" Ref="U10"  Part="1"
-F 0 "U5" H 6300 2775 50  0000 C CNN
+AR Path="/600C5001/60248238/6016C9C5/60149FEF" Ref="U32"  Part="4"
+AR Path="/600C5001/60248238/6016C700/60149FEF" Ref="U32"  Part="3"
+AR Path="/600C5001/60248238/6016C4DC/60149FEF" Ref="U32"  Part="2"
+AR Path="/600C5001/60248238/6014201D/60149FEF" Ref="U32"  Part="1"
+AR Path="/600C5001/60260EB9/6016C9C5/60149FEF" Ref="U27"  Part="4"
+AR Path="/600C5001/60260EB9/6016C700/60149FEF" Ref="U27"  Part="3"
+AR Path="/600C5001/60260EB9/6016C4DC/60149FEF" Ref="U27"  Part="2"
+AR Path="/600C5001/60260EB9/6014201D/60149FEF" Ref="U27"  Part="1"
+F 0 "U32" H 6300 2775 50  0000 C CNN
 F 1 "74LS32" H 6300 2684 50  0000 C CNN
 F 2 "Package_DIP:DIP-14_W7.62mm" H 6300 2450 50  0001 C CNN
@@
 $EndComp
 $Comp
-L 74xx:74LS86 U1
+L 74xx:74LS86 U28
 U 1 1 60149FD0
 P 4100 2850
-AR Path="/600C5001/60248238/6016C9C5/60149FD0" Ref="U1"  Part="4"
-AR Path="/600C5001/60248238/6016C700/60149FD0" Ref="U1"  Part="3"
-AR Path="/600C5001/60248238/6016C4DC/60149FD0" Ref="U1"  Part="2"
-AR Path="/600C5001/60248238/6014201D/60149FD0" Ref="U1"  Part="1"
-AR Path="/600C5001/60260EB9/6016C9C5/60149FD0" Ref="U6"  Part="4"
-AR Path="/600C5001/60260EB9/6016C700/60149FD0" Ref="U6"  Part="3"
-AR Path="/600C5001/60260EB9/6016C4DC/60149FD0" Ref="U6"  Part="2"
-AR Path="/600C5001/60260EB9/6014201D/60149FD0" Ref="U6"  Part="1"
-F 0 "U1" H 4100 3175 50  0000 C CNN
+AR Path="/600C5001/60248238/6016C9C5/60149FD0" Ref="U28"  Part="4"
+AR Path="/600C5001/60248238/6016C700/60149FD0" Ref="U28"  Part="3"
+AR Path="/600C5001/60248238/6016C4DC/60149FD0" Ref="U28"  Part="2"
+AR Path="/600C5001/60248238/6014201D/60149FD0" Ref="U28"  Part="1"
+AR Path="/600C5001/60260EB9/6016C9C5/60149FD0" Ref="U23"  Part="4"
+AR Path="/600C5001/60260EB9/6016C700/60149FD0" Ref="U23"  Part="3"
+AR Path="/600C5001/60260EB9/6016C4DC/60149FD0" Ref="U23"  Part="2"
+AR Path="/600C5001/60260EB9/6014201D/60149FD0" Ref="U23"  Part="1"
+F 0 "U28" H 4100 3175 50  0000 C CNN
 F 1 "74LS86" H 4100 3084 50  0000 C CNN
 F 2 "Package_DIP:DIP-14_W7.62mm" H 4100 2850 50  0001 C CNN
