File: schematic/CPU/4BitFullAdder.sch (KiCad schematic (older format))
At the start: 5 parts, among them U1 74LS86, U2 74LS08, U3 74LS86, U4 74LS08, U5 74LS32

Commit message: schematic with henry
Parts:
- renumbered U1 to U28, U2 to U29, U3 to U30, U4 to U31, U5 to U32
Changed lines of the file:
@@
 $Descr A4 11693 8268
 encoding utf-8
-Sheet 9 17
+Sheet 9 18
 Title "ALU"
 Date "2021-01-20"
@@
 AR Path="/60248238/601C37F5" Ref="#PWR?"  Part="1"
 AR Path="/60260EB9/601C37F5" Ref="#PWR?"  Part="1"
-AR Path="/600C5001/60248238/601C37F5" Ref="#PWR013"  Part="1"
-AR Path="/600C5001/60260EB9/601C37F5" Ref="#PWR023"  Part="1"
-F 0 "#PWR013" H 5650 850 50  0001 C CNN
+AR Path="/600C5001/60248238/601C37F5" Ref="#PWR099"  Part="1"
+AR Path="/600C5001/60260EB9/601C37F5" Ref="#PWR089"  Part="1"
+F 0 "#PWR099" H 5650 850 50  0001 C CNN
 F 1 "+5V" H 5665 1173 50  0000 C CNN
 F 2 "" H 5650 1000 50  0001 C CNN
@@
 AR Path="/60248238/601C25DD" Ref="#PWR?"  Part="1"
 AR Path="/60260EB9/601C25DD" Ref="#PWR?"  Part="1"
-AR Path="/600C5001/60248238/601C25DD" Ref="#PWR011"  Part="1"
-AR Path="/600C5001/60260EB9/601C25DD" Ref="#PWR021"  Part="1"
-F 0 "#PWR011" H 5000 850 50  0001 C CNN
+AR Path="/600C5001/60248238/601C25DD" Ref="#PWR097"  Part="1"
+AR Path="/600C5001/60260EB9/601C25DD" Ref="#PWR087"  Part="1"
+F 0 "#PWR097" H 5000 850 50  0001 C CNN
 F 1 "+5V" H 5015 1173 50  0000 C CNN
 F 2 "" H 5000 1000 50  0001 C CNN
@@
 AR Path="/60248238/60189268" Ref="U?"  Part="5"
 AR Path="/60260EB9/60189268" Ref="U?"  Part="5"
-AR Path="/600C5001/60248238/60189268" Ref="U4"  Part="5"
-AR Path="/600C5001/60260EB9/60189268" Ref="U9"  Part="5"
-F 0 "U4" H 5230 1596 50  0000 L CNN
+AR Path="/600C5001/60248238/60189268" Ref="U31"  Part="5"
+AR Path="/600C5001/60260EB9/60189268" Ref="U26"  Part="5"
+F 0 "U31" H 5230 1596 50  0000 L CNN
 F 1 "74LS08" H 5230 1505 50  0000 L CNN
 F 2 "Package_DIP:DIP-14_W7.62mm" H 5000 1550 50  0001 C CNN
@@
 AR Path="/60248238/601A9C21" Ref="#PWR?"  Part="1"
 AR Path="/60260EB9/601A9C21" Ref="#PWR?"  Part="1"
-AR Path="/600C5001/60248238/601A9C21" Ref="#PWR06"  Part="1"
-AR Path="/600C5001/60260EB9/601A9C21" Ref="#PWR016"  Part="1"
-F 0 "#PWR06" H 2900 1850 50  0001 C CNN
+AR Path="/600C5001/60248238/601A9C21" Ref="#PWR092"  Part="1"
+AR Path="/600C5001/60260EB9/601A9C21" Ref="#PWR082"  Part="1"
+F 0 "#PWR092" H 2900 1850 50  0001 C CNN
 F 1 "GND" H 2905 1927 50  0000 C CNN
 F 2 "" H 2900 2100 50  0001 C CNN
@@
 AR Path="/60248238/601A9101" Ref="#PWR?"  Part="1"
 AR Path="/60260EB9/601A9101" Ref="#PWR?"  Part="1"
-AR Path="/600C5001/60248238/601A9101" Ref="#PWR08"  Part="1"
-AR Path="/600C5001/60260EB9/601A9101" Ref="#PWR018"  Part="1"
-F 0 "#PWR08" H 3650 1850 50  0001 C CNN
+AR Path="/600C5001/60248238/601A9101" Ref="#PWR094"  Part="1"
+AR Path="/600C5001/60260EB9/601A9101" Ref="#PWR084"  Part="1"
+F 0 "#PWR094" H 3650 1850 50  0001 C CNN
 F 1 "GND" H 3655 1927 50  0000 C CNN
 F 2 "" H 3650 2100 50  0001 C CNN
@@
 AR Path="/60248238/601A8BDE" Ref="#PWR?"  Part="1"
 AR Path="/60260EB9/601A8BDE" Ref="#PWR?"  Part="1"
-AR Path="/600C5001/60248238/601A8BDE" Ref="#PWR010"  Part="1"
-AR Path="/600C5001/60260EB9/601A8BDE" Ref="#PWR020"  Part="1"
-F 0 "#PWR010" H 4300 1850 50  0001 C CNN
+AR Path="/600C5001/60248238/601A8BDE" Ref="#PWR096"  Part="1"
+AR Path="/600C5001/60260EB9/601A8BDE" Ref="#PWR086"  Part="1"
+F 0 "#PWR096" H 4300 1850 50  0001 C CNN
 F 1 "GND" H 4305 1927 50  0000 C CNN
 F 2 "" H 4300 2100 50  0001 C CNN
@@
 AR Path="/60248238/601A8769" Ref="#PWR?"  Part="1"
 AR Path="/60260EB9/601A8769" Ref="#PWR?"  Part="1"
-AR Path="/600C5001/60248238/601A8769" Ref="#PWR012"  Part="1"
-AR Path="/600C5001/60260EB9/601A8769" Ref="#PWR022"  Part="1"
-F 0 "#PWR012" H 5000 1850 50  0001 C CNN
+AR Path="/600C5001/60248238/601A8769" Ref="#PWR098"  Part="1"
+AR Path="/600C5001/60260EB9/601A8769" Ref="#PWR088"  Part="1"
+F 0 "#PWR098" H 5000 1850 50  0001 C CNN
 F 1 "GND" H 5005 1927 50  0000 C CNN
 F 2 "" H 5000 2100 50  0001 C CNN
@@
 AR Path="/60248238/601A81A4" Ref="#PWR?"  Part="1"
 AR Path="/60260EB9/601A81A4" Ref="#PWR?"  Part="1"
-AR Path="/600C5001/60248238/601A81A4" Ref="#PWR014"  Part="1"
-AR Path="/600C5001/60260EB9/601A81A4" Ref="#PWR024"  Part="1"
-F 0 "#PWR014" H 5650 1850 50  0001 C CNN
+AR Path="/600C5001/60248238/601A81A4" Ref="#PWR0100"  Part="1"
+AR Path="/600C5001/60260EB9/601A81A4" Ref="#PWR090"  Part="1"
+F 0 "#PWR0100" H 5650 1850 50  0001 C CNN
 F 1 "GND" H 5655 1927 50  0000 C CNN
 F 2 "" H 5650 2100 50  0001 C CNN
@@
 AR Path="/60248238/601A601F" Ref="#PWR?"  Part="1"
 AR Path="/60260EB9/601A601F" Ref="#PWR?"  Part="1"
-AR Path="/600C5001/60248238/601A601F" Ref="#PWR09"  Part="1"
-AR Path="/600C5001/60260EB9/601A601F" Ref="#PWR019"  Part="1"
-F 0 "#PWR09" H 4300 850 50  0001 C CNN
+AR Path="/600C5001/60248238/601A601F" Ref="#PWR095"  Part="1"
+AR Path="/600C5001/60260EB9/601A601F" Ref="#PWR085"  Part="1"
+F 0 "#PWR095" H 4300 850 50  0001 C CNN
 F 1 "+5V" H 4315 1173 50  0000 C CNN
 F 2 "" H 4300 1000 50  0001 C CNN
@@
 AR Path="/60248238/601A5A36" Ref="#PWR?"  Part="1"
 AR Path="/60260EB9/601A5A36" Ref="#PWR?"  Part="1"
-AR Path="/600C5001/60248238/601A5A36" Ref="#PWR07"  Part="1"
-AR Path="/600C5001/60260EB9/601A5A36" Ref="#PWR017"  Part="1"
-F 0 "#PWR07" H 3650 850 50  0001 C CNN
+AR Path="/600C5001/60248238/601A5A36" Ref="#PWR093"  Part="1"
+AR Path="/600C5001/60260EB9/601A5A36" Ref="#PWR083"  Part="1"
+F 0 "#PWR093" H 3650 850 50  0001 C CNN
 F 1 "+5V" H 3665 1173 50  0000 C CNN
 F 2 "" H 3650 1000 50  0001 C CNN
@@
 AR Path="/60248238/601A53ED" Ref="#PWR?"  Part="1"
 AR Path="/60260EB9/601A53ED" Ref="#PWR?"  Part="1"
-AR Path="/600C5001/60248238/601A53ED" Ref="#PWR05"  Part="1"
-AR Path="/600C5001/60260EB9/601A53ED" Ref="#PWR015"  Part="1"
-F 0 "#PWR05" H 2900 850 50  0001 C CNN
+AR Path="/600C5001/60248238/601A53ED" Ref="#PWR091"  Part="1"
+AR Path="/600C5001/60260EB9/601A53ED" Ref="#PWR081"  Part="1"
+F 0 "#PWR091" H 2900 850 50  0001 C CNN
 F 1 "+5V" H 2915 1173 50  0000 C CNN
 F 2 "" H 2900 1000 50  0001 C CNN
@@
 AR Path="/60248238/6018B67E" Ref="U?"  Part="5"
 AR Path="/60260EB9/6018B67E" Ref="U?"  Part="5"
-AR Path="/600C5001/60248238/6018B67E" Ref="U5"  Part="5"
-AR Path="/600C5001/60260EB9/6018B67E" Ref="U10"  Part="5"
-F 0 "U5" H 5880 1596 50  0000 L CNN
+AR Path="/600C5001/60248238/6018B67E" Ref="U32"  Part="5"
+AR Path="/600C5001/60260EB9/6018B67E" Ref="U27"  Part="5"
+F 0 "U32" H 5880 1596 50  0000 L CNN
 F 1 "74LS32" H 5880 1505 50  0000 L CNN
 F 2 "Package_DIP:DIP-14_W7.62mm" H 5650 1550 50  0001 C CNN
@@
 AR Path="/60248238/60186DED" Ref="U?"  Part="5"
 AR Path="/60260EB9/60186DED" Ref="U?"  Part="5"
-AR Path="/600C5001/60248238/60186DED" Ref="U2"  Part="5"
-AR Path="/600C5001/60260EB9/60186DED" Ref="U7"  Part="5"
-F 0 "U2" H 3880 1596 50  0000 L CNN
+AR Path="/600C5001/60248238/60186DED" Ref="U29"  Part="5"
+AR Path="/600C5001/60260EB9/60186DED" Ref="U24"  Part="5"
+F 0 "U29" H 3880 1596 50  0000 L CNN
 F 1 "74LS08" H 3880 1505 50  0000 L CNN
 F 2 "Package_DIP:DIP-14_W7.62mm" H 3650 1550 50  0001 C CNN
@@
 AR Path="/60248238/6018470D" Ref="U?"  Part="5"
 AR Path="/60260EB9/6018470D" Ref="U?"  Part="5"
-AR Path="/600C5001/60248238/6018470D" Ref="U3"  Part="5"
-AR Path="/600C5001/60260EB9/6018470D" Ref="U8"  Part="5"
-F 0 "U3" H 4530 1596 50  0000 L CNN
+AR Path="/600C5001/60248238/6018470D" Ref="U30"  Part="5"
+AR Path="/600C5001/60260EB9/6018470D" Ref="U25"  Part="5"
+F 0 "U30" H 4530 1596 50  0000 L CNN
 F 1 "74LS86" H 4530 1505 50  0000 L CNN
 F 2 "Package_DIP:DIP-14_W7.62mm" H 4300 1550 50  0001 C CNN
@@
 AR Path="/60248238/601820B8" Ref="U?"  Part="5"
 AR Path="/60260EB9/601820B8" Ref="U?"  Part="5"
-AR Path="/600C5001/60248238/601820B8" Ref="U1"  Part="5"
-AR Path="/600C5001/60260EB9/601820B8" Ref="U6"  Part="5"
-F 0 "U1" H 3130 1596 50  0000 L CNN
+AR Path="/600C5001/60248238/601820B8" Ref="U28"  Part="5"
+AR Path="/600C5001/60260EB9/601820B8" Ref="U23"  Part="5"
+F 0 "U28" H 3130 1596 50  0000 L CNN
 F 1 "74LS86" H 3130 1505 50  0000 L CNN
 F 2 "Package_DIP:DIP-14_W7.62mm" H 2900 1550 50  0001 C CNN
@@
 Wire Wire Line
 	4050 2750 4350 2750
+Text HLabel 4450 4850 2    50   Output ~ 0
+SignCout
+Wire Wire Line
+	4250 4850 4450 4850
+Connection ~ 4250 4850
 $EndSCHEMATC
