File: schematic/CPU/Alu.sch (KiCad schematic (older format))
At the start: 28 parts, among them U11 74LS86, U12 74LS86, U13 74LS157, U14 74LS157, U15 74LS157, U16 74LS157, U17 74LS157, U18 74LS157, U30 74LS374, U36 74LS245, U41 74LS32, U42 74LS32

Commit message: schematic finished
Connections:
- wire segments 300 -> 309
Other:
- note added: "board 00"
- note added: "board 01"
- note added: "board 10/11"
- note added: "board 11"
- note added: "board 12"
- moved on the sheet: U11A, U11B, U11C, U11D, U11E, U12E, U13, U15, U16, U18

Commit message: pre upgrade to vivado 2021
Parts:
- removed U30: 74LS374, Package_DIP:DIP-20_W7.62mm, symbol 74xx:74LS374
- removed U41, U42: 74LS32, Package_DIP:DIP-14_W7.62mm, symbol 74xx:74LS32
- added U29: 74AS825, symbol 74xx:74AS825
- added U41, U42: 74LS08, symbol 74xx:74LS08
Connections:
- net labels added: clk, ~ctrlAluYWE~, ~reset~
- net labels removed: y_cp
- wire segments 309 -> 296
- no-connect marks 2 -> 4
Other:
- note removed: "board 00"
- note removed: "board 01"
- note removed: "board 10/11"
- note removed: "board 11"
- note removed: "board 12"
- moved on the sheet: R1, R2, R3, R4, R5, R6, R7, R8, U11A, U11B, U11C, U11D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

Commit message: fibonacci works again with new memory design
Connections:
- net labels added: bus0, bus1, bus2, bus3, bus4, bus5, bus6, bus7
- net labels removed: aluNOE, aluOp0, aluOp1, b3, b4, b5, b6, b7, sub, y0, y1, y2, y3, y4, y5, y6, y7
- wire segments 296 -> 303
Other:
- moved on the sheet: U13, U17, U18, U36

Commit message: schematic with henry
Parts:
- removed D1, D2, D3, D4, D5, D6, D7, D8: LED, LED_THT:LED_D3.0mm, symbol Device:LED
- removed R1, R2, R3, R4, R5, R6, R7, R8: 1k, Resistor_THT:R_Axial_DIN0207_L6.3mm_D2.5mm_P7.62mm_Horizontal, symbol Device:R
- removed U13, U14, U15, U16, U17, U18: 74LS157, Package_DIP:DIP-16_W7.62mm, symbol 74xx:74LS157
- removed U41, U42: 74LS08, symbol 74xx:74LS08
- added D10, D11, D12, D13, D14, D15, D16, D9: LED_Small, symbol Device:LED_Small
- added RN3: 220, Resistor_THT:R_Array_SIP9, symbol Device:R_Network08
- added U11: 74ABT540, symbol 8bitCPU-rescue:74ABT540
- added U12: 74F521, symbol 8bitCPU-rescue:74F521
- added unit 2 of U2
- added unit 3 of U2
- added unit 4 of U2
- added unit 5 of U3
- added unit 1 of U4
- added U5, U6, U7, U8: 74LS153, symbol 74xx:74LS153
- U9: renamed from U29; symbol 74xx:74AS825 -> 8bitCPU-rescue:74AS825-74xx
- renumbered U36 to U10, U11 to U2, U12 to U2, U11 to U3, U12 to U3, U11 to U4, U12 to U4
Connections:
- net labels added: adder0, adder1, adder2, adder3, adder4, adder5, adder6, adder7, flagCarry, flagOverflow, shift0, shift1, shift2, shift3, shift4, shift5, shift6, shift7
- net labels removed: adderY0, adderY1, adderY2, adderY3, adderY4, adderY5, adderY6, adderY7
- wire segments 303 -> 253
- no-connect marks 4 -> 9
Other:
- moved on the sheet: U10, U2A, U2E, U3A, U3B, U3C, U3D, U4B, U4C, U4D, U4E

Commit message: updated verilog from schematic
Parts:
- added U97: 74AS825, symbol 8bitCPU-rescue:74AS825-74xx
Connections:
- net +5V: now also U97.10 (D7), U97.24 (Vcc), U97.7 (D4), U97.8 (D5), U97.9 (D6)
- net GND: now also U97.1 (~OE1~), U97.12 (GND), U97.2 (~OE2~), U97.23 (~OE3~)
- net clk: now also U97.13 (CLK)
- net flagCarry: now also U97.20 (Q2); no longer U4.2
- net flagNZero: now also U97.21 (Q1); no longer U12.19 (P=R)
- net flagNegative: now also U97.22 (Q0); no longer U10.9 (A7), U11.9 (A7), U12.18 (R7), U9.15 (Q7)
- net flagOverflow: now also U97.19 (Q3); no longer U4.3
- net ~ctrlAluYWE~: now also U97.14 (~CLKEN~)
- net ~reset~: now also U97.11 (~CLR~)
- net at U10.2 (A0), U11.2 (A0), U9.22 (Q0): no longer U12.3 (R0)
- net at U10.3 (A1), U11.3 (A1), U9.21 (Q1): no longer U12.5 (R1)
- net at U10.4 (A2), U11.4 (A2), U9.20 (Q2): no longer U12.7 (R2)
- net at U10.5 (A3), U11.5 (A3), U9.19 (Q3): no longer U12.9 (R3)
- net at U10.6 (A4), U11.6 (A4), U9.18 (Q4): no longer U12.12 (R4)
- net at U10.7 (A5), U11.7 (A5), U9.17 (Q5): no longer U12.14 (R5)
- net at U10.8 (A6), U11.8 (A6), U9.16 (Q6): no longer U12.16 (R6)
- net flagN: now reaches U8.9 (Zb), U9.10 (D7)
- net flagN: now also U12.18 (R7), U97.3 (D0)
- net at U5.7 (Za), U9.3 (D0): now also U12.3 (R0)
- net at U5.9 (Zb), U9.4 (D1): now also U12.5 (R1)
- net at U6.7 (Za), U9.5 (D2): now also U12.7 (R2)
- net at U6.9 (Zb), U9.6 (D3): now also U12.9 (R3)
- net at U7.7 (Za), U9.7 (D4): now also U12.12 (R4)
- net at U7.9 (Zb), U9.8 (D5): now also U12.14 (R5)
- net at U8.7 (Za), U9.9 (D6): now also U12.16 (R6)
- net Adder1/SignCout renamed flagC
- net flagC: now also U97.5 (D2)
- new net: U10.9 (A7), U11.9 (A7), U9.15 (Q7)
- new net Adder1/Cout: U4.2
- new net flagNZ: U12.19 (P=R), U97.4 (D1)
- new net flagO: U4.3, U97.6 (D3)
- no-connect marks 9 -> 13
Other:
- moved on the sheet: U12, U4A, U9

Commit message: updated some more verilog
Connections:
- net at U2.4: now also U12.19 (P=R), U2.5
- net flagZ: now reaches U2.6
- net flagZ: now also U97.4 (D1)
- removed net flagNZ: U12.19 (P=R), U97.4 (D1)
- net flagNZero renamed flagZero
- net flagO renamed flagV
- no-connect marks 13 -> 10
Other:
- moved on the sheet: U2B
Changed lines of the file:
@@
 	4200 5500 4200 5950
 Text GLabel 18400 12450 2    50   Output ~ 0
-flagNZero
+flagZero
 Wire Wire Line
 	15250 4850 15450 4850
@@
 L 74xx:74LS86 U2
 U 2 1 615DEB20
-P 3250 7850
-F 0 "U2" H 3250 8175 50  0000 C CNN
-F 1 "74LS86" H 3250 8084 50  0000 C CNN
-F 2 "Package_DIP:DIP-14_W7.62mm" H 3250 7850 50  0001 C CNN
-F 3 "74xx/74ls86.pdf" H 3250 7850 50  0001 C CNN
-	2    3250 7850
+P 15850 4850
+F 0 "U2" H 15850 5175 50  0000 C CNN
+F 1 "74LS86" H 15850 5084 50  0000 C CNN
+F 2 "Package_DIP:DIP-14_W7.62mm" H 15850 4850 50  0001 C CNN
+F 3 "74xx/74ls86.pdf" H 15850 4850 50  0001 C CNN
+	2    15850 4850
 	1    0    0    -1
 $EndComp
@@
 	1    0    0    -1
 $EndComp
-NoConn ~ 2950 7750
-NoConn ~ 2950 7950
-NoConn ~ 3550 7850
 NoConn ~ 3500 8400
 NoConn ~ 3500 9000
@@
 Wire Wire Line
 	13800 8600 14550 8600
-Text Label 15450 4850 0    50   ~ 0
-flagNZ
 Text Label 15050 7250 0    50   ~ 0
 flagN
@@
 	16900 12950 17050 12950
 Text Label 16950 12450 2    50   ~ 0
-flagNZ
+flagZ
 Text Label 16950 12550 2    50   ~ 0
 flagC
 Text Label 16950 12650 2    50   ~ 0
-flagO
+flagV
 Wire Wire Line
 	5950 7350 6650 7350
@@
 flagC
 Text Label 7450 7250 0    50   ~ 0
-flagO
+flagV
 Wire Wire Line
 	7250 7250 7450 7250
+Text Label 16250 4850 0    50   ~ 0
+flagZ
+Wire Wire Line
+	16250 4850 16150 4850
+Wire Wire Line
+	15450 4850 15450 4750
+Wire Wire Line
+	15450 4750 15550 4750
+Wire Wire Line
+	15450 4850 15450 4950
+Wire Wire Line
+	15450 4950 15550 4950
+Connection ~ 15450 4850
 $EndSCHEMATC

Commit message: renamed project
Parts:
- U11: symbol 8bitCPU-rescue:74ABT540 -> MEDiC-rescue:74ABT540
- U12: symbol 8bitCPU-rescue:74F521 -> MEDiC-rescue:74F521
- U9, U97: symbol 8bitCPU-rescue:74AS825-74xx -> MEDiC-rescue:74AS825-74xx
Changed lines of the file:
@@
 $EndComp
 $Comp
-L 8bitCPU-rescue:74AS825-74xx U?
+L MEDiC-rescue:74AS825-74xx U?
 U 1 1 614109DB
 P 15050 8400
@@
 	12200 2000 12200 7900
 $Comp
-L 8bitCPU-rescue:74F521 U12
+L MEDiC-rescue:74F521 U12
 U 1 1 6303CD49
 P 15350 5650
@@
 Connection ~ 16450 8000
 $Comp
-L 8bitCPU-rescue:74ABT540 U11
+L MEDiC-rescue:74ABT540 U11
 U 1 1 632647A0
 P 17900 10700
@@
 $EndComp
 $Comp
-L 8bitCPU-rescue:74AS825-74xx U?
+L MEDiC-rescue:74AS825-74xx U?
 U 1 1 615311D5
 P 17650 12850

Commit message: renamed project
Parts:
- U11: symbol MEDiC-rescue:74ABT540 -> EDiC-rescue:74ABT540
- U12: symbol MEDiC-rescue:74F521 -> EDiC-rescue:74F521
- U9, U97: symbol MEDiC-rescue:74AS825-74xx -> EDiC-rescue:74AS825-74xx
Changed lines of the file:
@@
 $EndComp
 $Comp
-L MEDiC-rescue:74AS825-74xx U?
+L EDiC-rescue:74AS825-74xx U?
 U 1 1 614109DB
 P 15050 8400
@@
 	12200 2000 12200 7900
 $Comp
-L MEDiC-rescue:74F521 U12
+L EDiC-rescue:74F521 U12
 U 1 1 6303CD49
 P 15350 5650
@@
 Connection ~ 16450 8000
 $Comp
-L MEDiC-rescue:74ABT540 U11
+L EDiC-rescue:74ABT540 U11
 U 1 1 632647A0
 P 17900 10700
@@
 $EndComp
 $Comp
-L MEDiC-rescue:74AS825-74xx U?
+L EDiC-rescue:74AS825-74xx U?
 U 1 1 615311D5
 P 17650 12850
