File: schematic/CPU/Alu.sch (KiCad schematic (older format))
At the start: 21 parts, among them U10 74LS245, U11 74ABT540, U12 74F521, U2 74LS86, U3 74LS86, U4 74LS86, U5 74LS153, U6 74LS153, U7 74LS153, U8 74LS153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

Commit message: schematic: alu/shifter carry fix
Parts:
- added U?: 74LS151, symbol 74xx:74LS151
Connections:
- net labels added: flagCShift
- wire segments 280 -> 290
- no-connect marks 10 -> 15
Changed lines of the file:
@@
 a0
 $Sheet
-S 5050 8100 800  1500
+S 5050 8100 800  1700
 U 60297135
 F0 "shifter" 50
@@
 F20 "y6" O R 5850 8750 50
 F21 "y7" O R 5850 8850 50
+F22 "oldCFlag" I L 5050 9650 50
+F23 "flagC" O R 5850 9050 50
 $EndSheet
 Wire Wire Line
@@
 	16950 12450 17150 12450
 Wire Wire Line
-	16950 12550 17150 12550
-Wire Wire Line
 	16950 12650 17150 12650
 NoConn ~ 18150 12750
@@
 Text Label 16950 12450 2    50   ~ 0
 flagZ
-Text Label 16950 12550 2    50   ~ 0
-flagC
 Text Label 16950 12650 2    50   ~ 0
 flagV
@@
 	15450 4950 15550 4950
 Connection ~ 15450 4850
+$Comp
+L power:GND #PWR?
+U 1 1 619E0241
+P 16000 14150
+AR Path="/608A8AE7/619E0241" Ref="#PWR?"  Part="1"
+AR Path="/600C5001/619E0241" Ref="#PWR?"  Part="1"
+F 0 "#PWR?" H 16000 13900 50  0001 C CNN
+F 1 "GND" H 16005 13977 50  0000 C CNN
+F 2 "" H 16000 14150 50  0001 C CNN
+F 3 "" H 16000 14150 50  0001 C CNN
+	1    16000 14150
+	1    0    0    -1
+$EndComp
+$Comp
+L power:+5V #PWR?
+U 1 1 619E0247
+P 16000 12250
+AR Path="/608A8AE7/619E0247" Ref="#PWR?"  Part="1"
+AR Path="/600C5001/619E0247" Ref="#PWR?"  Part="1"
+F 0 "#PWR?" H 16000 12100 50  0001 C CNN
+F 1 "+5V" H 16000 12500 50  0000 C CNN
+F 2 "" H 16000 12250 50  0001 C CNN
+F 3 "" H 16000 12250 50  0001 C CNN
+	1    16000 12250
+	1    0    0    -1
+$EndComp
+$Comp
+L 74xx:74LS151 U?
+U 1 1 619E024D
+P 16000 13150
+AR Path="/608A8AE7/619E024D" Ref="U?"  Part="1"
+AR Path="/600C5001/619E024D" Ref="U?"  Part="1"
+F 0 "U?" H 16000 14231 50  0000 C CNN
+F 1 "74LS151" H 16000 14140 50  0000 C CNN
+F 2 "" H 16000 13150 50  0001 C CNN
+F 3 "http://www.ti.com/lit/gpn/sn74LS151" H 16000 13150 50  0001 C CNN
+	1    16000 13150
+	1    0    0    -1
+$EndComp
+$Comp
+L power:GND #PWR?
+U 1 1 619E0253
+P 15500 13850
+AR Path="/608A8AE7/619E0253" Ref="#PWR?"  Part="1"
+AR Path="/600C5001/619E0253" Ref="#PWR?"  Part="1"
+F 0 "#PWR?" H 15500 13600 50  0001 C CNN
+F 1 "GND" H 15505 13677 50  0000 C CNN
+F 2 "" H 15500 13850 50  0001 C CNN
+F 3 "" H 15500 13850 50  0001 C CNN
+	1    15500 13850
+	1    0    0    -1
+$EndComp
+NoConn ~ 16500 12650
+Wire Wire Line
+	16500 12550 17150 12550
+Text GLabel 15500 13450 0    50   Input ~ 0
+ctrlAluOp0
+Text GLabel 15500 13550 0    50   Input ~ 0
+ctrlAluOp1
+Text Label 15300 12550 2    50   ~ 0
+flagC
+Wire Wire Line
+	15300 12550 15400 12550
+Wire Wire Line
+	15400 12550 15400 12650
+Connection ~ 15400 12550
+Wire Wire Line
+	15400 12550 15500 12550
+Wire Wire Line
+	15500 12650 15400 12650
+Wire Wire Line
+	15500 13850 15500 13650
+Connection ~ 15500 13850
+Wire Wire Line
+	15500 12750 15400 12750
+Wire Wire Line
+	15400 12750 15400 12650
+Connection ~ 15400 12650
+Wire Wire Line
+	15300 12850 15500 12850
+NoConn ~ 15500 12950
+NoConn ~ 15500 13050
+NoConn ~ 15500 13150
+NoConn ~ 15500 13250
+Text Label 15300 12850 2    50   ~ 0
+flagCShift
+Text Label 6000 9050 0    50   ~ 0
+flagCShift
+Wire Wire Line
+	5850 9050 6000 9050
+Text GLabel 4950 9650 0    50   Input ~ 0
+flagCarry
+Wire Wire Line
+	4950 9650 5050 9650
 $EndSCHEMATC

Commit message: fixed uart_rx and snake
Parts:
- gave numbers to parts that had none: 1
Changed lines of the file:
@@
 P 16000 14150
 AR Path="/608A8AE7/619E0241" Ref="#PWR?"  Part="1"
-AR Path="/600C5001/619E0241" Ref="#PWR?"  Part="1"
-F 0 "#PWR?" H 16000 13900 50  0001 C CNN
+AR Path="/600C5001/619E0241" Ref="#PWR0326"  Part="1"
+F 0 "#PWR0326" H 16000 13900 50  0001 C CNN
 F 1 "GND" H 16005 13977 50  0000 C CNN
 F 2 "" H 16000 14150 50  0001 C CNN
@@
 P 16000 12250
 AR Path="/608A8AE7/619E0247" Ref="#PWR?"  Part="1"
-AR Path="/600C5001/619E0247" Ref="#PWR?"  Part="1"
-F 0 "#PWR?" H 16000 12100 50  0001 C CNN
+AR Path="/600C5001/619E0247" Ref="#PWR0325"  Part="1"
+F 0 "#PWR0325" H 16000 12100 50  0001 C CNN
 F 1 "+5V" H 16000 12500 50  0000 C CNN
 F 2 "" H 16000 12250 50  0001 C CNN
@@
 P 16000 13150
 AR Path="/608A8AE7/619E024D" Ref="U?"  Part="1"
-AR Path="/600C5001/619E024D" Ref="U?"  Part="1"
-F 0 "U?" H 16000 14231 50  0000 C CNN
+AR Path="/600C5001/619E024D" Ref="U101"  Part="1"
+F 0 "U101" H 16000 14231 50  0000 C CNN
 F 1 "74LS151" H 16000 14140 50  0000 C CNN
 F 2 "" H 16000 13150 50  0001 C CNN
@@
 P 15500 13850
 AR Path="/608A8AE7/619E0253" Ref="#PWR?"  Part="1"
-AR Path="/600C5001/619E0253" Ref="#PWR?"  Part="1"
-F 0 "#PWR?" H 15500 13600 50  0001 C CNN
+AR Path="/600C5001/619E0253" Ref="#PWR0324"  Part="1"
+F 0 "#PWR0324" H 15500 13600 50  0001 C CNN
 F 1 "GND" H 15505 13677 50  0000 C CNN
 F 2 "" H 15500 13850 50  0001 C CNN
@@
 Wire Wire Line
 	4950 9650 5050 9650
+Wire Notes Line rgb(255, 0, 0)
+	6300 6550 6300 7650
+Wire Notes Line rgb(255, 0, 0)
+	6300 7650 8000 7650
+Wire Notes Line rgb(255, 0, 0)
+	8000 7650 8000 6550
+Wire Notes Line rgb(255, 0, 0)
+	8000 6550 6300 6550
+Wire Notes Line rgb(255, 0, 0)
+	6500 8900 5550 8900
+Wire Notes Line rgb(255, 0, 0)
+	5550 8900 5550 9200
+Wire Notes Line rgb(255, 0, 0)
+	5550 9200 6500 9200
+Wire Notes Line rgb(255, 0, 0)
+	6500 9200 6500 8900
+Wire Notes Line rgb(255, 0, 0)
+	4500 9550 5450 9550
+Wire Notes Line rgb(255, 0, 0)
+	5450 9550 5450 9750
+Wire Notes Line rgb(255, 0, 0)
+	5450 9750 4500 9750
+Wire Notes Line rgb(255, 0, 0)
+	4500 9750 4500 9550
+Wire Notes Line rgb(255, 0, 0)
+	15250 4300 15250 5150
+Wire Notes Line rgb(255, 0, 0)
+	15250 5150 16550 5150
+Wire Notes Line rgb(255, 0, 0)
+	16550 5150 16550 4300
+Wire Notes Line rgb(255, 0, 0)
+	16550 4300 15250 4300
+Wire Notes Line rgb(255, 0, 0)
+	14600 11750 19200 11750
+Wire Notes Line rgb(255, 0, 0)
+	19200 11750 19200 14450
+Wire Notes Line rgb(255, 0, 0)
+	19200 14450 14600 14450
+Wire Notes Line rgb(255, 0, 0)
+	14600 14450 14600 11750
 $EndSCHEMATC
