File: schematic/CPU/Clock.sch (KiCad schematic (older format))
At the start: 35 parts, among them Q1 BC337, Q2 BC337, Q3 BC337, Q4 BC337, SW1 clk_switch, SW2 SW_SPDT, SW3 continue_switch, U50 NA555P, U51 NA555P, U69 74LS157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

Commit message: schematic with henry
Parts:
- removed C1, C3, C8: 10nF, Capacitor_THT:C_Radial_D6.3mm_H5.0mm_P2.50mm, symbol Device:C_Small
- removed C2, C7: 1uF, Capacitor_THT:CP_Radial_D5.0mm_P2.50mm, symbol Device:CP1_Small
- removed C9: 10uF, Capacitor_THT:CP_Radial_D5.0mm_P2.50mm, symbol Device:CP1_Small
- removed D55: clk, LED_THT:LED_D3.0mm, symbol Device:LED
- removed Q1, Q2, Q3, Q4: BC337, Package_TO_SOT_THT:TO-92_Inline, symbol Transistor_BJT:BC337
- removed R52, R53, R57, R62, R63, R71: 1k, Resistor_THT:R_Axial_DIN0207_L6.3mm_D2.5mm_P7.62mm_Horizontal, symbol Device:R
- removed R56: 1M, Resistor_THT:R_Axial_DIN0207_L6.3mm_D2.5mm_P7.62mm_Horizontal, symbol Device:R
- removed R64, R65: 100k, symbol Device:R
- removed R66, R67, R68, R69: 10k, symbol Device:R
- removed R70: 1k, symbol Device:R
- removed R72: 10k, Resistor_THT:R_Axial_DIN0207_L6.3mm_D2.5mm_P7.62mm_Horizontal, symbol Device:R
- removed RV1: 1M, Potentiometer_THT:Potentiometer_Bourns_PTV09A-1_Single_Vertical, symbol Device:R_POT
- removed SW1: clk_switch, Button_Switch_THT:SW_PUSH_6mm, symbol Switch:SW_Push
- removed SW2: SW_SPDT, symbol Switch:SW_SPDT
- removed SW3: continue_switch, Button_Switch_THT:SW_PUSH_6mm, symbol Switch:SW_Push
- removed U50, U51, U71: NA555P, Package_DIP:DIP-8_W7.62mm, symbol Timer:NA555P
- removed U69: 74LS157, symbol 74xx:74LS157
- removed U70: 74LS00, symbol 74xx:74LS00
- added C1, C2, C3, C4: 100n, symbol Device:C
- added R1, R2, R3, R4: 10k, symbol Device:R
- added R5, R6, R7, R8: 220k, symbol Device:R
- added SW1, SW3, SW4: SW_SPST, symbol Switch:SW_SPST
- added SW2, SW5: SW_MEC_5G, symbol Switch:SW_MEC_5G
- added U33: 74LS14, symbol 74xx:74LS14
- added U34: ds1813, symbol 8bitCPU-rescue:ds1813
- added U35: 74LS273, symbol 74xx:74LS273
- added U36, U38: 74LS08, symbol 74xx:74LS08
- added U37: 74LS32, symbol 74xx:74LS32
- added U39: 74LS151, symbol 74xx:74LS151
- added U95: 74ABT540, symbol 8bitCPU-rescue:74ABT540
- added X1: CXO_DIP14, Oscillator:Oscillator_DIP-14, symbol Oscillator:CXO_DIP14
Connections:
- net labels added: clk', i0, i1, i2, r0, r1, r2, s0, s1, s2, s3, s4, s5, ~breakpointEnable~, ~breakpointHit~, ~ctrlInstrFinished~
- net labels removed: clk0, clk1, clkSel, haltPulse
- wire segments 87 -> 129
- no-connect marks 11 -> 10
Other:
- note added: "D"
- note added: "Q"
- note added: "Switch Instruction or Cycle\n(Closed: Instruction, Open: Cycle)"
- note added: "Switch Step or Run\n(Closed: Step, Open: Run)"
- note added: "Switch enable breakpoint\n(Closed: Disable breakpoint, Open: Enable breakpoint)"
- note added: "reset switch"
- note added: "step switch\n(do one step when pressed)"
- note removed: "clock gen"
- note removed: "clock select (debounce)"
- note removed: "halt amp"
- note removed: "halt latch"
- note removed: "manual clock button (debounce)"
- note removed: "pulse invert"

Commit message: renamed project
Parts:
- U34: symbol 8bitCPU-rescue:ds1813 -> MEDiC-rescue:ds1813
- U95: symbol 8bitCPU-rescue:74ABT540 -> MEDiC-rescue:74ABT540
Changed lines of the file:
@@
 $EndComp
 $Comp
-L 8bitCPU-rescue:ds1813 U34
+L MEDiC-rescue:ds1813 U34
 U 1 1 6164C30A
 P 2450 7950
@@
 reset switch
 $Comp
-L 8bitCPU-rescue:74ABT540 U95
+L MEDiC-rescue:74ABT540 U95
 U 1 1 63BAC286
 P 5000 9800

Commit message: renamed project
Parts:
- U34: symbol MEDiC-rescue:ds1813 -> EDiC-rescue:ds1813
- U95: symbol MEDiC-rescue:74ABT540 -> EDiC-rescue:74ABT540
Changed lines of the file:
@@
 $EndComp
 $Comp
-L MEDiC-rescue:ds1813 U34
+L EDiC-rescue:ds1813 U34
 U 1 1 6164C30A
 P 2450 7950
@@
 reset switch
 $Comp
-L MEDiC-rescue:74ABT540 U95
+L EDiC-rescue:74ABT540 U95
 U 1 1 63BAC286
 P 5000 9800
