File: schematic/CPU/Regset.sch (KiCad schematic (older format))
At the start: 39 parts, among them U31 74LS374, U32 74LS157, U33 74LS157, U34 74LS374, U35 74LS157, U39 74LS157, U43 74LS245

Commit message: schematic finished
Other:
- note added: "board 02"
- note added: "board 03\n"
- moved on the sheet: R10, R11, R12, R13, R14, R15, R16, R17, R18, R19, R20, R21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

Commit message: pre upgrade to vivado 2021
Parts:
- removed U31, U34: 74LS374, Package_DIP:DIP-20_W7.62mm, symbol 74xx:74LS374
- removed U32, U33: 74LS157, Package_DIP:DIP-16_W7.62mm, symbol 74xx:74LS157
- removed U43: 74LS245, Package_DIP:DIP-20_W7.62mm, symbol 74xx:74LS245
- added U33, U34: 74AS825, symbol 74xx:74AS825
- added U43, U68: 74LS157, symbol 74xx:74LS157
- added U78: 74LS245, symbol 74xx:74LS245
- U35, U39: footprint Package_DIP:DIP-16_W7.62mm -> (none)
Connections:
- net labels added: bus0, bus1, bus2, bus3, bus4, bus5, bus6, bus7, clk, ~ctrlReg0WE~, ~ctrlReg1WE~, ~reset~
- net labels removed: b0, b1, b2, b3, b4, b5, b6, b7, d0, d1, d2, d3, d4, d5, d6, d7, r0_cp, r1_cp
- wire segments 67 -> 81
Other:
- note removed: "board 02"
- note removed: "board 03\n"

Commit message: fibonacci works again with new memory design
Connections:
- net labels added: ctrlRegAluSel
- net labels removed: ctrlAluSel
Changed lines of the file:
@@
 $Descr A3 16535 11693
 encoding utf-8
-Sheet 19 20
+Sheet 15 17
 Title ""
 Date ""
@@
 r17
 Text GLabel 5550 4900 0    50   Input ~ 0
-ctrlAluSel
+ctrlRegAluSel
 Text GLabel 5550 7400 0    50   Input ~ 0
-ctrlAluSel
+ctrlRegAluSel
 Text GLabel 7600 4900 0    50   Input ~ 0
 ctrlRegBusSel

Commit message: schematic with henry
Parts:
- removed D10, D11, D12, D13, D14, D15, D16, D17, D18, D19, D20, D21, D22, D23, D24, D9: LED, LED_THT:LED_D3.0mm, symbol Device:LED
- removed R10, R11, R12, R13, R14, R15, R16, R17, R18, R19, R20, R21, R22, R23, R24, R9: 1k, Resistor_THT:R_Axial_DIN0207_L6.3mm_D2.5mm_P7.62mm_Horizontal, symbol Device:R
- removed U43, U68: 74LS157, symbol 74xx:74LS157
- added D17, D18, D19, D20, D21, D22, D23, D24, D25, D26, D27, D28, D29, D30, D31, D32: LED_Small, symbol Device:LED_Small
- added RN4, RN5: 220, Resistor_THT:R_Array_SIP9, symbol Device:R_Network08
- added U45: 74LS245, symbol 74xx:74LS245
- added U46, U47: 74ABT540, symbol 8bitCPU-rescue:74ABT540
- U40: renamed from U33; symbol 74xx:74AS825 -> 8bitCPU-rescue:74AS825-74xx
- U41: renamed from U34; symbol 74xx:74AS825 -> 8bitCPU-rescue:74AS825-74xx
- renumbered U35 to U42, U39 to U43, U78 to U44
Connections:
- net labels added: ~ctrlReg0BusOE~, ~ctrlReg1BusOE~
- net labels removed: ctrlRegBusSel, ~ctrlRegBusOE~
- wire segments 81 -> 66
Other:
- moved on the sheet: U44

Commit message: renamed project
Parts:
- U40, U41: symbol 8bitCPU-rescue:74AS825-74xx -> MEDiC-rescue:74AS825-74xx
- U46, U47: symbol 8bitCPU-rescue:74ABT540 -> MEDiC-rescue:74ABT540
Changed lines of the file:
@@
 ~ctrlReg0WE~
 $Comp
-L 8bitCPU-rescue:74AS825-74xx U40
+L MEDiC-rescue:74AS825-74xx U40
 U 1 1 611197FA
 P 4050 4200
@@
 ~ctrlReg1WE~
 $Comp
-L 8bitCPU-rescue:74AS825-74xx U41
+L MEDiC-rescue:74AS825-74xx U41
 U 1 1 61169563
 P 4050 6700
@@
 r17
 $Comp
-L 8bitCPU-rescue:74ABT540 U?
+L MEDiC-rescue:74ABT540 U?
 U 1 1 633E01ED
 P 11050 4350
@@
 r07
 $Comp
-L 8bitCPU-rescue:74ABT540 U?
+L MEDiC-rescue:74ABT540 U?
 U 1 1 633F48E3
 P 11050 6500

Commit message: renamed project
Parts:
- U40, U41: symbol MEDiC-rescue:74AS825-74xx -> EDiC-rescue:74AS825-74xx
- U46, U47: symbol MEDiC-rescue:74ABT540 -> EDiC-rescue:74ABT540
Changed lines of the file:
@@
 ~ctrlReg0WE~
 $Comp
-L MEDiC-rescue:74AS825-74xx U40
+L EDiC-rescue:74AS825-74xx U40
 U 1 1 611197FA
 P 4050 4200
@@
 ~ctrlReg1WE~
 $Comp
-L MEDiC-rescue:74AS825-74xx U41
+L EDiC-rescue:74AS825-74xx U41
 U 1 1 61169563
 P 4050 6700
@@
 r17
 $Comp
-L MEDiC-rescue:74ABT540 U?
+L EDiC-rescue:74ABT540 U?
 U 1 1 633E01ED
 P 11050 4350
@@
 r07
 $Comp
-L MEDiC-rescue:74ABT540 U?
+L EDiC-rescue:74ABT540 U?
 U 1 1 633F48E3
 P 11050 6500
