File: schematic/CPU/Memory.sch (KiCad schematic (older format))
At the start: 16 parts, among them U32 74AS867, U341 74LS08, U79 74AS867, U80 74AS867, U81 28C256, U82 74LS157, U83 74LS157, U84 74AS825, U85 28C256, U86 AS6C4008-55PCN, U87 74AS825, U88 28C256, U89 74LS245, U90 74AS825, U91 74LS08, U92 74LS08

Commit message: fibonacci works again with new memory design
Parts:
- removed unit 4 of U341
- removed U82, U83: 74LS157, symbol 74xx:74LS157
- added U30, U37, U38, U45, U46, U47: 74LS245, symbol 74xx:74LS245
- added U31, U40: 74AS825, symbol 74xx:74AS825
- added U52: 74LS04, symbol 74xx:74LS04
Connections:
- net labels added: ctrlMemInstrImmToRam, ctrlMemSPUp, mar10, mar11, mar12, mar13, mar14, mar15, mar8, mar9, ramAddress0, ramAddress1, ramAddress10, ramAddress11, ramAddress12, ramAddress13, ramAddress14, ramAddress15, ramAddress2, ramAddress3, ramAddress4, ramAddress5, ramAddress6, ramAddress7, ramAddress8, ramAddress9, select0, select1, select2, select3, select4, select5, select6, select7, ~ctrlMemInstrOE~, ~ctrlMemInstrWE~, ~ctrlMemMar0WE~, ~ctrlMemMar1WE~, ~ctrlMemPCIncr~, ~ctrlMemPCLoad~, ~ctrlMemRamOE~, ~ctrlMemRamWE~, ~ctrlMemSPEn~, ~instrImm0ToRam~, ~instrImm1Select~, ~instrImm1ToRam~, ~mar1ToRam~, ~spToRam~
- net labels removed: sp0, sp1, sp2, sp3, sp4, sp5, sp6, sp7, spUp, ~ctrlInstrWE~, ~ctrlPCIncr~, ~ctrlPCLoad~, ~ctrlRamOE~, ~ctrlRamWE~, ~spEn~
- wire segments 298 -> 322
- no-connect marks 13 -> 9
Other:
- note added: "24bit instructions:\nrom2 23:16 - instruction to decode\nrom1&0 15:0 - immediate:\n7:0 data for ALU OP or reg\n15:0 address for PC (jump) or RAM (memory OP)"
- note added: "mar0"
- note added: "mar1"
- note added: "ramAddress:\n7:0 -> instrImm or mar0 (depending on ctrlMemInstrImmToRam)\n15:0 -> instrImm or mar1 or sp (depending on ctrlMemInstrImmToRam and selectStackMem)"
- note added: "~instrImm0ToRam~=!ctrlMemInstrImmToRam"
- note added: "~instrImm1ToRam~=!(!ctrlMemInstrImmToRam and ~selectStackMem~)"
- note removed: "24bit instructions:\nrom2 23:16 - instruction to decode\nrom1&0 15:0 - immediate:\n7:0 data for ALU OP\n15:0 address for PC (jump) or RAM (memory OP)"
- note removed: "upper 256 byte -> stack dependant:\na16 is high and a15:a8 is sp instead of 0xff"
- moved on the sheet: U341A, U341C, U86, U88, U89, U91A, U91B, U91C, U91D, U91E, U92A, U92B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

Commit message: schematic with henry
Parts:
- removed unit 1 of U91
- removed unit 2 of U91
- removed unit 3 of U91
- removed unit 4 of U92
- removed unit 1 of U92
- removed unit 2 of U92
- removed unit 3 of U92
- added D33, D34, D35, D36, D37, D38, D39, D40, D41, D42, D43, D44, D45, D46, D47, D48: LED_Small, symbol Device:LED_Small
- added RN6, RN7: 10k, Resistor_THT:R_Array_SIP9, symbol Device:R_Network08
- added RN8, RN9: 220, Resistor_THT:R_Array_SIP9, symbol Device:R_Network08
- added SW6, SW7, SW8, SW9: SW_Coded_SH-7050, symbol Switch:SW_Coded_SH-7050
- added U49, U50, U51, U52: 74LS245, symbol 74xx:74LS245
- added U53, U60, U76, U79: 74F521, symbol 8bitCPU-rescue:74F521
- added U57, U58: 74ABT540, symbol 8bitCPU-rescue:74ABT540
- added U80: 74LS04, symbol 74xx:74LS04
- U54: renamed from U32; symbol 74xx:74AS867 -> 8bitCPU-rescue:74AS867-74xx
- U55: renamed from U79; symbol 74xx:74AS867 -> 8bitCPU-rescue:74AS867-74xx
- U56: renamed from U80; symbol 74xx:74AS867 -> 8bitCPU-rescue:74AS867-74xx
- U63: renamed from U31; symbol 74xx:74AS825 -> 8bitCPU-rescue:74AS825-74xx
- U64: renamed from U84; symbol 74xx:74AS825 -> 8bitCPU-rescue:74AS825-74xx
- U68: renamed from U40; symbol 74xx:74AS825 -> 8bitCPU-rescue:74AS825-74xx
- U70: renamed from U87; symbol 74xx:74AS825 -> 8bitCPU-rescue:74AS825-74xx
- U71: renamed from U90; symbol 74xx:74AS825 -> 8bitCPU-rescue:74AS825-74xx
- renumbered U341 to U36, U91 to U38, U341 to U38, U52 to U48, U341 to U59, U91 to U59, U30 to U61, U81 to U62, U37 to U65, U38 to U66, U85 to U67, U88 to U69, U45 to U72, U46 to U73, U47 to U74, U89 to U75, U86 to U77, U92 to U78
Connections:
- net labels added: comp0, comp1, comp10, comp11, comp12, comp13, comp14, comp15, comp2, comp3, comp4, comp5, comp6, comp7, comp8, comp9, ioAddr0, ioAddr1, ioAddr2, ioAddr3, ioAddr4, ioAddr5, ioAddr6, ioAddr7, ioSelect, pcIn0, pcIn1, pcIn10, pcIn11, pcIn12, pcIn13, pcIn14, pcIn15, pcIn2, pcIn3, pcIn4, pcIn5, pcIn6, pcIn7, pcIn8, pcIn9, ~breakpointEnable~, ~breakpointHit~, ~ctrlMemPC0FromBus~, ~ctrlMemPC1FromBus~, ~ctrlMemPCEn~, ~ioOE~, ~ioWE~, ~ramCE~
- net labels removed: ~ctrlMemPCIncr~
- wire segments 322 -> 487
- no-connect marks 9 -> 4
Other:
- note added: "Invertierung beachten!"
- moved on the sheet: U36B, U38C, U38D, U38E, U48A, U48B, U48C, U48D, U48E, U48F, U48G, U59A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

Commit message: updated verilog from schematic
Other:
- note added: "select == 0xff: stack\nselect == 0xfe: io\notherwise: ram"
- note added: "~instrImm0ToRam~=~ctrlMemInstrImmToRam~\n\n~instrImm1ToRam~=!(~ctrlMemInstrImmToRam~ and ~selectStackMem~)\n\n~mar1ToRam~=!(ctrlMemInstrImmToRam and ~selectStackMem~)"
- note removed: "~instrImm0ToRam~=!ctrlMemInstrImmToRam"
- note removed: "~instrImm1ToRam~=!(!ctrlMemInstrImmToRam and ~selectStackMem~)"
Changed lines of the file:
@@
 Text Label 18750 9550 0    50   ~ 0
 ~instrImm1Select~
-Text Notes 17450 8950 0    50   ~ 0
-~instrImm1ToRam~=!(!ctrlMemInstrImmToRam and ~selectStackMem~)
 Wire Wire Line
 	20200 10650 20250 10650
@@
 	1    0    0    -1
 $EndComp
-Text Notes 17450 8800 0    50   ~ 0
-~instrImm0ToRam~=!ctrlMemInstrImmToRam
-Text Notes 17450 8650 0    100  ~ 20
+Text Notes 17500 9150 0    50   ~ 0
+~instrImm0ToRam~=~ctrlMemInstrImmToRam~\n\n~instrImm1ToRam~=!(~ctrlMemInstrImmToRam~ and ~selectStackMem~)\n\n~mar1ToRam~=!(ctrlMemInstrImmToRam and ~selectStackMem~)
+Text Notes 17450 8650 0    100  ~ 0
 ramAddress:\n7:0 -> instrImm or mar0 (depending on ctrlMemInstrImmToRam)\n15:0 -> instrImm or mar1 or sp (depending on ctrlMemInstrImmToRam and selectStackMem)
 $Comp
@@
 Text Label 7550 18000 2    50   ~ 0
 pc7
+Text Notes 18800 11700 0    100  ~ 0
+select == 0xff: stack\nselect == 0xfe: io\notherwise: ram
 $EndSCHEMATC

Commit message: renamed project
Parts:
- U53, U60, U76, U79: symbol 8bitCPU-rescue:74F521 -> MEDiC-rescue:74F521
- U54, U55, U56: symbol 8bitCPU-rescue:74AS867-74xx -> MEDiC-rescue:74AS867-74xx
- U57, U58: symbol 8bitCPU-rescue:74ABT540 -> MEDiC-rescue:74ABT540
- U63, U64, U68, U70, U71: symbol 8bitCPU-rescue:74AS825-74xx -> MEDiC-rescue:74AS825-74xx
Changed lines of the file:
@@
 $EndComp
 $Comp
-L 8bitCPU-rescue:74AS867-74xx U54
+L MEDiC-rescue:74AS867-74xx U54
 U 1 1 614A13D4
 P 8350 4700
@@
 $EndComp
 $Comp
-L 8bitCPU-rescue:74AS867-74xx U55
+L MEDiC-rescue:74AS867-74xx U55
 U 1 1 614A1BAD
 P 8350 7650
@@
 	10150 5100 10050 5100
 $Comp
-L 8bitCPU-rescue:74AS867-74xx U56
+L MEDiC-rescue:74AS867-74xx U56
 U 1 1 614C84B2
 P 8350 9800
@@
 $EndComp
 $Comp
-L 8bitCPU-rescue:74AS825-74xx U70
+L MEDiC-rescue:74AS825-74xx U70
 U 1 1 622368AD
 P 14850 2250
@@
 ~ctrlMemInstrWE~
 $Comp
-L 8bitCPU-rescue:74AS825-74xx U71
+L MEDiC-rescue:74AS825-74xx U71
 U 1 1 622CCE3A
 P 15800 4500
@@
 	12750 4300 12900 4300
 $Comp
-L 8bitCPU-rescue:74AS825-74xx U64
+L MEDiC-rescue:74AS825-74xx U64
 U 1 1 6255A4D7
 P 12250 4800
@@
 $EndComp
 $Comp
-L 8bitCPU-rescue:74AS825-74xx U63
+L MEDiC-rescue:74AS825-74xx U63
 U 1 1 6172F6E1
 P 10700 7650
@@
 $EndComp
 $Comp
-L 8bitCPU-rescue:74AS825-74xx U68
+L MEDiC-rescue:74AS825-74xx U68
 U 1 1 61818E6C
 P 13350 7350
@@
 ~ctrlMemPC1FromBus~
 $Comp
-L 8bitCPU-rescue:74F521 U53
+L MEDiC-rescue:74F521 U53
 U 1 1 616FD36C
 P 8000 12900
@@
 $EndComp
 $Comp
-L 8bitCPU-rescue:74F521 U60
+L MEDiC-rescue:74F521 U60
 U 1 1 616FE128
 P 10000 12850
@@
 comp14
 $Comp
-L 8bitCPU-rescue:74F521 U76
+L MEDiC-rescue:74F521 U76
 U 1 1 62289ACE
 P 18950 12800
@@
 	19000 12000 18850 12000
 $Comp
-L 8bitCPU-rescue:74F521 U79
+L MEDiC-rescue:74F521 U79
 U 1 1 625D2667
 P 21250 12750
@@
 	22650 13300 22300 13300
 $Comp
-L 8bitCPU-rescue:74ABT540 U?
+L MEDiC-rescue:74ABT540 U?
 U 1 1 634E144D
 P 8350 17800
@@
 	9350 18000 8950 18000
 $Comp
-L 8bitCPU-rescue:74ABT540 U?
+L MEDiC-rescue:74ABT540 U?
 U 1 1 6363F628
 P 8350 19900

Commit message: fibonacci works again, sp etc needs to be tested
Parts:
- added U100: AS6C4008-55PCN, Package_DIP:DIP-32_W15.24mm, symbol Memory_RAM:AS6C4008-55PCN
- added unit 2 of U80
- added U98, U99: 74LS245, symbol 74xx:74LS245
Connections:
- net ~ctrlMemPC1FromBus~ is gone; now on net ctrlMemPCFromImm: U48.11, U49.19 (CE)
- net +5V: now also U100.32 (VCC), U98.1 (A->B), U98.20 (VCC), U99.1 (A->B), U99.20 (VCC)
- net GND: now also U100.16 (VSS), U98.10 (GND), U99.10 (GND)
- net bus0: now also U99.18 (B0); no longer U49.2 (A0)
- net bus1: now also U99.17 (B1); no longer U49.3 (A1)
- net bus2: now also U99.16 (B2); no longer U49.4 (A2)
- net bus3: now also U99.15 (B3); no longer U49.5 (A3)
- net bus4: now also U99.14 (B4); no longer U49.6 (A4)
- net bus5: now also U99.13 (B5); no longer U49.7 (A5)
- net bus6: now also U99.12 (B6); no longer U49.8 (A6)
- net bus7: now also U99.11 (B7); no longer U49.9 (A7)
- net ioAddr0: now also U100.12 (A0)
- net ioAddr1: now also U100.11 (A1)
- net ioAddr2: now also U100.10 (A2)
- net ioAddr3: now also U100.9 (A3)
- net ioAddr4: now also U100.8 (A4)
- net ioAddr5: now also U100.7 (A5)
- net ioAddr6: now also U100.6 (A6)
- net ioAddr7: now also U100.5 (A7)
- net pc0: now also U99.2 (A0)
- net pc1: now also U99.3 (A1)
- net pc10: now also U98.4 (A2)
- net pc11: now also U98.5 (A3)
- net pc12: now also U98.6 (A4)
- net pc13: now also U98.7 (A5)
- net pc14: now also U98.8 (A6)
- net pc15: now also U98.9 (A7)
- net pc2: now also U99.4 (A2)
- net pc3: now also U99.5 (A3)
- net pc4: now also U99.6 (A4)
- net pc5: now also U99.7 (A5)
- net pc6: now also U99.8 (A6)
- net pc7: now also U99.9 (A7)
- net pc8: now also U98.2 (A0)
- net pc9: now also U98.3 (A1)
- net ramAddress10: now also U100.23 (A10)
- net ramAddress11: now also U100.25 (A11)
- net ramAddress12: now also U100.4 (A12)
- net ramAddress13: now also U100.28 (A13)
- net ramAddress14: now also U100.3 (A14)
- net ramAddress15: now also U100.31 (A15)
- net ramAddress8: now also U100.27 (A8)
- net ramAddress9: now also U100.26 (A9)
- net selectStackMem: now also U100.2 (A16)
- net ~ctrlMemRamWE~: now also U100.29 (WE#)
- net ~ramCE~: now also U100.22 (CE#)
- net ctrlMemInstrImmToRam renamed ctrlMemInstrImmToRamAddr
- net ~ctrlMemPC0FromBus~ renamed ctrlMemPCFromImm
- new net: U100.24 (OE#), U80.4
- new net ram2data0: U100.13 (DQ0), U49.2 (A0), U98.18 (B0)
- new net ram2data1: U100.14 (DQ1), U49.3 (A1), U98.17 (B1)
- new net ram2data2: U100.15 (DQ2), U49.4 (A2), U98.16 (B2)
- new net ram2data3: U100.17 (DQ3), U49.5 (A3), U98.15 (B3)
- new net ram2data4: U100.18 (DQ4), U49.6 (A4), U98.14 (B4)
- new net ram2data5: U100.19 (DQ5), U49.7 (A5), U98.13 (B5)
- new net ram2data6: U100.20 (DQ6), U49.8 (A6), U98.12 (B6)
- new net ram2data7: U100.21 (DQ7), U49.9 (A7), U98.11 (B7)
- new net ~ctrlMemPCToRam~: U80.3, U98.19 (CE), U99.19 (CE)
- no-connect marks 4 -> 6
Other:
- note added: "ramAddress:\n7:0 -> instrImm or mar0 (depending on ctrlMemInstrImmToRamAddr)\n15:0 -> instrImm or mar1 or sp (depending on ctrlMemInstrImmToRam and selectStackMem)"
- note added: "~instrImm0ToRam~=~ctrlMemInstrImmToRamAddr~\n\n~instrImm1ToRam~=!(~ctrlMemInstrImmToRam~ and ~selectStackMem~)\n\n~mar1ToRam~=!(ctrlMemInstrImmToRam and ~selectStackMem~)"
- note removed: "ramAddress:\n7:0 -> instrImm or mar0 (depending on ctrlMemInstrImmToRam)\n15:0 -> instrImm or mar1 or sp (depending on ctrlMemInstrImmToRam and selectStackMem)"
- note removed: "~instrImm0ToRam~=~ctrlMemInstrImmToRam~\n\n~instrImm1ToRam~=!(~ctrlMemInstrImmToRam~ and ~selectStackMem~)\n\n~mar1ToRam~=!(ctrlMemInstrImmToRam and ~selectStackMem~)"
- moved on the sheet: U48D, U48E

Commit message: renamed project
Parts:
- U53, U60, U76, U79: symbol MEDiC-rescue:74F521 -> EDiC-rescue:74F521
- U54, U55, U56: symbol MEDiC-rescue:74AS867-74xx -> EDiC-rescue:74AS867-74xx
- U57, U58: symbol MEDiC-rescue:74ABT540 -> EDiC-rescue:74ABT540
- U63, U64, U68, U70, U71: symbol MEDiC-rescue:74AS825-74xx -> EDiC-rescue:74AS825-74xx
Changed lines of the file:
@@
 $EndComp
 $Comp
-L MEDiC-rescue:74AS867-74xx U54
+L EDiC-rescue:74AS867-74xx U54
 U 1 1 614A13D4
 P 8350 4700
@@
 $EndComp
 $Comp
-L MEDiC-rescue:74AS867-74xx U55
+L EDiC-rescue:74AS867-74xx U55
 U 1 1 614A1BAD
 P 8350 7650
@@
 	10150 5100 10050 5100
 $Comp
-L MEDiC-rescue:74AS867-74xx U56
+L EDiC-rescue:74AS867-74xx U56
 U 1 1 614C84B2
 P 8350 9800
@@
 $EndComp
 $Comp
-L MEDiC-rescue:74AS825-74xx U70
+L EDiC-rescue:74AS825-74xx U70
 U 1 1 622368AD
 P 14850 2250
@@
 ~ctrlMemInstrWE~
 $Comp
-L MEDiC-rescue:74AS825-74xx U71
+L EDiC-rescue:74AS825-74xx U71
 U 1 1 622CCE3A
 P 15800 4500
@@
 	12750 4300 12900 4300
 $Comp
-L MEDiC-rescue:74AS825-74xx U64
+L EDiC-rescue:74AS825-74xx U64
 U 1 1 6255A4D7
 P 12250 4800
@@
 $EndComp
 $Comp
-L MEDiC-rescue:74AS825-74xx U63
+L EDiC-rescue:74AS825-74xx U63
 U 1 1 6172F6E1
 P 10700 7650
@@
 $EndComp
 $Comp
-L MEDiC-rescue:74AS825-74xx U68
+L EDiC-rescue:74AS825-74xx U68
 U 1 1 61818E6C
 P 13350 7350
@@
 ctrlMemPCFromImm
 $Comp
-L MEDiC-rescue:74F521 U53
+L EDiC-rescue:74F521 U53
 U 1 1 616FD36C
 P 8000 12900
@@
 $EndComp
 $Comp
-L MEDiC-rescue:74F521 U60
+L EDiC-rescue:74F521 U60
 U 1 1 616FE128
 P 10000 12850
@@
 comp14
 $Comp
-L MEDiC-rescue:74F521 U76
+L EDiC-rescue:74F521 U76
 U 1 1 62289ACE
 P 18950 12800
@@
 	19000 12000 18850 12000
 $Comp
-L MEDiC-rescue:74F521 U79
+L EDiC-rescue:74F521 U79
 U 1 1 625D2667
 P 21250 12750
@@
 	22650 13300 22300 13300
 $Comp
-L MEDiC-rescue:74ABT540 U?
+L EDiC-rescue:74ABT540 U?
 U 1 1 634E144D
 P 8350 17800
@@
 	9350 18000 8950 18000
 $Comp
-L MEDiC-rescue:74ABT540 U?
+L EDiC-rescue:74ABT540 U?
 U 1 1 6363F628
 P 8350 19900

Commit message: debugged debugging
Parts:
- added U? (x2): 74LS32, symbol 74xx:74LS32
- added U?: 74LS08, symbol 74xx:74LS08
Connections:
- net ~ctrlMemPCEn~: now also U?.1; no longer U54.23 (~ENP~), U55.23 (~ENP~)
- net ~ctrlMemPCLoad~: now also U?.2
- net ~ctrlMemSPEn~: now also U?.1; no longer U56.23 (~ENP~)
- new net: U?.1, U?.3
- new net halt: U?.2, U?.2
- new net ~pcEn~: U54.23 (~ENP~), U55.23 (~ENP~), U?.3
- new net ~spEn~: U56.23 (~ENP~), U?.3
Changed lines of the file:
@@
 Wire Wire Line
 	7150 5400 7850 5400
-Text GLabel 7850 5500 0    50   Input ~ 0
-~ctrlMemPCEn~
-Text GLabel 7850 8450 0    50   Input ~ 0
+Text GLabel 5650 1700 0    50   Input ~ 0
 ~ctrlMemPCEn~
 Text GLabel 7800 2850 0    50   Input ~ 0
@@
 Text GLabel 7850 10200 0    50   Input ~ 0
 clk
-Text GLabel 7800 10600 0    50   Input ~ 0
+Text GLabel 5650 1150 0    50   Input ~ 0
 ~ctrlMemSPEn~
-Wire Wire Line
-	7800 10600 7850 10600
 $Comp
 L power:GND #PWR0178
@@
 Text GLabel 4050 10150 0    50   Input ~ 0
 ctrlMemPCFromImm
+$Comp
+L 74xx:74LS32 U?
+U 1 1 61A2880A
+P 6050 1800
+F 0 "U?" H 6050 2125 50  0000 C CNN
+F 1 "74LS32" H 6050 2034 50  0000 C CNN
+F 2 "" H 6050 1800 50  0001 C CNN
+F 3 "http://www.ti.com/lit/gpn/sn74LS32" H 6050 1800 50  0001 C CNN
+	1    6050 1800
+	1    0    0    -1
+$EndComp
+Wire Wire Line
+	6350 1800 6450 1800
+Wire Wire Line
+	6450 1800 6450 1900
+Wire Wire Line
+	6450 1900 6550 1900
+Wire Wire Line
+	5650 1700 5750 1700
+Text Label 7350 2000 0    50   ~ 0
+~pcEn~
+Wire Wire Line
+	7350 2000 7150 2000
+Text GLabel 5650 1900 0    50   Input ~ 0
+halt
+Wire Wire Line
+	5650 1900 5750 1900
+Text Label 7700 5500 2    50   ~ 0
+~pcEn~
+Wire Wire Line
+	7700 5500 7850 5500
+Text Label 7700 8450 2    50   ~ 0
+~pcEn~
+Wire Wire Line
+	7700 8450 7850 8450
+$Comp
+L 74xx:74LS08 U?
+U 1 1 61D31E8E
+P 6850 2000
+F 0 "U?" H 6850 2325 50  0000 C CNN
+F 1 "74LS08" H 6850 2234 50  0000 C CNN
+F 2 "" H 6850 2000 50  0001 C CNN
+F 3 "http://www.ti.com/lit/gpn/sn74LS08" H 6850 2000 50  0001 C CNN
+	1    6850 2000
+	1    0    0    -1
+$EndComp
+Text GLabel 6350 2100 0    50   Input ~ 0
+~ctrlMemPCLoad~
+Wire Wire Line
+	6350 2100 6550 2100
+$Comp
+L 74xx:74LS32 U?
+U 1 1 61DAB1DF
+P 6050 1250
+F 0 "U?" H 6050 1575 50  0000 C CNN
+F 1 "74LS32" H 6050 1484 50  0000 C CNN
+F 2 "" H 6050 1250 50  0001 C CNN
+F 3 "http://www.ti.com/lit/gpn/sn74LS32" H 6050 1250 50  0001 C CNN
+	1    6050 1250
+	1    0    0    -1
+$EndComp
+Wire Wire Line
+	5650 1150 5750 1150
+Text GLabel 5650 1350 0    50   Input ~ 0
+halt
+Wire Wire Line
+	5650 1350 5750 1350
+Text Label 6500 1250 0    50   ~ 0
+~spEn~
+Wire Wire Line
+	6500 1250 6350 1250
+Text Label 7700 10600 2    50   ~ 0
+~spEn~
+Wire Wire Line
+	7700 10600 7850 10600
 $EndSCHEMATC

Commit message: fixed uart_rx and snake
Parts:
- gave numbers to parts that had none: 2
Connections:
- net halt: now also U103.5; no longer U103.2
- net ~ctrlMemPCEn~: now also U103.4; no longer U103.1
- net at U105.1: now also U103.6; no longer U103.3
Changed lines of the file:
@@
 ctrlMemPCFromImm
 $Comp
-L 74xx:74LS32 U?
-U 1 1 61A2880A
+L 74xx:74LS32 U103
+U 2 1 61A2880A
 P 6050 1800
-F 0 "U?" H 6050 2125 50  0000 C CNN
+F 0 "U103" H 6050 2125 50  0000 C CNN
 F 1 "74LS32" H 6050 2034 50  0000 C CNN
 F 2 "" H 6050 1800 50  0001 C CNN
 F 3 "http://www.ti.com/lit/gpn/sn74LS32" H 6050 1800 50  0001 C CNN
-	1    6050 1800
+	2    6050 1800
 	1    0    0    -1
 $EndComp
@@
 	7700 8450 7850 8450
 $Comp
-L 74xx:74LS08 U?
+L 74xx:74LS08 U105
 U 1 1 61D31E8E
 P 6850 2000
-F 0 "U?" H 6850 2325 50  0000 C CNN
+F 0 "U105" H 6850 2325 50  0000 C CNN
 F 1 "74LS08" H 6850 2234 50  0000 C CNN
 F 2 "" H 6850 2000 50  0001 C CNN
@@
 	6350 2100 6550 2100
 $Comp
-L 74xx:74LS32 U?
+L 74xx:74LS32 U103
 U 1 1 61DAB1DF
 P 6050 1250
-F 0 "U?" H 6050 1575 50  0000 C CNN
+F 0 "U103" H 6050 1575 50  0000 C CNN
 F 1 "74LS32" H 6050 1484 50  0000 C CNN
 F 2 "" H 6050 1250 50  0001 C CNN
@@
 Wire Wire Line
 	7700 10600 7850 10600
+Wire Notes Line rgb(255, 0, 0)
+	5050 2250 7650 2250
+Wire Notes Line rgb(255, 0, 0)
+	7650 2250 7650 850
+Wire Notes Line rgb(255, 0, 0)
+	7650 850  5050 850
+Wire Notes Line rgb(255, 0, 0)
+	5050 850  5050 2250
+Wire Notes Line rgb(255, 0, 0)
+	7450 5550 7750 5550
+Wire Notes Line rgb(255, 0, 0)
+	7750 5550 7750 5350
+Wire Notes Line rgb(255, 0, 0)
+	7750 5350 7450 5350
+Wire Notes Line rgb(255, 0, 0)
+	7450 5350 7450 5550
+Wire Notes Line rgb(255, 0, 0)
+	7500 8500 7800 8500
+Wire Notes Line rgb(255, 0, 0)
+	7500 8500 7500 8300
+Wire Notes Line rgb(255, 0, 0)
+	7500 8300 7800 8300
+Wire Notes Line rgb(255, 0, 0)
+	7800 8300 7800 8500
+Wire Notes Line rgb(255, 0, 0)
+	7500 10650 7500 10450
+Wire Notes Line rgb(255, 0, 0)
+	7500 10450 7750 10450
+Wire Notes Line rgb(255, 0, 0)
+	7750 10450 7750 10650
+Wire Notes Line rgb(255, 0, 0)
+	7500 10650 7750 10650
+Wire Notes Line rgb(255, 0, 0)
+	12350 8150 12350 7950
+Wire Notes Line rgb(255, 0, 0)
+	12350 7950 11150 7950
+Wire Notes Line rgb(255, 0, 0)
+	11150 7950 11150 8150
+Wire Notes Line rgb(255, 0, 0)
+	20600 8150 20600 5200
+Wire Notes Line rgb(255, 0, 0)
+	20600 5200 24650 5200
+Wire Notes Line rgb(255, 0, 0)
+	24650 5200 24650 8150
+Wire Notes Line rgb(255, 0, 0)
+	24650 8150 20600 8150
+Wire Notes Line rgb(255, 0, 0)
+	11150 8150 12350 8150
+Wire Notes Line rgb(255, 0, 0)
+	550  8650 3100 8650
+Wire Notes Line rgb(255, 0, 0)
+	3100 8650 3100 10350
+Wire Notes Line rgb(255, 0, 0)
+	3100 10350 4100 10350
+Wire Notes Line rgb(255, 0, 0)
+	4100 10350 4100 9950
+Wire Notes Line rgb(255, 0, 0)
+	4100 9950 3500 9950
+Wire Notes Line rgb(255, 0, 0)
+	3500 9950 3500 6100
+Wire Notes Line rgb(255, 0, 0)
+	3500 6100 4200 6100
+Wire Notes Line rgb(255, 0, 0)
+	4200 6100 4200 5750
+Wire Notes Line rgb(255, 0, 0)
+	4200 5750 3500 5750
+Wire Notes Line rgb(255, 0, 0)
+	3500 5750 3500 3750
+Wire Notes Line rgb(255, 0, 0)
+	3500 3750 550  3750
+Wire Notes Line rgb(255, 0, 0)
+	550  3750 550  8650
 $EndSCHEMATC
