File: schematic/CPU/Memory.sch (KiCad schematic (older format))
At the start: 64 parts, among them SW6 SW_Coded_SH-7050, SW7 SW_Coded_SH-7050, SW8 SW_Coded_SH-7050, SW9 SW_Coded_SH-7050, U100 AS6C4008-55PCN, U103 74LS32, U105 74LS08, U36 74LS08, U38 74LS08, U48 74LS04, U49 74LS245, U50 74LS245, U51 74LS245, U52 74LS245, U53 74F521, U54 74AS867, U55 74AS867, U56 74AS867, U57 74ABT540, U58 74ABT540, U59 74LS08, U60 74F521, U61 74LS245, U62 28C256, U63 74AS825, U64 74AS825, U65 74LS245, U66 74LS245, U67 28C256, U68 74AS825, U69 28C256, U70 74AS825, U71 74AS825, U72 74LS245, U73 74LS245, U74 74LS245, U75 74LS245, U76 74F521, U77 AS6C4008-55PCN, U78 74LS08, U79 74F521, U80 74LS04, U98 74LS245, U99 74LS245

Commit message: restructured folders
Parts:
- removed unit 2 of U48
Connections:
- net labels added: ~ioCE~, ~selectStackMem~
- net labels removed: ioSelect, selectStackMem
- wire segments 540 -> 539
Other:
- note added: "ramAddress:\n7:0 -> instrImm or mar0 (depending on ctrlMemInstrImmToRamAddr)\n15:0 -> instrImm or mar1 or sp (depending on ctrlMemInstrImmToRam and ~selectStackMem~)"
- note removed: "ramAddress:\n7:0 -> instrImm or mar0 (depending on ctrlMemInstrImmToRamAddr)\n15:0 -> instrImm or mar1 or sp (depending on ctrlMemInstrImmToRam and selectStackMem)"
Changed lines of the file:
@@
 $EndComp
 Text Label 18300 7450 2    50   ~ 0
-selectStackMem
+~selectStackMem~
 Wire Wire Line
 	18300 7450 18600 7450
@@
 Text Label 20250 10650 0    50   ~ 0
 ~instrImm1ToRam~
-Wire Wire Line
-	18500 10750 18600 10750
-$Comp
-L 74xx:74LS04 U48
-U 2 1 62160147
-P 18200 10750
-F 0 "U48" H 18200 11067 50  0000 C CNN
-F 1 "74LS04" H 18200 10976 50  0000 C CNN
-F 2 "" H 18200 10750 50  0001 C CNN
-F 3 "http://www.ti.com/lit/gpn/sn74LS04" H 18200 10750 50  0001 C CNN
-	2    18200 10750
-	1    0    0    -1
-$EndComp
 Text Label 17750 10750 2    50   ~ 0
-selectStackMem
+~selectStackMem~
 Wire Wire Line
 	18600 9400 18750 9400
@@
 ~instrImm0ToRam~=~ctrlMemInstrImmToRamAddr~\n\n~instrImm1ToRam~=!(~ctrlMemInstrImmToRam~ and ~selectStackMem~)\n\n~mar1ToRam~=!(ctrlMemInstrImmToRam and ~selectStackMem~)
 Text Notes 17450 8650 0    100  ~ 0
-ramAddress:\n7:0 -> instrImm or mar0 (depending on ctrlMemInstrImmToRamAddr)\n15:0 -> instrImm or mar1 or sp (depending on ctrlMemInstrImmToRam and selectStackMem)
+ramAddress:\n7:0 -> instrImm or mar0 (depending on ctrlMemInstrImmToRamAddr)\n15:0 -> instrImm or mar1 or sp (depending on ctrlMemInstrImmToRam and ~selectStackMem~)
 $Comp
 L 74xx:74LS08 U38
@@
 ~spToRam~
 Wire Wire Line
-	17750 10750 17900 10750
-Wire Wire Line
 	18600 10750 18600 11100
 Wire Wire Line
@@
 	17700 13800 17850 13800
 Text Label 19000 12000 0    50   ~ 0
-selectStackMem
+~selectStackMem~
 Wire Wire Line
 	19000 12000 18850 12000
@@
 Connection ~ 20000 13550
 Text GLabel 22650 11950 2    50   Output ~ 0
-ioSelect
+~ioCE~
 Wire Wire Line
 	21150 11950 21250 11950
@@
 $EndComp
 Text Label 21300 7450 2    50   ~ 0
-selectStackMem
+~selectStackMem~
 Wire Wire Line
 	21300 7450 21600 7450
@@
 Wire Notes Line rgb(255, 0, 0)
 	550  3750 550  8650
+Wire Wire Line
+	17750 10750 18600 10750
+Wire Notes Line
+	22900 12100 22550 12100
+Wire Notes Line
+	22550 12100 22550 11800
+Wire Notes Line
+	22550 11800 22900 11800
+Wire Notes Line
+	22900 11800 22900 12100
+Wire Notes Line
+	18900 11850 19650 11850
+Wire Notes Line
+	19650 11850 19650 12100
+Wire Notes Line
+	19650 12100 18900 12100
+Wire Notes Line
+	18900 12100 18900 11850
+Wire Notes Line
+	17100 10600 17100 10850
+Wire Notes Line
+	17100 10850 18550 10850
+Wire Notes Line
+	18550 10850 18550 10600
+Wire Notes Line
+	18550 10600 17100 10600
+Wire Notes Line
+	20650 7500 20650 7300
+Wire Notes Line
+	20650 7300 21350 7300
+Wire Notes Line
+	21350 7300 21350 7500
+Wire Notes Line
+	21350 7500 20650 7500
+Wire Notes Line
+	17650 7300 18350 7300
+Wire Notes Line
+	18350 7300 18350 7550
+Wire Notes Line
+	18350 7550 17650 7550
+Wire Notes Line
+	17650 7300 17650 7550
 $EndSCHEMATC
