File: schematic/CPU/Memory.kicad_sch (KiCad schematic)
At the start: 64 parts, among them SW6 SW_Coded_SH-7050, SW7 SW_Coded_SH-7050, SW8 SW_Coded_SH-7050, SW9 SW_Coded_SH-7050, U100 AS6C4008-55PCN, U103 74LS32, U105 74LS08, U36 74LS08, U38 74LS08, U48 74LS04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

Commit message: ttl fpga: factorization works in sim and fpga
Parts:
- removed unit 5 of U59
- removed U78: 74LS08, symbol 74xx:74LS08
- renumbered U59 to U38, U36 to U38
