File: schematic/CPU/io.kicad_sch (KiCad schematic)
At the start: 10 parts, among them SW10 SW_Coded_SH-7050, SW11 SW_Coded_SH-7050, U88 74F521, U89 74LS32, U90 74LS32, U91 74LS245, U92 74LS273, U93 5082_7340, U94 5082_7340

Commit message: netlist simulation works
Parts:
- removed U92: 74LS273, symbol 74xx:74LS273
- added U92: 74AS825, symbol EDiC-rescue:74AS825-74xx
Connections:
- net +5V: now also U92.24 (Vcc)
- net GND: now also U92.1 (~{OE1}), U92.12 (GND), U92.2 (~{OE2}), U92.23 (~{OE3})
- net bus0: now also U91.18 (B0), U92.3 (D0); no longer U91.11 (B7)
- net bus1: now also U91.17 (B1), U92.4 (D1); no longer U91.12 (B6)
- net bus2: now also U91.16 (B2), U92.5 (D2); no longer U91.13 (B5)
- net bus3: now also U91.15 (B3), U92.6 (D3); no longer U91.14 (B4)
- net bus4: now also U91.14 (B4), U92.7 (D4); no longer U91.15 (B3)
- net bus5: now also U91.13 (B5), U92.8 (D5); no longer U91.16 (B2)
- net bus6: now also U91.12 (B6), U92.9 (D6); no longer U91.17 (B1)
- net bus7: now also U91.11 (B7), U92.10 (D7); no longer U91.18 (B0)
- net ~{reset}: now also U92.11 (~{CLR})
- net at U89.3: now also U92.14 (~{CLKEN})
- net at U94.8 (IN0): now also U92.18 (Q4)
- net at U94.1 (IN2): now also U92.17 (Q5)
- net at U94.2 (IN4): now also U92.16 (Q6)
- net at U94.3 (IN8): now also U92.15 (Q7)
- net at U93.8 (IN0): now also U92.22 (Q0)
- net at U93.1 (IN2): now also U92.21 (Q1)
- net at U93.2 (IN4): now also U92.20 (Q2)
- net at U93.3 (IN8): now also U92.19 (Q3)
- new net clk: U92.13 (CLK)
Other:
- note added: "different register"
- note added: "order"
- moved on the sheet: U89A

Commit message: ttl fpga: factorization works in sim and fpga
Other:
- note removed: "different register"
Changed lines of the file:
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@@
-    (stroke (width 0) (type default) (color 0 0 0 0))
-  )
-  (polyline (pts (xy 52.07 88.9) (xy 41.91 88.9))
     (stroke (width 0) (type default) (color 0 0 0 0))
   )
@@
     (stroke (width 0) (type default) (color 0 0 0 0))
   )
-  (polyline (pts (xy 41.91 88.9) (xy 41.91 93.98))
-    (stroke (width 0) (type default) (color 0 0 0 0))
-  )
   (wire (pts (xy 203.2 68.58) (xy 203.2 66.04))
     (stroke (width 0) (type default) (color 0 0 0 0))
@@
   )
   (wire (pts (xy 53.34 45.72) (xy 62.23 45.72))
-    (stroke (width 0) (type default) (color 0 0 0 0))
-  )
-  (polyline (pts (xy 52.07 93.98) (xy 52.07 88.9))
     (stroke (width 0) (type default) (color 0 0 0 0))
   )
@@
     (stroke (width 0) (type default) (color 221 133 0 1))
   )
-  (polyline (pts (xy 41.91 93.98) (xy 52.07 93.98))
-    (stroke (width 0) (type default) (color 0 0 0 0))
-  )
   (wire (pts (xy 124.46 88.9) (xy 128.27 88.9))
     (stroke (width 0) (type default) (color 0 0 0 0))
@@
   )
   (text "Invertierung beachten!" (at 83.82 105.41 0)
-    (effects (font (size 1.27 1.27)) (justify left bottom))
-  )
-  (text "different register" (at 147.32 30.48 0)
     (effects (font (size 1.27 1.27)) (justify left bottom))
   )
@@
     (pin "3")
   )
-  (symbol (lib_id "Switch:SW_Coded_SH-7050") (at 92.71 120.65 0)
+  (symbol (lib_id "Switch:SW_Coded_SH-7050") (at 92.71 120.65 0) (unit 1)
     (in_bom yes) (on_board yes)
     (property "Reference" "SW10" (id 0) (at 94.1578 108.7882 0))
@@
     (pin "C")
   )
-  (symbol (lib_id "Device:R_Network08") (at 121.92 104.14 0)
+  (symbol (lib_id "Device:R_Network08") (at 121.92 104.14 0) (unit 1)
     (in_bom yes) (on_board yes)
     (property "Reference" "RN10" (id 0) (at 131.7752 102.9716 0)
@@
     (pin "9")
   )
-  (symbol (lib_id "power:GND") (at 107.95 114.3 0)
+  (symbol (lib_id "power:GND") (at 107.95 114.3 0) (unit 1)
     (in_bom yes) (on_board yes)
     (property "Reference" "#PWR0294" (id 0) (at 107.95 120.65 0)
@@
     (pin "1")
   )
-  (symbol (lib_id "power:+5V") (at 111.76 99.06 0)
+  (symbol (lib_id "power:+5V") (at 111.76 99.06 0) (unit 1)
     (in_bom yes) (on_board yes)
     (property "Reference" "#PWR0296" (id 0) (at 111.76 102.87 0)
@@
     (pin "1")
   )
-  (symbol (lib_id "Switch:SW_Coded_SH-7050") (at 92.71 139.7 0)
+  (symbol (lib_id "Switch:SW_Coded_SH-7050") (at 92.71 139.7 0) (unit 1)
     (in_bom yes) (on_board yes)
     (property "Reference" "SW11" (id 0) (at 94.1578 127.8382 0))
@@
     (pin "C")
   )
-  (symbol (lib_id "power:GND") (at 107.95 133.35 0)
+  (symbol (lib_id "power:GND") (at 107.95 133.35 0) (unit 1)
     (in_bom yes) (on_board yes)
     (property "Reference" "#PWR0295" (id 0) (at 107.95 139.7 0)

Commit message: io: async register + reversed bus
Parts:
- removed U92: 74AS825, symbol EDiC-rescue:74AS825-74xx
- added U92: 74LS273, symbol 74xx:74LS273
Connections:
- net +5V: now also U92.20 (VCC)
- net GND: now also U92.10 (GND)
- net bus0: now also U91.11 (B7), U92.3 (D0); no longer U91.18 (B0)
- net bus1: now also U91.12 (B6), U92.4 (D1); no longer U91.17 (B1)
- net bus2: now also U91.13 (B5), U92.7 (D2); no longer U91.16 (B2)
- net bus3: now also U91.14 (B4), U92.8 (D3); no longer U91.15 (B3)
- net bus4: now also U91.15 (B3), U92.13 (D4); no longer U91.14 (B4)
- net bus5: now also U91.16 (B2), U92.14 (D5); no longer U91.13 (B5)
- net bus6: now also U91.17 (B1), U92.17 (D6); no longer U91.12 (B6)
- net bus7: now also U91.18 (B0), U92.18 (D7); no longer U91.11 (B7)
- net ~{reset}: now also U92.1 (~{Mr})
- net at U89.3: now also U92.11 (Cp)
- net at U93.1 (IN2): now also U92.5 (Q1)
- net at U93.2 (IN4): now also U92.6 (Q2)
- net at U93.3 (IN8): now also U92.9 (Q3)
- net at U93.8 (IN0): now also U92.2 (Q0)
- net at U94.1 (IN2): now also U92.15 (Q5)
- net at U94.2 (IN4): now also U92.16 (Q6)
- net at U94.3 (IN8): now also U92.19 (Q7)
- net at U94.8 (IN0): now also U92.12 (Q4)
Other:
- note removed: "order"
