File: schematic/CPU-Poster/Memory.sch (KiCad schematic (older format))
At the start: 64 parts, among them SW6 SW_Coded_SH-7050, SW7 SW_Coded_SH-7050, SW8 SW_Coded_SH-7050, SW9 SW_Coded_SH-7050, U100 AS6C4008-55PCN, U103 74LS32, U105 74LS08, U36 74LS08, U38 74LS08, U48 74LS04, U49 74LS245, U50 74LS245, U51 74LS245, U52 74LS245, U53 74F521, U54 74AS867, U55 74AS867, U56 74AS867, U57 74ABT540, U58 74ABT540, U59 74LS08, U60 74F521, U61 74LS245, U62 28C256, U63 74AS825, U64 74AS825, U65 74LS245, U66 74LS245, U67 28C256, U68 74AS825, U69 28C256, U70 74AS825, U71 74AS825, U72 74LS245, U73 74LS245, U74 74LS245, U75 74LS245, U76 74F521, U77 AS6C4008-55PCN, U78 74LS08, U79 74F521, U80 74LS04, U98 74LS245, U99 74LS245

Commit message: started with schematic poster
Parts:
- U53, U60, U76, U79: symbol EDiC-rescue:74F521 -> EDiCPoster-rescue:74F521
- U54, U55, U56: symbol EDiC-rescue:74AS867-74xx -> EDiCPoster-rescue:74AS867-74xx
- U57, U58: symbol EDiC-rescue:74ABT540 -> EDiCPoster-rescue:74ABT540
- U63, U64, U68, U70, U71: symbol EDiC-rescue:74AS825-74xx -> EDiCPoster-rescue:74AS825-74xx
Changed lines of the file:
@@
 $EndComp
 $Comp
-L EDiC-rescue:74AS867-74xx U54
+L EDiCPoster-rescue:74AS867-74xx U54
 U 1 1 614A13D4
 P 8350 4700
@@
 $EndComp
 $Comp
-L EDiC-rescue:74AS867-74xx U55
+L EDiCPoster-rescue:74AS867-74xx U55
 U 1 1 614A1BAD
 P 8350 7650
@@
 	10150 5100 10050 5100
 $Comp
-L EDiC-rescue:74AS867-74xx U56
+L EDiCPoster-rescue:74AS867-74xx U56
 U 1 1 614C84B2
 P 8350 9800
@@
 $EndComp
 $Comp
-L EDiC-rescue:74AS825-74xx U70
+L EDiCPoster-rescue:74AS825-74xx U70
 U 1 1 622368AD
 P 14850 2250
@@
 ~ctrlMemInstrWE~
 $Comp
-L EDiC-rescue:74AS825-74xx U71
+L EDiCPoster-rescue:74AS825-74xx U71
 U 1 1 622CCE3A
 P 15800 4500
@@
 	12750 4300 12900 4300
 $Comp
-L EDiC-rescue:74AS825-74xx U64
+L EDiCPoster-rescue:74AS825-74xx U64
 U 1 1 6255A4D7
 P 12250 4800
@@
 $EndComp
 $Comp
-L EDiC-rescue:74AS825-74xx U63
+L EDiCPoster-rescue:74AS825-74xx U63
 U 1 1 6172F6E1
 P 10700 7650
@@
 $EndComp
 $Comp
-L EDiC-rescue:74AS825-74xx U68
+L EDiCPoster-rescue:74AS825-74xx U68
 U 1 1 61818E6C
 P 13350 7350
@@
 ctrlMemPCFromImm
 $Comp
-L EDiC-rescue:74F521 U53
+L EDiCPoster-rescue:74F521 U53
 U 1 1 616FD36C
 P 8000 12900
@@
 $EndComp
 $Comp
-L EDiC-rescue:74F521 U60
+L EDiCPoster-rescue:74F521 U60
 U 1 1 616FE128
 P 10000 12850
@@
 comp14
 $Comp
-L EDiC-rescue:74F521 U76
+L EDiCPoster-rescue:74F521 U76
 U 1 1 62289ACE
 P 18950 12800
@@
 	19000 12000 18850 12000
 $Comp
-L EDiC-rescue:74F521 U79
+L EDiCPoster-rescue:74F521 U79
 U 1 1 625D2667
 P 21250 12750
@@
 	22650 13300 22300 13300
 $Comp
-L EDiC-rescue:74ABT540 U?
+L EDiCPoster-rescue:74ABT540 U?
 U 1 1 634E144D
 P 8350 17800
@@
 	9350 18000 8950 18000
 $Comp
-L EDiC-rescue:74ABT540 U?
+L EDiCPoster-rescue:74ABT540 U?
 U 1 1 6363F628
 P 8350 19900
