File: schematic/CPU-Poster/EDiCPoster.sch (KiCad schematic (older format))
At the start: 285 parts, among them U1 74ABT540

Commit message: reposition in poster
Other:
- note added: "EDiC - Educational Digital Computer"
- moved on the sheet: D1, D2, D3, D4, D5, D6, D7, D8, D?, RN1, RN2, RN?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
