File: schematic/CPU-Poster/EDiCPoster.kicad_sch (KiCad schematic)
At the start: 285 parts, among them U1 74ABT540

Commit message: poster passed erc, check
Parts:
- removed R? (x7): 1k, symbol Device:R
- removed U? (x3): 74LS08, symbol 74xx:74LS08
- removed U?: 74LS04, symbol 74xx:74LS04
- removed U? (x2): 74LS86, Package_DIP:DIP-14_W7.62mm, symbol 74xx:74LS86
- removed U? (x3): 74LS08, Package_DIP:DIP-14_W7.62mm, symbol 74xx:74LS08
- added R10: 0R0, symbol Device:R
- added R9: 1k, symbol Device:R
- added unit 2 of U103
- added unit 4 of U103
- added unit 3 of U103
- added unit 5 of U103
- added unit 4 of U25
- added unit 3 of U25
- added unit 5 of U25
- added unit 7 of U51
- added unit 5 of U53
- added unit 4 of U53
- added unit 3 of U53
- added unit 3 of U56
- added unit 2 of U56
- added unit 5 of U56
- added unit 4 of U56
- added unit 5 of U57
- added unit 5 of U75
- added unit 4 of U75
- added unit 5 of U80
- added unit 3 of U80
- added unit 2 of U80
- added unit 4 of U80
- added unit 5 of U81
- added unit 2 of U81
- added unit 4 of U81
- added unit 3 of U81
- added unit 4 of U97
- added unit 2 of U97
- added unit 6 of U97
- added unit 5 of U97
- added unit 3 of U97
- added unit 7 of U97
- added unit 5 of U98
- added unit 3 of U98
- added unit 4 of U98
- U58: renamed from U?; value ds1813 -> DS1813
- U75: renamed from U?; footprint Package_DIP:DIP-14_W7.62mm -> (none)
- X1: renamed from X?; value CXO_DIP14 -> 1MHz
- gave numbers to parts that had none: 180
- renumbered U1 to U19
Connections:
- net +5V: now also U1.14 (VCC), U10.14 (VCC), U11.14 (VCC), U12.14 (VCC), U2.14 (VCC), U3.14 (VCC), U4.14 (VCC), U42.14 (VCC), U49.14 (VCC), U5.14 (VCC), U50.14 (VCC), U6.14 (VCC), U7.14 (VCC), U8.14 (VCC), U9.14 (VCC), R9.1, U103.14 (VCC), U25.14 (VCC), U51.14 (VCC), U53.14 (VCC), U56.14 (VCC), U57.14 (VCC), U75.14 (VCC), U80.14 (VCC), U81.14 (VCC), U97.14 (VCC), U98.14 (VCC); no longer U100.1 (A->B), U23.1 (A->B), U24.1 (A->B), U44.1 (A->B), U48.10 (D7), U48.7 (D4), U48.8 (D5), U48.9 (D6), U49.1, U49.1, U49.2, U49.2, U50.1, U50.1, U50.2, U50.2, U54.1 (A->B), U55.1 (A->B), U61.1 (A->B), U62.1 (A->B), U63.12 (I7), U63.13 (I6), U63.14 (I5), U63.15 (I4), U67.27 (~{WE}), U68.27 (~{WE}), U69.27 (~{WE}), U70.1 (A->B), U71.1 (A->B), U75.1, U79.1 (A->B), U82.1 (A->B), U83.1 (A->B), U84.1 (A->B), U86.27 (~{WE}), U87.27 (~{WE}), U89.1 (A->B), U90.1 (A->B), U91.1 (A->B), U92.12 (R4), U92.14 (R5), U92.16 (R6), U92.18 (R7), U92.5 (R1), U92.7 (R2), U92.9 (R3), U93.12 (R4), U93.14 (R5), U93.16 (R6), U93.18 (R7), U93.3 (R0), U93.5 (R1), U93.7 (R2), U93.9 (R3)
- net GND: now also U1.7 (GND), U10.7 (GND), U11.7 (GND), U12.7 (GND), U2.7 (GND), U3.7 (GND), U4.7 (GND), U42.7 (GND), U49.7 (GND), U5.7 (GND), U50.7 (GND), U6.7 (GND), U7.7 (GND), U8.7 (GND), U9.7 (GND), R10.1, U103.7 (GND), U25.7 (GND), U51.7 (GND), U53.7 (GND), U56.7 (GND), U57.7 (GND), U75.7 (GND), U80.7 (GND), U81.7 (GND), U97.7 (GND), U98.7 (GND); no longer U101.4 (BL), U101.5 (LE), U102.4 (BL), U102.5 (LE), U13.1 (~{OE1}), U13.2 (~{OE2}), U13.23 (~{OE3}), U14.1 (~{OE1}), U14.2 (~{OE2}), U14.23 (~{OE3}), U15.15 (E), U16.15 (E), U17.15 (E), U18.15 (E), U19.1 (~{OE1}), U19.19 (~{OE2}), U20.15 (E), U21.13 (I1d), U21.15 (E), U22.7 (~{E}), U26.15 (E), U27.10 (I1c), U27.13 (I1d), U27.15 (E), U28.1 (Ea), U28.15 (Eb), U29.1 (Ea), U29.15 (Eb), U30.1 (Ea), U30.15 (Eb), U31.1 (Ea), U31.15 (Eb), U32.15 (E), U33.10 (I1c), U33.13 (I1d), U33.15 (E), U33.3 (I1a), U33.6 (I1b), U34.1 (~{OE1}), U34.19 (~{OE2}), U35.1 (~{OE1}), U35.19 (~{OE2}), U36.15 (E), U37.15 (E), U38.1 (~{OE1}), U38.19 (~{OE2}), U39.1 (~{OE1}), U39.19 (~{OE2}), U40.1 (~{OE1}), U40.2 (~{OE2}), U40.23 (~{OE3}), U41.1 (G), U41.11 (P4), U41.13 (P5), U41.15 (P6), U41.17 (P7), U41.2 (P0), U41.4 (P1), U41.6 (P2), U41.8 (P3), U43.7 (~{E}), U43.9 (S2), U45.1 (~{OE1}), U45.19 (~{OE2}), U48.1 (~{OE1}), U48.2 (~{OE2}), U48.23 (~{OE3}), U59.11 (~{ENT}), U63.7 (~{E}), U63.9 (S2), U64.1 (~{OE1}), U64.19 (~{OE2}), U65.2 (~{OE2}), U65.23 (~{OE3}), U66.1 (~{OE1}), U66.2 (~{OE2}), U66.23 (~{OE3}), U67.20 (~{CS}), U67.22 (~{OE}), U68.20 (~{CS}), U68.22 (~{OE}), U69.20 (~{CS}), U69.22 (~{OE}), U72.1 (~{OE1}), U72.2 (~{OE2}), U72.23 (~{OE3}), U73.1 (~{OE1}), U73.2 (~{OE2}), U73.23 (~{OE3}), U74.1 (~{OE1}), U74.2 (~{OE2}), U74.23 (~{OE3}), U76.1 (~{OE1}), U76.19 (~{OE2}), U76.6 (A4), U77.1 (~{OE1}), U77.2 (~{OE2}), U77.23 (~{OE3}), U78.1 (OE), U85.10 (D7), U85.11 (~{ENT}), U85.3 (D0), U85.4 (D1), U85.5 (D2), U85.6 (D3), U85.7 (D4), U85.8 (D5), U85.9 (D6), U86.20 (~{CS}), U86.22 (~{OE}), U87.20 (~{CS}), U87.22 (~{OE}), U88.20 (~{CS}), U88.22 (~{OE}), U92.1 (G), U92.3 (R0), U93.1 (G), U94.12 (R4), U94.14 (R5), U94.16 (R6), U94.18 (R7), U94.3 (R0), U94.5 (R1), U94.7 (R2), U94.9 (R3)
- net a0: now also U15.2 (I0a), U16.13 (I1d)
- net a1: now also U15.5 (I0b), U16.10 (I1c), U2.4, U3.4; no longer U2.1, U3.1
- net a2: now also U15.11 (I0c), U16.6 (I1b), U2.9, U3.9; no longer U2.1, U3.1
- net a3: now also U15.14 (I0d), U16.3 (I1a), U2.12, U3.12; no longer U2.1, U3.1
- net a4: now also U15.13 (I1d), U16.2 (I0a)
- net a5: now also U15.10 (I1c), U16.5 (I0b), U8.4, U9.4; no longer U8.1, U9.1
- net a6: now also U15.6 (I1b), U16.11 (I0c), U8.9, U9.9; no longer U8.1, U9.1
- net a7: now also U15.3 (I1a), U16.14 (I0d), U8.12, U9.12; no longer U8.1, U9.1
- net adder1: now also U4.6; no longer U4.3
- net adder2: now also U4.8; no longer U4.3
- net adder3: now also U4.11; no longer U4.3
- net adder5: now also U10.6; no longer U10.3
- net adder6: now also U10.8; no longer U10.3
- net adder7: now also U10.11; no longer U10.3
- net and1: now also U2.6, U6.4; no longer U2.3, U6.1
- net and2: now also U2.8, U6.9; no longer U2.3, U6.1
- net and3: now also U2.11, U6.12; no longer U2.3, U6.1
- net and5: now also U12.4, U8.6; no longer U12.1, U8.3
- net and6: now also U12.9, U8.8; no longer U12.1, U8.3
- net and7: now also U12.12, U8.11; no longer U12.1, U8.3
- net bus1: now also U1.4; no longer U1.1
- net bus2: now also U1.9; no longer U1.1
- net bus3: now also U1.12; no longer U1.1
- net bus5: now also U7.4; no longer U7.1
- net bus6: now also U7.9; no longer U7.1
- net bus7: now also U7.12; no longer U7.1
- net ctrlAluSub: now also U1.10, U1.13, U1.5, U7.10, U7.13, U7.5; no longer U1.2, U1.2, U1.2, U7.2, U7.2, U7.2
- net ctrlMemInstrImmToRamAddr: now also U51.9, U57.12; no longer U51.1, U57.1
- net ctrlMemPCFromImm: now also U51.11; no longer U51.1
- net decodeAddr0: now also U75.4; no longer U75.1
- net decodeAddr1: now also U75.5; no longer U75.2
- net decodeAddr2: now also U75.9; no longer U75.1
- net flagC: now also U10.12, U11.12, U12.8; no longer U10.1, U11.1, U12.3
- net flagCarry: now also U22.4 (I0)
- net flagZ: now also U25.6; no longer U25.3
- net i0: now also U42.4; no longer U42.2
- net i2: now also U42.13; no longer U42.1
- net r0: now also U42.6; no longer U42.2
- net s3: now also U42.11; no longer U42.1
- net s4: now also U50.6; no longer U50.3
- net selectStackMem: now also U51.3; no longer U51.1
- net xor1: now also U3.6, U4.5, U5.5; no longer U3.3, U4.2, U5.2
- net xor2: now also U3.8, U4.10, U5.10; no longer U3.3, U4.2, U5.2
- net xor3: now also U3.11, U4.13, U5.13; no longer U3.3, U4.2, U5.2
- net xor5: now also U10.5, U11.5, U9.6; no longer U10.2, U11.2, U9.3
- net xor6: now also U10.10, U11.10, U9.8; no longer U10.2, U11.2, U9.3
- net xor7: now also U10.13, U11.13, U9.11; no longer U10.2, U11.2, U9.3
- net ~{breakpointEnable}: now also U42.8; no longer U42.2
- net ~{ctrlInstrFinished}: now also U49.5; no longer U49.2
- net ~{ctrlMemPCLoad}: now also U57.4; no longer U57.1
- net ~{ctrlMemRamOE}: now also U98.5; no longer U98.2
- net ~{instrImm0ToRam}: now also U51.8, U57.9; no longer U51.2, U57.1
- net ~{instrImm1ToRam}: now also U51.6; no longer U51.2
- net ~{mar1ToRam}: now also U51.12; no longer U51.2
- net ~{reset}: now also U53.5, U57.5; no longer U53.2, U57.2
- net ~{spToRam}: now also U51.4, U57.10, U57.13; no longer U51.2, U57.2, U57.2
- net GNDREF: now reaches U43.12 (I7)
- net GNDREF: now also U101.4 (BL), U101.5 (LE), U102.4 (BL), U102.5 (LE), U13.1 (~{OE1}), U13.2 (~{OE2}), U13.23 (~{OE3}), U14.1 (~{OE1}), U14.2 (~{OE2}), U14.23 (~{OE3}), U15.15 (E), U16.15 (E), U17.15 (E), U18.15 (E), U19.1 (~{OE1}), U19.19 (~{OE2}), U20.15 (E), U21.13 (I1d), U21.15 (E), U22.7 (~{E}), U26.15 (E), U27.10 (I1c), U27.13 (I1d), U27.15 (E), U28.1 (Ea), U28.15 (Eb), U29.1 (Ea), U29.15 (Eb), U30.1 (Ea), U30.15 (Eb), U31.1 (Ea), U31.15 (Eb), U32.15 (E), U33.10 (I1c), U33.13 (I1d), U33.15 (E), U33.3 (I1a), U33.6 (I1b), U34.1 (~{OE1}), U34.19 (~{OE2}), U35.1 (~{OE1}), U35.19 (~{OE2}), U36.15 (E), U37.15 (E), U38.1 (~{OE1}), U38.19 (~{OE2}), U39.1 (~{OE1}), U39.19 (~{OE2}), U40.1 (~{OE1}), U40.2 (~{OE2}), U40.23 (~{OE3}), U41.1 (G), U41.11 (P4), U41.13 (P5), U41.15 (P6), U41.17 (P7), U41.2 (P0), U41.4 (P1), U41.6 (P2), U41.8 (P3), U43.13 (I6), U43.14 (I5), U43.15 (I4), U43.7 (~{E}), U43.9 (S2), U45.1 (~{OE1}), U45.19 (~{OE2}), U48.1 (~{OE1}), U48.2 (~{OE2}), U48.23 (~{OE3}), U49.10, U49.12, U49.13, U49.9, U50.10, U50.12, U50.13, U50.9, U59.11 (~{ENT}), U63.7 (~{E}), U63.9 (S2), U64.1 (~{OE1}), U64.19 (~{OE2}), U65.2 (~{OE2}), U65.23 (~{OE3}), U66.1 (~{OE1}), U66.2 (~{OE2}), U66.23 (~{OE3}), U67.20 (~{CS}), U67.22 (~{OE}), U68.20 (~{CS}), U68.22 (~{OE}), U69.20 (~{CS}), U69.22 (~{OE}), U72.1 (~{OE1}), U72.2 (~{OE2}), U72.23 (~{OE3}), U73.1 (~{OE1}), U73.2 (~{OE2}), U73.23 (~{OE3}), U74.1 (~{OE1}), U74.2 (~{OE2}), U74.23 (~{OE3}), U76.1 (~{OE1}), U76.19 (~{OE2}), U76.6 (A4), U77.1 (~{OE1}), U77.2 (~{OE2}), U77.23 (~{OE3}), U78.1 (OE), U85.10 (D7), U85.11 (~{ENT}), U85.3 (D0), U85.4 (D1), U85.5 (D2), U85.6 (D3), U85.7 (D4), U85.8 (D5), U85.9 (D6), U86.20 (~{CS}), U86.22 (~{OE}), U87.20 (~{CS}), U87.22 (~{OE}), U88.20 (~{CS}), U88.22 (~{OE}), U92.1 (G), U92.3 (R0), U93.1 (G), U94.12 (R4), U94.14 (R5), U94.16 (R6), U94.18 (R7), U94.3 (R0), U94.5 (R1), U94.7 (R2), U94.9 (R3), U95.1 (A18), U95.30 (A17), U96.1 (A18), U96.30 (A17), R10.2, U103.10, U103.12, U103.13, U103.4, U103.5, U103.9, U25.10, U25.12, U25.13, U25.9, U53.10, U53.12, U53.13, U53.9, U56.10, U56.12, U56.13, U56.4, U56.5, U56.9, U75.12, U75.13, U80.10, U80.12, U80.13, U80.4, U80.5, U80.9, U81.10, U81.12, U81.13, U81.4, U81.5, U81.9, U97.11, U97.13, U97.3, U97.5, U97.9, U98.10, U98.12, U98.13, U98.9
- net at U10.1, U11.1: now also U6.11; no longer U6.3
- net at U25.2: now also U12.11; no longer U12.3
- net at U59.1 (S0), U60.1 (S0): now also U57.6; no longer U57.3
- net at U54.19 (CE), U55.19 (CE): now also U51.10; no longer U51.2
- net at U94.19 (P=R), U98.1: now also U98.4; no longer U98.1
- net at U100.19 (CE): now also U98.6; no longer U98.3
- net at U103.3: now also U53.4; no longer U53.1
- net at U77.11 (~{CLR}): now also U53.6; no longer U53.3
- net HT: now reaches U88.27 (~{WE})
- net HT: now also U100.1 (A->B), U23.1 (A->B), U24.1 (A->B), U44.1 (A->B), U48.10 (D7), U48.7 (D4), U48.8 (D5), U48.9 (D6), U54.1 (A->B), U55.1 (A->B), U61.1 (A->B), U62.1 (A->B), U63.12 (I7), U63.13 (I6), U63.14 (I5), U63.15 (I4), U67.27 (~{WE}), U68.27 (~{WE}), U69.27 (~{WE}), U70.1 (A->B), U71.1 (A->B), U75.1, U77.6 (D3), U79.1 (A->B), U82.1 (A->B), U83.1 (A->B), U84.1 (A->B), U86.27 (~{WE}), U87.27 (~{WE}), U89.1 (A->B), U90.1 (A->B), U91.1 (A->B), U92.12 (R4), U92.14 (R5), U92.16 (R6), U92.18 (R7), U92.5 (R1), U92.7 (R2), U92.9 (R3), U93.12 (R4), U93.14 (R5), U93.16 (R6), U93.18 (R7), U93.3 (R0), U93.5 (R1), U93.7 (R2), U93.9 (R3), R9.2
- net at U77.4 (D1): now also U75.6; no longer U75.3
- net at U77.5 (D2): now also U75.8; no longer U75.3
- net at U53.3: now also U75.10; no longer U75.2
- net at C3.1, R7.1: now also U42.3; no longer U42.1
- net at C4.1, R8.1: now also U42.5; no longer U42.1
- net at C1.1, R5.1: now also U42.9; no longer U42.1
- net at U49.2: now also U42.10; no longer U42.2
- net at U50.3: now also U49.4; no longer U49.1
- net spS1: no longer names the net of U80.3, U85.2 (S1)
- net ~{spEn}: no longer names the net of U81.3, U85.23 (~{ENP})
- new net: U25.4, U25.5, U41.19 (P=R)
- new net: U4.4, U5.4, U6.3
- new net: U1.6, U2.5, U3.5
- new net: U5.6, U6.5
- new net: U4.9, U5.9, U6.6
- new net: U1.8, U2.10, U3.10
- new net: U5.8, U6.10
- new net: U4.12, U5.12, U6.8
- new net: U1.11, U2.13, U3.13
- new net: U5.11, U6.13
- new net: U10.4, U11.4, U12.3
- new net: U7.6, U8.5, U9.5
- new net: U11.6, U12.5
- new net: U10.9, U11.9, U12.6
- new net: U7.8, U8.10, U9.10
- new net: U11.8, U12.10
- new net: U7.11, U8.13, U9.13
- new net: U11.11, U12.13
- new net: U51.13, U57.8
- new net: U51.5, U57.11
- new net: U49.6, U50.4
- new net: U42.12, U50.5
- no-connect marks 33 -> 46
Other:
- note added: "24bit instructions: rom2 23:16 - instruction to decode rom1&0 15:0 - immediateValue: 7:0 data for ALU Operation or Registers 15:0 address for Program Counter (jump) or RAM (memory OP)"
- note removed: "24bit instructions: rom2 23:16 - instruction to decode rom1&0 15:0 - immediate: 7:0 data for ALU OP or reg 15:0 address for PC (jump) or RAM (memory OP)"
- moved on the sheet: C1, C2, C3, C4, D25, D26, D27, D28, D29, D30, D31, D32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

Commit message: started anotating poster
Parts:
- removed unit 2 of U103
- removed unit 4 of U103
- removed unit 3 of U103
- removed unit 5 of U103
- removed unit 3 of U56
- removed unit 2 of U56
- removed unit 5 of U81
- removed unit 2 of U81
- removed unit 4 of U81
- removed unit 3 of U81
- renumbered U81 to U56, U103 to U56
Connections:
- net halt: now also U56.10, U56.5; no longer U56.2, U56.2
- net ~{ctrlInstrFinished}: now also U56.9; no longer U56.1
- net ~{ctrlMemSPEn}: now also U56.4; no longer U56.1
- net at U85.23 (~{ENP}): now also U56.6; no longer U56.3
- net at U53.4: now also U56.8; no longer U56.3
- no-connect marks 46 -> 38
Other:
- note added: "ALU Result"
- note added: "ALU Result Flags"
- note added: "ALU Select"
- note added: "Adder Bit0"
- note added: "Adder Bit1"
- note added: "Adder Bit2"
- note added: "Adder Bit3"
- note added: "Adder Bit4"
- note added: "Adder Bit5"
- note added: "Adder Bit6"
- note added: "Adder Bit7"
- note added: "Address for the memory: bits 7..0 -> MAR[ 7..0] or Instruction Immediate Value bits 15..0 -> MAR[15..0] or Instruction Immediate Value or Stack Pointer"
- note added: "Barrel Shifter"
- note added: "Carry Flag Shifter"
- note added: "Clock/Reset & Debug User Interface"
- note added: "Instruction Step Counter & Instruction Decoder"
- note added: "Memory Address Registers"
- note added: "Power & Ground"
- note added: "Program Counter & Breakpoint Detection"
- note added: "Registers"
- note removed: "Invertierung beachten!"
- note removed: "ramAddress: 7:0 -> instrImm or mar0 (depending on ctrlMemInstrImmToRamAddr) 15:0 -> instrImm or mar1 or sp (depending on ctrlMemInstrImmToRam and selectStackMem)"
- moved on the sheet: C1, C2, C3, C4, D1, D10, D11, D12, D13, D14, D15, D16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

Commit message: restructured folders
Parts:
- removed unit 2 of U51
- removed U70, U71: 74LS245, symbol 74xx:74LS245
- removed unit 4 of U97
- removed unit 2 of U97
- removed unit 6 of U97
- removed unit 5 of U97
- removed unit 3 of U97
- removed unit 7 of U97
- added J1: IOExpansion-33Pins, symbol Connector_Generic:Conn_2Rows-33Pins
- added U? (x2): 74LS245, symbol 74xx:74LS245
- renumbered U101 to U100, U102 to U101, U97 to U51, U98 to U97, U99 to U98, U100 to U99
Connections:
- net selectStackMem is gone; now on net ~{spToRam}: U93.19 (P=R), U95.2 (A16), U96.2 (A16)
- net +5V: now also J1.11 (Pin_11), J1.17 (Pin_17), J1.2 (Pin_2), J1.5 (Pin_5), J1.8 (Pin_8), U?.20 (VCC), U?.20 (VCC)
- net GND: now also J1.14 (Pin_14), J1.20 (Pin_20), J1.23 (Pin_23), J1.26 (Pin_26), J1.29 (Pin_29), J1.30 (Pin_30), J1.33 (Pin_33), U?.10 (GND), U?.10 (GND)
- net HT: now also U?.1 (A->B), U?.1 (A->B)
- net bus0: now also J1.4 (Pin_4), U?.18 (B0)
- net bus1: now also J1.6 (Pin_6), U?.17 (B1)
- net bus2: now also J1.10 (Pin_10), U?.16 (B2)
- net bus3: now also J1.12 (Pin_12), U?.15 (B3)
- net bus4: now also J1.16 (Pin_16), U?.14 (B4)
- net bus5: now also J1.18 (Pin_18), U?.13 (B5)
- net bus6: now also J1.22 (Pin_22), U?.12 (B6)
- net bus7: now also J1.24 (Pin_24), U?.11 (B7)
- net clk: now also J1.32 (Pin_32)
- net pc0: now also U?.2 (A0)
- net pc1: now also U?.3 (A1)
- net pc10: now also U?.4 (A2)
- net pc11: now also U?.5 (A3)
- net pc12: now also U?.6 (A4)
- net pc13: now also U?.7 (A5)
- net pc14: now also U?.8 (A6)
- net pc15: now also U?.9 (A7)
- net pc2: now also U?.4 (A2)
- net pc3: now also U?.5 (A3)
- net pc4: now also U?.6 (A4)
- net pc5: now also U?.7 (A5)
- net pc6: now also U?.8 (A6)
- net pc7: now also U?.9 (A7)
- net pc8: now also U?.2 (A0)
- net pc9: now also U?.3 (A1)
- net ram2data0: now also U?.18 (B0)
- net ram2data1: now also U?.17 (B1)
- net ram2data2: now also U?.16 (B2)
- net ram2data3: now also U?.15 (B3)
- net ram2data4: now also U?.14 (B4)
- net ram2data5: now also U?.13 (B5)
- net ram2data6: now also U?.12 (B6)
- net ram2data7: now also U?.11 (B7)
- net ~{ctrlMemPCToRam}: now also U51.3, U?.19 (CE), U?.19 (CE); no longer U51.1
- net ~{ctrlMemRamOE}: now also J1.27 (Pin_27)
- net ~{ctrlMemRamWE}: now also J1.25 (Pin_25)
- net ~{reset}: now also J1.31 (Pin_31)
- net at U96.24 (OE#): now also U51.4; no longer U51.2
- net ioAddr0 renamed ramAddress0
- net ramAddress0: now also J1.1 (Pin_1)
- net ioAddr1 renamed ramAddress1
- net ramAddress1: now also J1.3 (Pin_3)
- net ioAddr2 renamed ramAddress2
- net ramAddress2: now also J1.7 (Pin_7)
- net ioAddr3 renamed ramAddress3
- net ramAddress3: now also J1.9 (Pin_9)
- net ioAddr4 renamed ramAddress4
- net ramAddress4: now also J1.13 (Pin_13)
- net ioAddr5 renamed ramAddress5
- net ramAddress5: now also J1.15 (Pin_15)
- net ioAddr6 renamed ramAddress6
- net ramAddress6: now also J1.19 (Pin_19)
- net ioAddr7 renamed ramAddress7
- net ramAddress7: now also J1.21 (Pin_21)
- net ioSelect renamed ~{ioCE}
- net ~{ioCE}: now also J1.28 (Pin_28)
- no-connect marks 38 -> 33
Other:
- note added: "24bit instructions: rom2 23:16 - instruction to decode rom1&0 15: 0 - immediateValue: - 15:0 address for Program Counter (jump) or RAM (Memory Oeration) - 7:0 data for ALU Operation or Registers"
- note added: "Address == 0x00"
- note added: "Address Map: 0x0000 - 0xfdff: usual RAM 0xfe00 - 0xfeff: Memory Mapped IO 0xff00 - 0xffff: Stack / Function Local RAM"
- note added: "Breakpoint Detection & Program Counter LEDs"
- note added: "Built-In IO for testing"
- note added: "IO Connector"
- note added: "Instruction EEPROMs"
- note added: "Memory Address Select Logic"
- note added: "Memory Address: bits 7..0 -> MAR[ 7..0] or Instruction Immediate Value bits 15..0 -> MAR[15..0] or Instruction Immediate Value or Stack Pointer"
- note added: "Program Counter"
- note added: "Stack Pointer & Second RAM for Function Calls"
- note added: "This CPU has the following features: - 8 bit Data Bus - ALU with Add and Shift Unit - 16 bit Address Bus - 2 general purpose 8 bit Registers - 16 bit Program Counter for 24 bit Instructions - 8 bit Stack Pointer for Function Local Memory - 256 8 bit General Purpose Memory Mapped Inputs and Outputs"
- note added: "Unused Logic Components"
- note added: "select == 0xfe: io select == 0xff: stack otherwise: ram"
- note removed: "24bit instructions: rom2 23:16 - instruction to decode rom1&0 15:0 - immediateValue: 7:0 data for ALU Operation or Registers 15:0 address for Program Counter (jump) or RAM (memory OP)"
- note removed: "Address for the memory: bits 7..0 -> MAR[ 7..0] or Instruction Immediate Value bits 15..0 -> MAR[15..0] or Instruction Immediate Value or Stack Pointer"
- note removed: "Program Counter & Breakpoint Detection"
- note removed: "ioAddress == 0x00"
- note removed: "select == 0xff: stack select == 0xfe: io otherwise: ram"
- note removed: "~{instrImm0ToRam}=~{ctrlMemInstrImmToRamAddr} ~{instrImm1ToRam}=!(~{ctrlMemInstrImmToRam} and ~{selectStackMem}) ~{mar1ToRam}=!(ctrlMemInstrImmToRam and ~{selectStackMem})"
- moved on the sheet: U25C, U25D, U49C, U49D, U50C, U50D, U53C, U53D, U56B, U56D, U75D, U80A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

Commit message: netlist2verilog converter started
Other:
- note added: "Bus Pull-Up + LEDs"
- note added: "Simple Built-In IO for Address 0x00"
- note added: "This CPU has the following features: - 8 bit Data Bus - ALU with Add and Shift Unit - 16 bit Address Bus (64kByte RAM + 64k Instructions) - 2 general purpose 8 bit Registers - 16 bit Program Counter for 24 bit Instructions - 8 bit Stack Pointer - 256 8 bit General Purpose Memory Mapped Inputs and Outputs"
- note removed: "Built-In IO for testing"
- note removed: "This CPU has the following features: - 8 bit Data Bus - ALU with Add and Shift Unit - 16 bit Address Bus - 2 general purpose 8 bit Registers - 16 bit Program Counter for 24 bit Instructions - 8 bit Stack Pointer for Function Local Memory - 256 8 bit General Purpose Memory Mapped Inputs and Outputs"
- moved on the sheet: U25A, U25C, U25D, U49C, U49D, U50C, U50D, U53C, U53D, U56D, U75D, U80B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
